File: hardware/ETH1CLCR2/Ethernet.sch (KiCad schematic (older format))
At the start: 43 parts, among them U301 LC03-3.3, U302 LAN8742A, U303 LC03-3.3, Y301 NX5032GA-25.000M-LN-CD-1

Commit message: Footprints assigned.
Parts:
- renumbered C301 to C201, C302 to C202, C303 to C203, C304 to C204, C305 to C205, C306 to C206, C307 to C207, C308 to C208, C309 to C209, C310 to C210, C311 to C211, C312 to C212, C313 to C213, C314 to C214, D301 to D201, D302 to D202, FB301 to FB201, L301 to L201, R301 to R201, R302 to R202, R303 to R203, R304 to R204, R305 to R205, R306 to R206, R307 to R207, R308 to R208, R309 to R209, R310 to R210, R311 to R211, R312 to R212, R313 to R213, R314 to R214, R315 to R215, R316 to R216, R317 to R217, R318 to R218, R319 to R219, R320 to R220, R321 to R221, U301 to U201, U302 to U202, U303 to U203, Y301 to Y201
