File: hardware/ETH1CLCR2/FGEN.sch (KiCad schematic (older format))
At the start: 77 parts, among them Q801 BC847, Q802 BC847, Q803 BC857, Q804 BC847, Q805 BC857, Q806 BC857, U901 LM318, U902 AD5452YRMZ, U903 LT1468, U904 MC33078, U905 AD9835, U906 ECS-3225SMV-500-GP-TR, U907 74AHCT1G08, U908 REF192, U909 TL072, U910 AD5689BRUZ

Commit message: Schematic design
Parts:
- removed C807: 220n, Capacitor_SMD:C_0603_1608Metric_Pad1.08x0.95mm_HandSolder, symbol Device:C
- removed C808: 1n, symbol Device:C
- removed C919, C920: 100n, Capacitor_SMD:C_0603_1608Metric_Pad1.08x0.95mm_HandSolder, symbol Device:C
- removed unit 1 of D901
- removed unit 2 of D901
- removed R823: 1k/.1%, Resistor_SMD:R_0603_1608Metric_Pad0.98x0.95mm_HandSolder, symbol Device:R
- removed R824: 24k9/.1%, Resistor_SMD:R_0603_1608Metric_Pad0.98x0.95mm_HandSolder, symbol Device:R
- removed R825: 100k/.1%, Resistor_SMD:R_0603_1608Metric_Pad0.98x0.95mm_HandSolder, symbol Device:R
- removed R826: 33k2/.1%, Resistor_SMD:R_0603_1608Metric_Pad0.98x0.95mm_HandSolder, symbol Device:R
- removed R911, R912: 1k96/.1%, Resistor_SMD:R_0603_1608Metric_Pad0.98x0.95mm_HandSolder, symbol Device:R
- removed R913, R916: 0, Resistor_SMD:R_0603_1608Metric_Pad0.98x0.95mm_HandSolder, symbol Device:R
- removed R914, R915: 10k, Resistor_SMD:R_0603_1608Metric_Pad0.98x0.95mm_HandSolder, symbol Device:R
- removed U909: TL072, Package_SO:SOIC-8_3.9x4.9mm_P1.27mm, symbol Amplifier_Operational:TL072
- removed U910: AD5689BRUZ, Package_SO:TSSOP-16_4.4x5mm_P0.65mm, symbol Analog_DAC:AD5689BRUZ
- R814, R815, R819, R820: value 22/1W -> 22/0.5W
- R817: value 10/1W -> 10/0.5W
Connections:
- net labels removed: DDS_DAC_RSTSEL, DDS_DAC_SCLK, DDS_DAC_SDIN, DDS_DAC_SDO, DDS_DAC_~LDAC, DDS_DAC_~RESET, DDS_DAC_~SYNC
- wire segments 292 -> 226
Other:
- moved on the sheet: C806, C901, C902, C903, C904, C905, C906, C907, C908, C909, C910, C911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

Commit message: Footprints assigned.
Parts:
- removed R809: 0, Resistor_SMD:R_0603_1608Metric_Pad0.98x0.95mm_HandSolder, symbol Device:R
- added TP1201, TP1202, TP1203: TestPoint, TestPoint:TestPoint_Plated_Hole_D2.0mm, symbol Connector:TestPoint
- added U1208: DG419LDY, Package_SO:SOIC-8_3.9x4.9mm_P1.27mm, symbol Analog_Switch:DG419LDY
- added U1209: SN74LVC1T45DBV, Package_TO_SOT_SMD:SOT-23-6, symbol Logic_LevelTranslator:SN74LVC1T45DBV
- C1207: renamed from C806; footprint (none) -> Capacitor_SMD:C_0603_1608Metric_Pad1.08x0.95mm_HandSolder
- R1211: renamed from R810; footprint (none) -> Resistor_SMD:R_0603_1608Metric_Pad0.98x0.95mm_HandSolder
- R1212: renamed from R811; footprint (none) -> Resistor_SMD:R_0603_1608Metric_Pad0.98x0.95mm_HandSolder
- R1213: renamed from R812; footprint (none) -> Resistor_SMD:R_0603_1608Metric_Pad0.98x0.95mm_HandSolder
- R1214: renamed from R813; footprint (none) -> Resistor_SMD:R_0603_1608Metric_Pad0.98x0.95mm_HandSolder
- R1215: renamed from R814; footprint (none) -> Resistor_SMD:R_1206_3216Metric_Pad1.30x1.75mm_HandSolder
- R1216: renamed from R815; footprint (none) -> Resistor_SMD:R_1206_3216Metric_Pad1.30x1.75mm_HandSolder
- R1217: renamed from R816; footprint (none) -> Resistor_SMD:R_0603_1608Metric_Pad0.98x0.95mm_HandSolder
- R1218: renamed from R817; footprint (none) -> Resistor_SMD:R_1206_3216Metric_Pad1.30x1.75mm_HandSolder
- R1219: renamed from R818; footprint (none) -> Resistor_SMD:R_0603_1608Metric_Pad0.98x0.95mm_HandSolder
- R1220: renamed from R819; footprint (none) -> Resistor_SMD:R_1206_3216Metric_Pad1.30x1.75mm_HandSolder
- R1221: renamed from R820; footprint (none) -> Resistor_SMD:R_1206_3216Metric_Pad1.30x1.75mm_HandSolder
- R1222: renamed from R821; footprint (none) -> Resistor_SMD:R_0603_1608Metric_Pad0.98x0.95mm_HandSolder
- R1223: renamed from R822; footprint (none) -> Resistor_SMD:R_0603_1608Metric_Pad0.98x0.95mm_HandSolder
- U1204: renamed from U904; footprint (none) -> Package_SO:SOIC-8_3.9x4.9mm_P1.27mm
- renumbered C901 to C1201, C902 to C1202, C903 to C1203, C904 to C1204, C905 to C1205, C906 to C1206, C907 to C1208, C908 to C1209, C909 to C1210, C910 to C1211, C911 to C1212, C912 to C1213, C913 to C1214, C914 to C1215, C915 to C1216, C916 to C1217, C917 to C1218, C918 to C1219, D901 to D1201, L901 to L1201, L902 to L1202, L903 to L1203, Q801 to Q1201, Q802 to Q1202, Q803 to Q1203, Q804 to Q1204, Q805 to Q1205, Q806 to Q1206, R901 to R1201, R902 to R1202, R903 to R1203, R904 to R1204, R905 to R1205, R906 to R1206, R907 to R1207, R908 to R1208, R909 to R1209, R910 to R1210, U901 to U1201, U902 to U1202, U903 to U1203, U905 to U1205, U906 to U1206, U907 to U1207, U908 to U1210
Connections:
- net +3V3: now also U1209.6 (VCCB)
- net +5V: now also U1208.5 (VL), U1209.1 (VCCA)
- net +5VA: now also U1208.4 (V+)
- net -5VA: now also U1208.7 (V-)
- net GND: now also U1208.3 (GND), U1209.2 (GND), U1209.5 (DIR)
- net H_CUR: now also TP1203.1
- net OSC: now also TP1202.1, U1208.2
- net at C1205.1, C1206.2, C1211.1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: now also TP1201.1
- net at C1206.1, R1204.2: now also U1208.1
- new net: U1208.6, U1209.3 (A)
- new net FGEN_SEL: U1209.4 (B)
- no-connect marks 8 -> 9

Commit message: Modification of the function generator schematic.
Parts:
- removed C1214, C1216, C1219: 100n, Capacitor_SMD:C_0603_1608Metric_Pad1.08x0.95mm_HandSolder, symbol Device:C
- removed C1215: 5p, Capacitor_SMD:C_0603_1608Metric_Pad1.08x0.95mm_HandSolder, symbol Device:C
- removed C1217: 10u, Capacitor_SMD:C_0805_2012Metric_Pad1.18x1.45mm_HandSolder, symbol Device:C
- removed C1218: 1u, Capacitor_SMD:C_0603_1608Metric_Pad1.08x0.95mm_HandSolder, symbol Device:C
- removed D1201: SD103ATW, Package_TO_SOT_SMD:SOT-363_SC-70-6, symbol Diode:SD103ATW
- removed Q1201, Q1202, Q1204: BC847, Package_TO_SOT_SMD:SOT-23, symbol Transistor_BJT:BC847
- removed Q1203, Q1205, Q1206: BC857, Package_TO_SOT_SMD:SOT-23, symbol Transistor_BJT:BC857
- removed TP1201, TP1202, TP1203: TestPoint, TestPoint:TestPoint_Plated_Hole_D2.0mm, symbol Connector:TestPoint
- removed U1201: LM318, Package_SO:SOIC-8_3.9x4.9mm_P1.27mm, symbol Amplifier_Operational:LM318M
- removed U1202: AD5452YRMZ, Package_SO:MSOP-8_3x3mm_P0.65mm, symbol ETH1CLCR2:AD545x
- removed U1203: LT1468, Package_SO:SOIC-8_3.9x4.9mm_P1.27mm, symbol ETH1CLCR2:LT1468
- removed U1204: MC33078, Package_SO:SOIC-8_3.9x4.9mm_P1.27mm, symbol Amplifier_Operational:MC33078
- removed U1205: AD9835, Package_SO:TSSOP-16_4.4x5mm_P0.65mm, symbol ETH1CLCR2:AD9835
- removed U1206: ECS-3225SMV-500-GP-TR, ETH1CLCR2:ECS, symbol ETH1CLCR2:ECS-3225SMV
- removed U1207: 74AHCT1G08, Package_TO_SOT_SMD:SOT-353_SC-70-5, symbol ETH1CLCR2:74AHCT1G08
- removed U1208: DG419LDY, Package_SO:SOIC-8_3.9x4.9mm_P1.27mm, symbol Analog_Switch:DG419LDY
- removed U1209: SN74LVC1T45DBV, Package_TO_SOT_SMD:SOT-23-6, symbol Logic_LevelTranslator:SN74LVC1T45DBV
- removed U1210: REF192, Package_SO:SSOP-8_3.9x5.05mm_P1.27mm, symbol Reference_Voltage:REF192
- added D1201, D1202: D, symbol Device:D
- added D1204, D1205, D1206, D1207: 5V6, symbol Device:D_Zener
- added FB1201: Ferrite_Bead_Small, symbol Device:Ferrite_Bead_Small
- added FB1202: Ferrite, symbol Device:Ferrite_Bead_Small
- added L1204: 10u, symbol Device:L
- added Q?: FDV301N, symbol Device:Q_NMOS_GSD
- added R1224, R1225, R? (x6): 150, symbol Device:R
- added R1226: 33, symbol Device:R
- added R1227: 100, symbol Device:R
- added R1228: 220, symbol Device:R
- added R1229: 100k, symbol Device:R
- added R?: 4k7, symbol Device:R
- added R? (x2): 47k, symbol Device:R
- added R? (x2): 2k2, symbol Device:R
- added RV1201: 100k, symbol Device:R_POT
- added U1201: AD9834, Package_SO:TSSOP-20_4.4x6.5mm_P0.65mm, symbol Interface:AD9834
- added U1202, U1204: AD8038, symbol ETH1CLCR2:AD8038
- added U1203: DAC7811, symbol ETH1CLCR2:DAC7811
- added U1205, U1206: LMH6639, symbol ETH1CLCR2:LMH6639
- added U1207: DG409, symbol ETH1CLCR2:DG409
- added U1208: AP1117-ADJ, Package_TO_SOT_SMD:SOT-223-3_TabPin2, symbol Regulator_Linear:AP1117-ADJ
- added U? (x3): LM393, symbol Comparator:LM393
- C1201: value 1p5 -> 4u7; footprint Capacitor_SMD:C_0603_1608Metric_Pad1.08x0.95mm_HandSolder -> (none)
- C1202: value 10n -> 100n; footprint Capacitor_SMD:C_0603_1608Metric_Pad1.08x0.95mm_HandSolder -> (none)
- C1203: value 4p7 -> 100p; footprint Capacitor_SMD:C_0603_1608Metric_Pad1.08x0.95mm_HandSolder -> (none)
- C1204: value 18p -> 4u7; footprint Capacitor_SMD:C_0603_1608Metric_Pad1.08x0.95mm_HandSolder -> (none)
- C1205: value 12p -> 68p; footprint Capacitor_SMD:C_0603_1608Metric_Pad1.08x0.95mm_HandSolder -> (none)
- C1206: value 10u -> 100p; footprint Capacitor_SMD:C_1206_3216Metric_Pad1.33x1.80mm_HandSolder -> (none)
- C1207: value 1u -> 4u7; footprint Capacitor_SMD:C_0603_1608Metric_Pad1.08x0.95mm_HandSolder -> (none)
- C1208: value 22p -> 3p3; footprint Capacitor_SMD:C_0603_1608Metric_Pad1.08x0.95mm_HandSolder -> (none)
- C1209, C1210: value 56p -> 100n; footprint Capacitor_SMD:C_0603_1608Metric_Pad1.08x0.95mm_HandSolder -> (none)
- C1211: value 22p -> 10u; footprint Capacitor_SMD:C_0603_1608Metric_Pad1.08x0.95mm_HandSolder -> (none)
- C1212: value 100n -> 10u; footprint Capacitor_SMD:C_0603_1608Metric_Pad1.08x0.95mm_HandSolder -> (none)
- C1213: footprint Capacitor_SMD:C_0603_1608Metric_Pad1.08x0.95mm_HandSolder -> (none)
- L1201, L1202, L1203: value 4u7 -> 10u; footprint Inductor_SMD:L_0603_1608Metric_Pad1.05x0.95mm_HandSolder -> (none)
- R1201: value 10k -> 6k8; footprint Resistor_SMD:R_0603_1608Metric_Pad0.98x0.95mm_HandSolder -> (none)
- R1202: value 1k -> 2k; footprint Resistor_SMD:R_0603_1608Metric_Pad0.98x0.95mm_HandSolder -> (none)
- R1203: value 1k -> 200; footprint Resistor_SMD:R_0603_1608Metric_Pad0.98x0.95mm_HandSolder -> (none)
- R1204: value 0 -> R; footprint Resistor_SMD:R_0603_1608Metric_Pad0.98x0.95mm_HandSolder -> (none)
- R1205: value 300 -> 200; footprint Resistor_SMD:R_0603_1608Metric_Pad0.98x0.95mm_HandSolder -> (none)
- R1206: value 300 -> R; footprint Resistor_SMD:R_0603_1608Metric_Pad0.98x0.95mm_HandSolder -> (none)
- R1207: value 1k/.1% -> R; footprint Resistor_SMD:R_0805_2012Metric_Pad1.20x1.40mm_HandSolder -> (none)
- R1208: value xxk/.1% -> 200; footprint Resistor_SMD:R_0805_2012Metric_Pad1.20x1.40mm_HandSolder -> (none)
- R1209: value 3k9 -> 100k; footprint Resistor_SMD:R_0603_1608Metric_Pad0.98x0.95mm_HandSolder -> (none)
- R1210: value 0 -> 220; footprint Resistor_SMD:R_0603_1608Metric_Pad0.98x0.95mm_HandSolder -> (none)
- R1211: value 1k/.1% -> 680; footprint Resistor_SMD:R_0603_1608Metric_Pad0.98x0.95mm_HandSolder -> (none)
- R1212: value 4k22/.1% -> 220; footprint Resistor_SMD:R_0603_1608Metric_Pad0.98x0.95mm_HandSolder -> (none)
- R1213: value 22k/.1% -> 68; footprint Resistor_SMD:R_0603_1608Metric_Pad0.98x0.95mm_HandSolder -> (none)
- R1214: value 3k9/.1% -> 33; footprint Resistor_SMD:R_0603_1608Metric_Pad0.98x0.95mm_HandSolder -> (none)
- R1215, R1221: value 22/0.5W -> 100; footprint Resistor_SMD:R_1206_3216Metric_Pad1.30x1.75mm_HandSolder -> (none)
- R1216: value 22/0.5W -> 200; footprint Resistor_SMD:R_1206_3216Metric_Pad1.30x1.75mm_HandSolder -> (none)
- R1217: value 470/.1% -> 330; footprint Resistor_SMD:R_0603_1608Metric_Pad0.98x0.95mm_HandSolder -> (none)
- R1218: value 10/0.5W -> 330; footprint Resistor_SMD:R_1206_3216Metric_Pad1.30x1.75mm_HandSolder -> (none)
- R1219: value 470/.1% -> 680; footprint Resistor_SMD:R_0603_1608Metric_Pad0.98x0.95mm_HandSolder -> (none)
- R1220: value 22/0.5W -> 680; footprint Resistor_SMD:R_1206_3216Metric_Pad1.30x1.75mm_HandSolder -> (none)
- R1222: value 22k/.1% -> 100; footprint Resistor_SMD:R_0603_1608Metric_Pad0.98x0.95mm_HandSolder -> (none)
- R1223: value 1k/.1% -> 150; footprint Resistor_SMD:R_0603_1608Metric_Pad0.98x0.95mm_HandSolder -> (none)
Connections:
- net labels added: +5VF, -5VF, AGNDF, GNDA, MCLK
- net labels removed: +2V5REF, +3.3V, +5VA, -5VA, DDS_AMPL, DDS_FGEN_FSELECT, DDS_FGEN_PSEL0, DDS_FGEN_PSEL1, DDS_FGEN_SCLK, DDS_FGEN_SDATA, DDS_FGEN_~FSYNC, DDS_MDAC_DIN, DDS_MDAC_SCLK, DDS_MDAC_~SYNC, FGEN_SEL, H_CUR, OSC
- wire segments 246 -> 276
- no-connect marks 9 -> 3

Commit message: Schematic
Parts:
- added C? (x2): CP, symbol Device:CP
- added D? (x2): D, symbol Device:D
- added K?: TQ2SA-5V, symbol ETH1CLCR2:TQ2SA-5V
- added R1239, R1240: 15k, symbol Device:R
- added R?: R, symbol Device:R
- added R? (x2): 1M, symbol Device:R
- gave numbers to parts that had none: 13
Connections:
- net labels added: +5VA, -5VA
- wire segments 276 -> 321
Other:
- moved on the sheet: C1211, C1212, R1226, R1227, R1228, R1231, R1232, R1233, R1234, R1235, R1236, R1237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
