File: hardware/ETH1CLCR2/IV_Converter.sch (KiCad schematic (older format))
At the start: 74 parts, among them K701 TQ2SA-5V, Q701 MMBFJ309LT1G, Q702 MMBFJ309LT1G, Q703 BC847, Q704 BC857, Q705 BC847

Commit message: Project based on https://hackaday.io/project/165409-precision-impedance-meter-asdflcr1
Parts:
- added R732: 0, symbol Device:R
- added R733: DNP, symbol Device:R
- added U701: ADA4817-1ARDZ, symbol ETH1CLCR2:ADA4817-1ARDZ
- gave numbers to parts that had none: 48
- renumbered C704 to C713, D703 to D701, D704 to D702, D701 to D709, D702 to D710, D705 to D711, Q705 to Q717, R708 to R729, R709 to R730, R710 to R731, R711 to R734
Connections:
- net +5VA: now also U701.7 (+), U701.8 (~PD)
- net -5VA: now also U701.4 (-)
- net GND: now also R733.2, U701.3 (INP), U701.9 (PAD)
- net at C702.2, C705.2, C708.2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: now also R732.2, U701.1, U701.2 (INN)
- net at Q701.2 (S), Q705.2 (S), Q709.2 (S)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: now also U701.6
- new net CUR_ZERO: R732.1, R733.1
Other:
- moved on the sheet: C713, R730, R731

Commit message: Schematic design
Parts:
- added C607, C608, C609, C610, C611, C612, C613, C614, C615, C616: 100n, symbol Device:C
- added U603, U604, U605, U606: SN74LVC1T45DBV, Package_TO_SOT_SMD:SOT-23-6, symbol Logic_LevelTranslator:SN74LVC1T45DBV
- C701, C704: value 4N7 -> 4n7
- R731: value 0R1 -> 0R1/.1%
Connections:
- net +5V: now also C607.1, C608.1, C609.1, C610.1, U603.1 (VCCA), U604.1 (VCCA), U605.1 (VCCA), U606.1 (VCCA)
- net +5VA: now also C615.1
- net -5VA: now also C616.1
- net GND: now also C607.2, C608.2, C609.2, C610.2, C611.2, C612.2, C613.2, C614.2, C615.2, C616.2, U603.2 (GND), U603.5 (DIR), U604.2 (GND), U604.5 (DIR), U605.2 (GND), U605.5 (DIR), U606.2 (GND), U606.5 (DIR)
- net IRR1: now also U603.4 (B); no longer R705.2, R707.2
- net IRR2: now also U604.4 (B); no longer R712.2, R714.2
- net IRR3: now also U605.4 (B); no longer R719.2, R721.2
- net IRR4: now also U606.4 (B); no longer R726.2, R728.2
- new net: R705.2, R707.2, U603.3 (A)
- new net: R712.2, R714.2, U604.3 (A)
- new net: R719.2, R721.2, U605.3 (A)
- new net: R726.2, R728.2, U606.3 (A)
- new net +3V3: C611.1, C612.1, C613.1, C614.1, U603.6 (VCCB), U604.6 (VCCB), U605.6 (VCCB), U606.6 (VCCB)
Other:
- moved on the sheet: R731

Commit message: Footprints assigned.
Parts:
- added TP601: TestPoint, TestPoint:TestPoint_Plated_Hole_D2.0mm, symbol Connector:TestPoint
- C601: renamed from C701; footprint (none) -> Capacitor_SMD:C_0603_1608Metric_Pad1.08x0.95mm_HandSolder
- C602: renamed from C702; footprint (none) -> Capacitor_SMD:C_0603_1608Metric_Pad1.08x0.95mm_HandSolder
- C603: renamed from C703; footprint (none) -> Capacitor_SMD:C_0603_1608Metric_Pad1.08x0.95mm_HandSolder
- C604: renamed from C704; footprint (none) -> Capacitor_SMD:C_0603_1608Metric_Pad1.08x0.95mm_HandSolder
- C605: renamed from C705; footprint (none) -> Capacitor_SMD:C_0603_1608Metric_Pad1.08x0.95mm_HandSolder
- C606: renamed from C706; footprint (none) -> Capacitor_SMD:C_0603_1608Metric_Pad1.08x0.95mm_HandSolder
- C607: renamed from C707; footprint (none) -> Capacitor_SMD:C_0603_1608Metric_Pad1.08x0.95mm_HandSolder
- C608: renamed from C708; footprint (none) -> Capacitor_SMD:C_0603_1608Metric_Pad1.08x0.95mm_HandSolder
- C609: renamed from C709; footprint (none) -> Capacitor_SMD:C_0603_1608Metric_Pad1.08x0.95mm_HandSolder
- C610: renamed from C710; footprint (none) -> Capacitor_SMD:C_0603_1608Metric_Pad1.08x0.95mm_HandSolder
- C611: renamed from C711; footprint (none) -> Capacitor_SMD:C_0603_1608Metric_Pad1.08x0.95mm_HandSolder
- C612: renamed from C712; footprint (none) -> Capacitor_SMD:C_0603_1608Metric_Pad1.08x0.95mm_HandSolder
- C613: renamed from C713; footprint (none) -> Capacitor_SMD:C_0603_1608Metric_Pad1.08x0.95mm_HandSolder
- C614: renamed from C607; footprint (none) -> Capacitor_SMD:C_0603_1608Metric_Pad1.08x0.95mm_HandSolder
- C615: renamed from C608; footprint (none) -> Capacitor_SMD:C_0603_1608Metric_Pad1.08x0.95mm_HandSolder
- C616: renamed from C609; footprint (none) -> Capacitor_SMD:C_0603_1608Metric_Pad1.08x0.95mm_HandSolder
- C617: renamed from C610; footprint (none) -> Capacitor_SMD:C_0603_1608Metric_Pad1.08x0.95mm_HandSolder
- C618: renamed from C611; footprint (none) -> Capacitor_SMD:C_0603_1608Metric_Pad1.08x0.95mm_HandSolder
- C619: renamed from C612; footprint (none) -> Capacitor_SMD:C_0603_1608Metric_Pad1.08x0.95mm_HandSolder
- C620: renamed from C613; footprint (none) -> Capacitor_SMD:C_0603_1608Metric_Pad1.08x0.95mm_HandSolder
- C621: renamed from C614; footprint (none) -> Capacitor_SMD:C_0603_1608Metric_Pad1.08x0.95mm_HandSolder
- C622: renamed from C615; footprint (none) -> Capacitor_SMD:C_0603_1608Metric_Pad1.08x0.95mm_HandSolder
- C623: renamed from C616; footprint (none) -> Capacitor_SMD:C_0603_1608Metric_Pad1.08x0.95mm_HandSolder
- D611: renamed from D711; value D -> 1N4148W; footprint (none) -> Diode_SMD:D_SOD-123
- K601: renamed from K701; footprint (none) -> ETH1CLCR2:SA
- Q601: renamed from Q701; footprint (none) -> Package_TO_SOT_SMD:SOT-23
- Q602: renamed from Q702; footprint (none) -> Package_TO_SOT_SMD:SOT-23
- Q605: renamed from Q705; footprint (none) -> Package_TO_SOT_SMD:SOT-23
- Q606: renamed from Q706; footprint (none) -> Package_TO_SOT_SMD:SOT-23
- Q609: renamed from Q709; footprint (none) -> Package_TO_SOT_SMD:SOT-23
- Q610: renamed from Q710; footprint (none) -> Package_TO_SOT_SMD:SOT-23
- Q613: renamed from Q713; footprint (none) -> Package_TO_SOT_SMD:SOT-23
- Q614: renamed from Q714; footprint (none) -> Package_TO_SOT_SMD:SOT-23
- R601: renamed from R701; footprint (none) -> Resistor_SMD:R_0603_1608Metric_Pad0.98x0.95mm_HandSolder
- R602: renamed from R702; footprint (none) -> Resistor_SMD:R_0603_1608Metric_Pad0.98x0.95mm_HandSolder
- R603: renamed from R703; footprint (none) -> Resistor_SMD:R_0603_1608Metric_Pad0.98x0.95mm_HandSolder
- R604: renamed from R704; footprint (none) -> Resistor_SMD:R_0603_1608Metric_Pad0.98x0.95mm_HandSolder
- R605: renamed from R705; footprint (none) -> Resistor_SMD:R_0603_1608Metric_Pad0.98x0.95mm_HandSolder
- R606: renamed from R706; footprint (none) -> Resistor_SMD:R_0603_1608Metric_Pad0.98x0.95mm_HandSolder
- R607: renamed from R707; footprint (none) -> Resistor_SMD:R_0603_1608Metric_Pad0.98x0.95mm_HandSolder
- R608: renamed from R708; footprint (none) -> Resistor_SMD:R_0603_1608Metric_Pad0.98x0.95mm_HandSolder
- R609: renamed from R709; footprint (none) -> Resistor_SMD:R_0603_1608Metric_Pad0.98x0.95mm_HandSolder
- R610: renamed from R710; footprint (none) -> Resistor_SMD:R_0603_1608Metric_Pad0.98x0.95mm_HandSolder
- R611: renamed from R711; footprint (none) -> Resistor_SMD:R_0603_1608Metric_Pad0.98x0.95mm_HandSolder
- R612: renamed from R712; footprint (none) -> Resistor_SMD:R_0603_1608Metric_Pad0.98x0.95mm_HandSolder
- R613: renamed from R713; footprint (none) -> Resistor_SMD:R_0603_1608Metric_Pad0.98x0.95mm_HandSolder
- R614: renamed from R714; footprint (none) -> Resistor_SMD:R_0603_1608Metric_Pad0.98x0.95mm_HandSolder
- R615: renamed from R715; footprint (none) -> Resistor_SMD:R_0603_1608Metric_Pad0.98x0.95mm_HandSolder
- R616: renamed from R716; footprint (none) -> Resistor_SMD:R_0603_1608Metric_Pad0.98x0.95mm_HandSolder
- R617: renamed from R717; footprint (none) -> Resistor_SMD:R_0603_1608Metric_Pad0.98x0.95mm_HandSolder
- R618: renamed from R718; footprint (none) -> Resistor_SMD:R_0603_1608Metric_Pad0.98x0.95mm_HandSolder
- R619: renamed from R719; footprint (none) -> Resistor_SMD:R_0603_1608Metric_Pad0.98x0.95mm_HandSolder
- R620: renamed from R720; footprint (none) -> Resistor_SMD:R_0603_1608Metric_Pad0.98x0.95mm_HandSolder
- R621: renamed from R721; footprint (none) -> Resistor_SMD:R_0603_1608Metric_Pad0.98x0.95mm_HandSolder
- R622: renamed from R722; footprint (none) -> Resistor_SMD:R_0603_1608Metric_Pad0.98x0.95mm_HandSolder
- R623: renamed from R723; footprint (none) -> Resistor_SMD:R_0603_1608Metric_Pad0.98x0.95mm_HandSolder
- R624: renamed from R724; footprint (none) -> Resistor_SMD:R_0603_1608Metric_Pad0.98x0.95mm_HandSolder
- R625: renamed from R725; footprint (none) -> Resistor_SMD:R_0603_1608Metric_Pad0.98x0.95mm_HandSolder
- R626: renamed from R726; footprint (none) -> Resistor_SMD:R_0603_1608Metric_Pad0.98x0.95mm_HandSolder
- R627: renamed from R727; footprint (none) -> Resistor_SMD:R_0603_1608Metric_Pad0.98x0.95mm_HandSolder
- R628: renamed from R728; footprint (none) -> Resistor_SMD:R_0603_1608Metric_Pad0.98x0.95mm_HandSolder
- R629: renamed from R729; footprint (none) -> Resistor_SMD:R_0603_1608Metric_Pad0.98x0.95mm_HandSolder
- R630: renamed from R730; value 47 -> 47/.1%; footprint (none) -> Resistor_SMD:R_0603_1608Metric_Pad0.98x0.95mm_HandSolder
- R631: renamed from R731; value 0R1/.1% -> 0R1; footprint (none) -> Resistor_SMD:R_0805_2012Metric_Pad1.20x1.40mm_HandSolder
- R632: renamed from R732; footprint (none) -> Resistor_SMD:R_0603_1608Metric_Pad0.98x0.95mm_HandSolder
- R633: renamed from R733; footprint (none) -> Resistor_SMD:R_0603_1608Metric_Pad0.98x0.95mm_HandSolder
- R634: renamed from R734; footprint (none) -> Resistor_SMD:R_0603_1608Metric_Pad0.98x0.95mm_HandSolder
- U605: renamed from U701; footprint (none) -> Package_SO:SOIC-8_3.9x4.9mm_P1.27mm
- renumbered D701 to D601, D702 to D602, D703 to D603, D704 to D604, D705 to D605, D706 to D606, D707 to D607, D708 to D608, D709 to D609, D710 to D610, Q703 to Q603, Q704 to Q604, Q707 to Q607, Q708 to Q608, Q711 to Q611, Q712 to Q612, Q715 to Q615, Q716 to Q616, Q717 to Q617, U603 to U601, U604 to U602, U605 to U603, U606 to U604
Connections:
- net at Q601.2 (S), Q605.2 (S), Q609.2 (S)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: now also TP601.1

Commit message: PCB layout
Parts:
- U605: footprint Package_SO:SOIC-8_3.9x4.9mm_P1.27mm -> Package_SO:SOIC-8-1EP_3.9x4.9mm_P1.27mm_EP2.29x3mm
Changed lines of the file:
@@
 F 0 "U605" H 8950 8850 50  0000 L CNN
 F 1 "ADA4817-1ARDZ" H 8700 8750 50  0000 L CNN
-F 2 "Package_SO:SOIC-8_3.9x4.9mm_P1.27mm" H 8850 8700 50  0001 C CNN
+F 2 "Package_SO:SOIC-8-1EP_3.9x4.9mm_P1.27mm_EP2.29x3mm" H 8850 8700 50  0001 C CNN
 F 3 "" H 8850 8700 50  0001 C CNN
 	1    8600 8550
