File: hardware/ETH1CLCR2/IV_Converter.sch (KiCad schematic (older format))
At the start: 92 parts, among them K601 TQ2SA-5V, Q601 MMBFJ309LT1G, Q602 MMBFJ309LT1G, Q603 BC847, Q604 BC857, Q605 MMBFJ309LT1G, Q606 MMBFJ309LT1G, Q607 BC847, Q608 BC857, Q609 MMBFJ309LT1G, Q610 MMBFJ309LT1G, Q611 BC847, Q612 BC857, Q613 MMBFJ309LT1G, Q614 MMBFJ309LT1G, Q615 BC847, Q616 BC857, Q617 BC847, U601 SN74LVC1T45DBV, U602 SN74LVC1T45DBV, U603 SN74LVC1T45DBV, U604 SN74LVC1T45DBV, U605 ADA4817-1ARDZ

Commit message: PCB layout
Parts:
- removed D601, D602, D603, D604, D605, D606, D607, D608: BAS16J, Package_TO_SOT_SMD:SOT-323_SC-70, symbol Diode:BAS16W
- added D601, D602, D603, D604, D605, D606, D607, D608: BAS16J, Diode_SMD:D_SOD-323_HandSoldering, symbol Device:D
Changed lines of the file:
@@
 	8000 1700 7900 1700
-$Comp
-L Diode:BAS16W D601
-U 1 1 60B9EFF1
-P 8700 1350
-F 0 "D601" H 8700 1567 50  0000 C CNN
-F 1 "BAS16J" H 8700 1476 50  0000 C CNN
-F 2 "Package_TO_SOT_SMD:SOT-323_SC-70" H 8700 1175 50  0001 C CNN
-F 3 "https://assets.nexperia.com/documents/data-sheet/BAS16_SER.pdf" H 8700 1350 50  0001 C CNN
-	1    8700 1350
-	1    0    0    -1
-$EndComp
-$Comp
-L Diode:BAS16W D602
-U 1 1 60BA092B
-P 8700 1700
-F 0 "D602" H 8700 1917 50  0000 C CNN
-F 1 "BAS16J" H 8700 1826 50  0000 C CNN
-F 2 "Package_TO_SOT_SMD:SOT-323_SC-70" H 8700 1525 50  0001 C CNN
-F 3 "https://assets.nexperia.com/documents/data-sheet/BAS16_SER.pdf" H 8700 1700 50  0001 C CNN
-	1    8700 1700
-	1    0    0    -1
-$EndComp
 $Comp
 L Device:C C603
@@
 	8000 3450 7900 3450
 $Comp
-L Diode:BAS16W D603
-U 1 1 60D05AB6
-P 8700 3100
-F 0 "D603" H 8700 3317 50  0000 C CNN
-F 1 "BAS16J" H 8700 3226 50  0000 C CNN
-F 2 "Package_TO_SOT_SMD:SOT-323_SC-70" H 8700 2925 50  0001 C CNN
-F 3 "https://assets.nexperia.com/documents/data-sheet/BAS16_SER.pdf" H 8700 3100 50  0001 C CNN
-	1    8700 3100
-	1    0    0    -1
-$EndComp
-$Comp
-L Diode:BAS16W D604
-U 1 1 60D05ABC
-P 8700 3450
-F 0 "D604" H 8700 3667 50  0000 C CNN
-F 1 "BAS16J" H 8700 3576 50  0000 C CNN
-F 2 "Package_TO_SOT_SMD:SOT-323_SC-70" H 8700 3275 50  0001 C CNN
-F 3 "https://assets.nexperia.com/documents/data-sheet/BAS16_SER.pdf" H 8700 3450 50  0001 C CNN
-	1    8700 3450
-	1    0    0    -1
-$EndComp
-$Comp
 L Device:C C606
 U 1 1 60D05AC2
@@
 	8000 5150 7900 5150
 $Comp
-L Diode:BAS16W D605
-U 1 1 60D16AC3
-P 8700 4800
-F 0 "D605" H 8700 5017 50  0000 C CNN
-F 1 "BAS16J" H 8700 4926 50  0000 C CNN
-F 2 "Package_TO_SOT_SMD:SOT-323_SC-70" H 8700 4625 50  0001 C CNN
-F 3 "https://assets.nexperia.com/documents/data-sheet/BAS16_SER.pdf" H 8700 4800 50  0001 C CNN
-	1    8700 4800
-	1    0    0    -1
-$EndComp
-$Comp
-L Diode:BAS16W D606
-U 1 1 60D16AC9
-P 8700 5150
-F 0 "D606" H 8700 5367 50  0000 C CNN
-F 1 "BAS16J" H 8700 5276 50  0000 C CNN
-F 2 "Package_TO_SOT_SMD:SOT-323_SC-70" H 8700 4975 50  0001 C CNN
-F 3 "https://assets.nexperia.com/documents/data-sheet/BAS16_SER.pdf" H 8700 5150 50  0001 C CNN
-	1    8700 5150
-	1    0    0    -1
-$EndComp
-$Comp
 L Device:C C609
 U 1 1 60D16ACF
@@
 Wire Wire Line
 	8000 6900 7900 6900
-$Comp
-L Diode:BAS16W D607
-U 1 1 60D16B6E
-P 8700 6550
-F 0 "D607" H 8700 6767 50  0000 C CNN
-F 1 "BAS16J" H 8700 6676 50  0000 C CNN
-F 2 "Package_TO_SOT_SMD:SOT-323_SC-70" H 8700 6375 50  0001 C CNN
-F 3 "https://assets.nexperia.com/documents/data-sheet/BAS16_SER.pdf" H 8700 6550 50  0001 C CNN
-	1    8700 6550
-	1    0    0    -1
-$EndComp
-$Comp
-L Diode:BAS16W D608
-U 1 1 60D16B74
-P 8700 6900
-F 0 "D608" H 8700 7117 50  0000 C CNN
-F 1 "BAS16J" H 8700 7026 50  0000 C CNN
-F 2 "Package_TO_SOT_SMD:SOT-323_SC-70" H 8700 6725 50  0001 C CNN
-F 3 "https://assets.nexperia.com/documents/data-sheet/BAS16_SER.pdf" H 8700 6900 50  0001 C CNN
-	1    8700 6900
-	1    0    0    -1
-$EndComp
 $Comp
 L Device:C C612
@@
 $EndComp
 Connection ~ 9600 8650
+$Comp
+L Device:D D604
+U 1 1 60B92993
+P 8700 3450
+F 0 "D604" H 8700 3667 50  0000 C CNN
+F 1 "BAS16J" H 8700 3576 50  0000 C CNN
+F 2 "Diode_SMD:D_SOD-323_HandSoldering" H 8700 3450 50  0001 C CNN
+F 3 "~" H 8700 3450 50  0001 C CNN
+	1    8700 3450
+	1    0    0    -1
+$EndComp
+$Comp
+L Device:D D603
+U 1 1 60B94896
+P 8700 3100
+F 0 "D603" H 8700 3317 50  0000 C CNN
+F 1 "BAS16J" H 8700 3226 50  0000 C CNN
+F 2 "Diode_SMD:D_SOD-323_HandSoldering" H 8700 3100 50  0001 C CNN
+F 3 "~" H 8700 3100 50  0001 C CNN
+	1    8700 3100
+	1    0    0    -1
+$EndComp
+$Comp
+L Device:D D601
+U 1 1 60B9A027
+P 8700 1350
+F 0 "D601" H 8700 1567 50  0000 C CNN
+F 1 "BAS16J" H 8700 1476 50  0000 C CNN
+F 2 "Diode_SMD:D_SOD-323_HandSoldering" H 8700 1350 50  0001 C CNN
+F 3 "~" H 8700 1350 50  0001 C CNN
+	1    8700 1350
+	1    0    0    -1
+$EndComp
+$Comp
+L Device:D D602
+U 1 1 60B9AC3C
+P 8700 1700
+F 0 "D602" H 8700 1917 50  0000 C CNN
+F 1 "BAS16J" H 8700 1826 50  0000 C CNN
+F 2 "Diode_SMD:D_SOD-323_HandSoldering" H 8700 1700 50  0001 C CNN
+F 3 "~" H 8700 1700 50  0001 C CNN
+	1    8700 1700
+	1    0    0    -1
+$EndComp
+$Comp
+L Device:D D605
+U 1 1 60B9E5DA
+P 8700 4800
+F 0 "D605" H 8700 5017 50  0000 C CNN
+F 1 "BAS16J" H 8700 4926 50  0000 C CNN
+F 2 "Diode_SMD:D_SOD-323_HandSoldering" H 8700 4800 50  0001 C CNN
+F 3 "~" H 8700 4800 50  0001 C CNN
+	1    8700 4800
+	1    0    0    -1
+$EndComp
+$Comp
+L Device:D D606
+U 1 1 60B9FDCF
+P 8700 5150
+F 0 "D606" H 8700 5367 50  0000 C CNN
+F 1 "BAS16J" H 8700 5276 50  0000 C CNN
+F 2 "Diode_SMD:D_SOD-323_HandSoldering" H 8700 5150 50  0001 C CNN
+F 3 "~" H 8700 5150 50  0001 C CNN
+	1    8700 5150
+	1    0    0    -1
+$EndComp
+$Comp
+L Device:D D607
+U 1 1 60BA073B
+P 8700 6550
+F 0 "D607" H 8700 6767 50  0000 C CNN
+F 1 "BAS16J" H 8700 6676 50  0000 C CNN
+F 2 "Diode_SMD:D_SOD-323_HandSoldering" H 8700 6550 50  0001 C CNN
+F 3 "~" H 8700 6550 50  0001 C CNN
+	1    8700 6550
+	1    0    0    -1
+$EndComp
+$Comp
+L Device:D D608
+U 1 1 60BA220E
+P 8700 6900
+F 0 "D608" H 8700 7117 50  0000 C CNN
+F 1 "BAS16J" H 8700 7026 50  0000 C CNN
+F 2 "Diode_SMD:D_SOD-323_HandSoldering" H 8700 6900 50  0001 C CNN
+F 3 "~" H 8700 6900 50  0001 C CNN
+	1    8700 6900
+	1    0    0    -1
+$EndComp
 $EndSCHEMATC

Commit message: PCB
Parts:
- TP601: footprint TestPoint:TestPoint_Plated_Hole_D2.0mm -> TestPoint:TestPoint_Pad_1.0x1.0mm
Changed lines of the file:
@@
 F 0 "TP601" V 9554 8838 50  0000 L CNN
 F 1 "TestPoint" V 9645 8838 50  0000 L CNN
-F 2 "TestPoint:TestPoint_Plated_Hole_D2.0mm" H 9800 8650 50  0001 C CNN
+F 2 "TestPoint:TestPoint_Pad_1.0x1.0mm" H 9800 8650 50  0001 C CNN
 F 3 "~" H 9800 8650 50  0001 C CNN
 	1    9600 8650

Commit message: PCB
Parts:
- added C613: DNP, Capacitor_SMD:C_0603_1608Metric_Pad1.08x0.95mm_HandSolder, symbol Device:C
- added C625, C626: 1u, Capacitor_SMD:C_0603_1608Metric_Pad1.08x0.95mm_HandSolder, symbol Device:C
- added R632: 2/.5%, Resistor_SMD:R_0603_1608Metric_Pad0.98x0.95mm_HandSolder, symbol Device:R
- R631: value 0R1 -> 2/.5%; footprint Resistor_SMD:R_0805_2012Metric_Pad1.20x1.40mm_HandSolder -> Resistor_SMD:R_0603_1608Metric_Pad0.98x0.95mm_HandSolder
- renumbered C613 to C614, C614 to C615, C615 to C616, C616 to C617, C617 to C618, C618 to C619, C619 to C620, C620 to C621, C621 to C622, C622 to C623, C623 to C624, R632 to R633, R633 to R634, R634 to R635
Connections:
- net +5VA: now also C625.1
- net -5VA: now also C626.1
- net GND: now also C625.2, C626.2, R632.2
- net at C602.2, C605.2, C608.2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: now also C613.2; no longer U605.1
- net at K601.4, K601.7, R631.1: now also R632.1
- new net: C613.1, U605.1
Other:
- moved on the sheet: C614, R630, U605

Commit message: BOM
Parts:
- R605, R607, R612, R614, R619, R621, R626, R628: value 10K -> 10k
Changed lines of the file:
@@
 P 5700 1600
 F 0 "R605" H 5770 1646 50  0000 L CNN
-F 1 "10K" H 5770 1555 50  0000 L CNN
+F 1 "10k" H 5770 1555 50  0000 L CNN
 F 2 "Resistor_SMD:R_0603_1608Metric_Pad0.98x0.95mm_HandSolder" V 5630 1600 50  0001 C CNN
 F 3 "~" H 5700 1600 50  0001 C CNN
@@
 P 7300 2050
 F 0 "R607" V 7093 2050 50  0000 C CNN
-F 1 "10K" V 7184 2050 50  0000 C CNN
+F 1 "10k" V 7184 2050 50  0000 C CNN
 F 2 "Resistor_SMD:R_0603_1608Metric_Pad0.98x0.95mm_HandSolder" V 7230 2050 50  0001 C CNN
 F 3 "~" H 7300 2050 50  0001 C CNN
@@
 P 5700 3350
 F 0 "R612" H 5770 3396 50  0000 L CNN
-F 1 "10K" H 5770 3305 50  0000 L CNN
+F 1 "10k" H 5770 3305 50  0000 L CNN
 F 2 "Resistor_SMD:R_0603_1608Metric_Pad0.98x0.95mm_HandSolder" V 5630 3350 50  0001 C CNN
 F 3 "~" H 5700 3350 50  0001 C CNN
@@
 P 7300 3800
 F 0 "R614" V 7093 3800 50  0000 C CNN
-F 1 "10K" V 7184 3800 50  0000 C CNN
+F 1 "10k" V 7184 3800 50  0000 C CNN
 F 2 "Resistor_SMD:R_0603_1608Metric_Pad0.98x0.95mm_HandSolder" V 7230 3800 50  0001 C CNN
 F 3 "~" H 7300 3800 50  0001 C CNN
@@
 P 5700 5050
 F 0 "R619" H 5770 5096 50  0000 L CNN
-F 1 "10K" H 5770 5005 50  0000 L CNN
+F 1 "10k" H 5770 5005 50  0000 L CNN
 F 2 "Resistor_SMD:R_0603_1608Metric_Pad0.98x0.95mm_HandSolder" V 5630 5050 50  0001 C CNN
 F 3 "~" H 5700 5050 50  0001 C CNN
@@
 P 7300 5500
 F 0 "R621" V 7093 5500 50  0000 C CNN
-F 1 "10K" V 7184 5500 50  0000 C CNN
+F 1 "10k" V 7184 5500 50  0000 C CNN
 F 2 "Resistor_SMD:R_0603_1608Metric_Pad0.98x0.95mm_HandSolder" V 7230 5500 50  0001 C CNN
 F 3 "~" H 7300 5500 50  0001 C CNN
@@
 P 5700 6800
 F 0 "R626" H 5770 6846 50  0000 L CNN
-F 1 "10K" H 5770 6755 50  0000 L CNN
+F 1 "10k" H 5770 6755 50  0000 L CNN
 F 2 "Resistor_SMD:R_0603_1608Metric_Pad0.98x0.95mm_HandSolder" V 5630 6800 50  0001 C CNN
 F 3 "~" H 5700 6800 50  0001 C CNN
@@
 P 7300 7250
 F 0 "R628" V 7093 7250 50  0000 C CNN
-F 1 "10K" V 7184 7250 50  0000 C CNN
+F 1 "10k" V 7184 7250 50  0000 C CNN
 F 2 "Resistor_SMD:R_0603_1608Metric_Pad0.98x0.95mm_HandSolder" V 7230 7250 50  0001 C CNN
 F 3 "~" H 7300 7250 50  0001 C CNN
