File: hardware/ETH1CLCR2/ETH1CLCR2.sch (KiCad schematic (older format))
At the start: 0 parts

Commit message: Project based on https://hackaday.io/project/165409-precision-impedance-meter-asdflcr1
Changed lines of the file:
@@
 $Descr A4 11693 8268
 encoding utf-8
-Sheet 1 7
+Sheet 1 10
 Title ""
 Date ""
@@
 $EndDescr
 $Sheet
-S 4850 2100 1500 2500
+S 7700 1950 1200 1100
+U 60955EFA
+F0 "Ethernet" 50
+F1 "Ethernet.sch" 50
+F2 "TX+" B R 8900 2050 50
+F3 "TX-" B R 8900 2150 50
+F4 "RX+" B R 8900 2350 50
+F5 "RX-" B R 8900 2450 50
+F6 "RMII_TXD1" B L 7700 2050 50
+F7 "RMII_TXD0" B L 7700 2150 50
+F8 "RMII_TXEN" B L 7700 2250 50
+F9 "RMII_RXD0" B L 7700 2350 50
+F10 "RMII_RXD1" B L 7700 2450 50
+F11 "RMII_CRS_DV" B L 7700 2550 50
+F12 "RMII_MDIO" B L 7700 2650 50
+F13 "RMII_MDC" B L 7700 2750 50
+F14 "NRST" B L 7700 2850 50
+F15 "REF_CLK" B L 7700 2950 50
+$EndSheet
+$Sheet
+S 7700 1250 1200 450
+U 60963D02
+F0 "Trigger" 50
+F1 "Trigger.sch" 50
+F2 "EXT_TRIG" B R 8900 1450 50
+F3 "TRIG_EN" I L 7700 1350 50
+F4 "TRIG_OUT" I L 7700 1450 50
+F5 "TRIG_IN" O L 7700 1550 50
+$EndSheet
+$Sheet
+S 9050 650  750  3100
+U 60A4F32B
+F0 "Connector" 50
+F1 "Connector.sch" 50
+F2 "TX-" B L 9050 2150 50
+F3 "RX-" B L 9050 2450 50
+F4 "TX+" B L 9050 2050 50
+F5 "RX+" B L 9050 2350 50
+F6 "EXT_TRIG" B L 9050 1450 50
+F7 "CXN_REL5" I L 9050 3650 50
+F8 "CXN_REL4" I L 9050 3550 50
+F9 "CXN_REL3" I L 9050 3450 50
+F10 "CXN_REL2" I L 9050 3350 50
+F11 "CXN_REL1" I L 9050 3250 50
+$EndSheet
+Wire Wire Line
+	7700 2950 7550 2950
+Wire Wire Line
+	7550 2850 7700 2850
+Wire Wire Line
+	7700 2750 7550 2750
+Wire Wire Line
+	7550 2650 7700 2650
+Wire Wire Line
+	7550 2550 7700 2550
+Wire Wire Line
+	7550 2450 7700 2450
+Wire Wire Line
+	7700 2350 7550 2350
+Wire Wire Line
+	7550 2250 7700 2250
+Wire Wire Line
+	7700 2150 7550 2150
+Wire Wire Line
+	7550 2050 7700 2050
+Wire Wire Line
+	8900 2050 9050 2050
+Wire Wire Line
+	9050 2150 8900 2150
+Wire Wire Line
+	8900 2350 9050 2350
+Wire Wire Line
+	9050 2450 8900 2450
+Wire Wire Line
+	8900 1450 9050 1450
+Wire Wire Line
+	7700 1350 7550 1350
+Wire Wire Line
+	7550 1450 7700 1450
+Wire Wire Line
+	7700 1550 7550 1550
+$Sheet
+S 4000 1250 1700 950
+U 60A7CBEB
+F0 "ADC" 50
+F1 "ADC.sch" 50
+F2 "ADC_RVS1" O R 5700 1350 50
+F3 "ADC_RVS2" O R 5700 1450 50
+F4 "ADC_~CS" I R 5700 1650 50
+F5 "ADC_SCLK" I R 5700 1750 50
+F6 "ADC_MOSI" I R 5700 1850 50
+F7 "ADC_MISO" O R 5700 1950 50
+$EndSheet
+$Sheet
+S 1900 1250 1300 950
+U 60B5CBD2
+F0 "I/V Converter" 50
+F1 "IV_Converter.sch" 50
+F2 "L_CUR" I L 1900 1350 50
+F3 "CUR_OUT" O R 3200 1350 50
+F4 "IRR0" I R 3200 1700 50
+F5 "IRR1" I R 3200 1800 50
+F6 "IRR2" I R 3200 1900 50
+F7 "IRR3" I R 3200 2000 50
+F8 "IRR4" I R 3200 2100 50
+F9 "CUR_ZERO" O R 3200 1450 50
+$EndSheet
+$Sheet
+S 1050 6900 1250 650
+U 610A8D82
+F0 "Reference" 50
+F1 "Reference.sch" 50
+$EndSheet
+$Sheet
+S 4000 2450 1700 2300
+U 610F1C70
+F0 "FGEN" 50
+F1 "FGEN.sch" 50
+F2 "DDS_FGEN_~FSYNC" I R 5700 2550 50
+F3 "DDS_FGEN_SDATA" I R 5700 2650 50
+F4 "DDS_FGEN_SCLK" I R 5700 2750 50
+F5 "DDS_FGEN_PSEL0" I R 5700 2850 50
+F6 "DDS_FGEN_PSEL1" I R 5700 2950 50
+F7 "DDS_FGEN_FSELECT" I R 5700 3050 50
+F8 "DDS_MDAC_~SYNC" I R 5700 3250 50
+F9 "DDS_MDAC_SCLK" I R 5700 3350 50
+F10 "DDS_MDAC_DIN" I R 5700 3450 50
+F11 "DDS_DAC_SCLK" I R 5700 3650 50
+F12 "DDS_DAC_SDIN" I R 5700 3750 50
+F13 "DDS_DAC_~SYNC" I R 5700 3850 50
+F14 "DDS_DAC_~LDAC" I R 5700 4250 50
+F15 "DDS_DAC_~RESET" I R 5700 4050 50
+F16 "DDS_DAC_RSTSEL" I R 5700 4150 50
+F17 "DDS_DAC_SDO" O R 5700 3950 50
+F18 "H_CUR" O L 4000 2550 50
+$EndSheet
+Wire Wire Line
+	6050 1650 5700 1650
+Wire Wire Line
+	5700 1750 6050 1750
+Wire Wire Line
+	6050 1850 5700 1850
+Wire Wire Line
+	5700 1950 6050 1950
+$Sheet
+S 6050 1250 1500 5100
 U 608E48A2
 F0 "MCU" 50
 F1 "MCU.sch" 50
-F2 "RMII_TXD1" B R 6350 2900 50
-F3 "RMII_TXD0" B R 6350 3000 50
-F4 "RMII_TXEN" B R 6350 3100 50
-F5 "RMII_RXD0" B R 6350 3200 50
-F6 "RMII_RXD1" B R 6350 3300 50
-F7 "RMII_CRS_DV" B R 6350 3400 50
-F8 "RMII_MDIO" B R 6350 3500 50
-F9 "RMII_MDC" B R 6350 3600 50
-F10 "REF_CLK" B R 6350 3800 50
-F11 "NRST" B R 6350 3700 50
-F12 "TRIG_EN" O R 6350 2200 50
-F13 "TRIG_OUT" O R 6350 2300 50
-F14 "TRIG_IN" I R 6350 2400 50
-$EndSheet
-$Sheet
-S 6500 2800 1200 1100
-U 60955EFA
-F0 "Ethernet" 50
-F1 "Ethernet.sch" 50
-F2 "TX+" B R 7700 2900 50
-F3 "TX-" B R 7700 3000 50
-F4 "RX+" B R 7700 3200 50
-F5 "RX-" B R 7700 3300 50
-F6 "RMII_TXD1" B L 6500 2900 50
-F7 "RMII_TXD0" B L 6500 3000 50
-F8 "RMII_TXEN" B L 6500 3100 50
-F9 "RMII_RXD0" B L 6500 3200 50
-F10 "RMII_RXD1" B L 6500 3300 50
-F11 "RMII_CRS_DV" B L 6500 3400 50
-F12 "RMII_MDIO" B L 6500 3500 50
-F13 "RMII_MDC" B L 6500 3600 50
-F14 "NRST" B L 6500 3700 50
-F15 "REF_CLK" B L 6500 3800 50
-$EndSheet
-$Sheet
-S 6500 2100 1200 450
-U 60963D02
-F0 "Trigger" 50
-F1 "Trigger.sch" 50
-F2 "EXT_TRIG" B R 7700 2300 50
-F3 "TRIG_EN" I L 6500 2200 50
-F4 "TRIG_OUT" I L 6500 2300 50
-F5 "TRIG_IN" O L 6500 2400 50
-$EndSheet
-$Sheet
-S 7850 1500 750  3100
-U 60A4F32B
-F0 "Connector" 50
-F1 "Connector.sch" 50
-F2 "TX-" B L 7850 3000 50
-F3 "RX-" B L 7850 3300 50
-F4 "TX+" B L 7850 2900 50
-F5 "RX+" B L 7850 3200 50
-F6 "EXT_TRIG" B L 7850 2300 50
-F7 "CXN_REL5" I L 7850 4500 50
-F8 "CXN_REL4" I L 7850 4400 50
-F9 "CXN_REL3" I L 7850 4300 50
-F10 "CXN_REL2" I L 7850 4200 50
-F11 "CXN_REL1" I L 7850 4100 50
-$EndSheet
-Wire Wire Line
-	6500 3800 6350 3800
-Wire Wire Line
-	6350 3700 6500 3700
-Wire Wire Line
-	6500 3600 6350 3600
-Wire Wire Line
-	6350 3500 6500 3500
-Wire Wire Line
-	6350 3400 6500 3400
-Wire Wire Line
-	6350 3300 6500 3300
-Wire Wire Line
-	6500 3200 6350 3200
-Wire Wire Line
-	6350 3100 6500 3100
-Wire Wire Line
-	6500 3000 6350 3000
-Wire Wire Line
-	6350 2900 6500 2900
-Wire Wire Line
-	7700 2900 7850 2900
-Wire Wire Line
-	7850 3000 7700 3000
-Wire Wire Line
-	7700 3200 7850 3200
-Wire Wire Line
-	7850 3300 7700 3300
-Wire Wire Line
-	7700 2300 7850 2300
-Wire Wire Line
-	6500 2200 6350 2200
-Wire Wire Line
-	6350 2300 6500 2300
-Wire Wire Line
-	6500 2400 6350 2400
-$Sheet
-S 2800 3050 1250 900
-U 60A7CBEB
-F0 "ADC" 50
-F1 "ADC.sch" 50
-$EndSheet
-$Sheet
-S 2400 4750 1700 950
-U 60B5CBD2
-F0 "I/V Converter" 50
-F1 "IV_Converter.sch" 50
+F2 "RMII_TXD1" B R 7550 2050 50
+F3 "RMII_TXD0" B R 7550 2150 50
+F4 "RMII_TXEN" B R 7550 2250 50
+F5 "RMII_RXD0" B R 7550 2350 50
+F6 "RMII_RXD1" B R 7550 2450 50
+F7 "RMII_CRS_DV" B R 7550 2550 50
+F8 "RMII_MDIO" B R 7550 2650 50
+F9 "RMII_MDC" B R 7550 2750 50
+F10 "REF_CLK" B R 7550 2950 50
+F11 "NRST" B R 7550 2850 50
+F12 "TRIG_EN" O R 7550 1350 50
+F13 "TRIG_OUT" O R 7550 1450 50
+F14 "TRIG_IN" I R 7550 1550 50
+F15 "SPI4_SCK" O R 7550 3350 50
+F16 "SPI4_NSS" O R 7550 3450 50
+F17 "SPI4_MISO" I R 7550 3550 50
+F18 "SPI4_MOSI" O R 7550 3250 50
+F19 "SPI5_NSS" O R 7550 4150 50
+F20 "SPI5_SCK" O R 7550 4050 50
+F21 "SPI5_MISO" I R 7550 3950 50
+F22 "SPI5_MOSI" O R 7550 3850 50
+F23 "SPI2_MOSI" O L 6050 2650 50
+F24 "SPI2_NSS" O L 6050 2550 50
+F25 "SPI2_SCK" O L 6050 2750 50
+F26 "SPI1_NSS" O L 6050 3250 50
+F27 "SPI1_SCK" O L 6050 3350 50
+F28 "SPI1_MOSI" O L 6050 3450 50
+F29 "SPI3_MOSI" O L 6050 1850 50
+F30 "SPI3_MISO" I L 6050 1950 50
+F31 "SPI3_SCK" O L 6050 1750 50
+F32 "SPI3_NSS" O L 6050 1650 50
+$EndSheet
+Wire Wire Line
+	6050 3250 5700 3250
+Wire Wire Line
+	5700 3350 6050 3350
+Wire Wire Line
+	5700 3450 6050 3450
+$Sheet
+S 1900 3000 1500 1100
+U 621B52CA
+F0 "Voltage Diff Amp" 50
+F1 "V_Diff_Amp.sch" 50
 $EndSheet
 $EndSCHEMATC

Commit message: Footprints assigned.
Parts:
- added J101: RF_Shield_One_Piece, symbol Device:RF_Shield_One_Piece
Connections:
- new net GND: J101.1 (Shield)

Commit message: PCB layout
Parts:
- J101: footprint (none) -> ETH1CLCR2:36107406S
Changed lines of the file:
@@
 F 0 "J101" H 2330 6589 50  0000 L CNN
 F 1 "RF_Shield_One_Piece" H 2330 6498 50  0000 L CNN
-F 2 "" H 1700 6500 50  0001 C CNN
+F 2 "ETH1CLCR2:36107406S" H 1700 6500 50  0001 C CNN
 F 3 "~" H 1700 6500 50  0001 C CNN
 	1    1700 6600

Commit message: Schematic
Changed lines of the file:
@@
 	3800 5150 6900 5150
-Wire Wire Line
-	6900 3000 6700 3000
-Wire Wire Line
-	6700 3100 6900 3100
 Wire Wire Line
 	4600 4450 6900 4450
@@
 F38 "IDIFF1" O L 6900 4650 50
 F39 "IDIFF0" O L 6900 4550 50
-F40 "DDS_FGEN_PSEL0" O L 6900 3300 50
-F41 "DDS_FGEN_PSEL1" O L 6900 3400 50
-F42 "DDS_FGEN_FSELECT" O L 6900 3500 50
-F43 "ADC_RVS1" I L 6900 1800 50
-F44 "ADC_RVS2" I L 6900 1900 50
-F45 "FGEN_SEL" O L 6900 4000 50
-$EndSheet
-$Sheet
-S 5000 2900 1700 1200
-U 610F1C70
-F0 "FGEN" 50
-F1 "FGEN.sch" 50
-F2 "DDS_FGEN_~FSYNC" I R 6700 3000 50
-F3 "DDS_FGEN_SDATA" I R 6700 3100 50
-F4 "DDS_FGEN_SCLK" I R 6700 3200 50
-F5 "DDS_FGEN_PSEL0" I R 6700 3300 50
-F6 "DDS_FGEN_PSEL1" I R 6700 3400 50
-F7 "DDS_FGEN_FSELECT" I R 6700 3500 50
-F8 "DDS_MDAC_~SYNC" I R 6700 3700 50
-F9 "DDS_MDAC_SCLK" I R 6700 3800 50
-F10 "DDS_MDAC_DIN" I R 6700 3900 50
-F11 "H_CUR" O L 5000 3100 50
-F12 "FGEN_SEL" I R 6700 4000 50
+F40 "ADC_RVS1" I L 6900 1800 50
+F41 "ADC_RVS2" I L 6900 1900 50
+F42 "FGEN_SEL" O L 6900 4000 50
 $EndSheet
 Wire Wire Line
@@
 	8400 4100 9900 4100
 Wire Wire Line
-	6900 3700 6700 3700
-Wire Wire Line
-	6700 3800 6900 3800
-Wire Wire Line
-	6900 3900 6700 3900
-Wire Wire Line
-	6900 3200 6700 3200
-Wire Wire Line
-	6900 3500 6700 3500
-Wire Wire Line
-	6700 3400 6900 3400
-Wire Wire Line
-	6900 3300 6700 3300
-Wire Wire Line
 	6900 1800 6700 1800
 Wire Wire Line
 	6700 1900 6900 1900
-Wire Wire Line
-	6900 4000 6700 4000
 $Comp
 L Device:RF_Shield_One_Piece J101
@@
 	1    0    0    -1
 $EndComp
+$Sheet
+S 5000 2900 1700 1200
+U 610F1C70
+F0 "FGEN" 50
+F1 "FGEN.sch" 50
+F2 "H_CUR" O L 5000 3100 50
+$EndSheet
+$Sheet
+S 4700 5550 1550 1000
+U 60EBBEA5
+F0 "Clock" 50
+F1 "Clock.sch" 50
+$EndSheet
 $EndSCHEMATC

Commit message: Schematic
Changed lines of the file:
@@
 $Descr A4 11693 8268
 encoding utf-8
-Sheet 1 12
+Sheet 1 13
 Title ""
 Date ""
@@
 S 5000 2900 1700 1200
 U 610F1C70
-F0 "FGEN" 50
-F1 "FGEN.sch" 50
+F0 "DDS" 50
+F1 "DDS.sch" 50
 F2 "H_CUR" O L 5000 3100 50
 $EndSheet

Commit message: Schematic
Parts:
- removed J101: RF_Shield_One_Piece, ETH1CLCR2:36107406S, symbol Device:RF_Shield_One_Piece
