File: hardware/ETH1CLCR2/MCU.sch (KiCad schematic (older format))
At the start: 42 parts, among them J201 Conn_02x01, J202 20021111-00010T4LF, U201 STM32H743ZI, U202 HDC1080, U203 24LC08B-E/MS, Y201 NX3225GD-8MHZ

Commit message: Schematic design
Connections:
- net ADC_RVS1: now reaches U201.114 (PD0,DFSDM1_CKIN6,DFSDM1_DATIN7,UART4_RX,CAN1_RX,FMC_D2,EVENTOUT)
- net ADC_RVS2: now reaches U201.115 (PD1,DFSDM1_DATIN6,DFSDM1_CKIN7,UART4_TX,CAN1_TX,FMC_D3,EVENTOUT)
- net CXN_REL5: now reaches U201.116 (PD2,TRACED2,TIM3_ETR,UART5_RX,SDMMC1_CMD,DCMI_D11,EVENTOUT)
- net CXN_REL4: now reaches U201.117 (PD3,DFSDM1_CKOUT,SPI2_SCK,I2S2_CK,DFSDM1_DATIN0,USART2_CTS,FMC_CLK,DCMI_D5,LCD_G7,EVENTOUT)
- net CXN_REL3: now reaches U201.118 (PD4,DFSDM1_CKIN0,USART2_RTS,FMC_NOE,EVENTOUT)
- net CXN_REL2: now reaches U201.119 (PD5,USART2_TX,FMC_NWE,EVENTOUT)
- net CXN_REL1: now reaches U201.122 (PD6,DFSDM1_CKIN4,SPI3_MOSI,I2S3_SD,SAI1_SD_A,USART2_RX,DFSDM1_DATIN1,SDMMC2_CK,FMC_NWAIT,DCMI_D10,LCD_B2,EVENTOUT)
- net IRR0: now reaches U201.133 (PB3,JTDO,TRACESWO,TIM2_CH2,SPI1_SCK,I2S1_CK,SPI3_SCK,I2S3_CK,SPI6_SCK,SDMMC2_D2,CAN3_RX,UART7_RX,EVENTOUT)
- net IRR1: now reaches U201.134 (PB4,NJTRST,TIM3_CH1,SPI1_MISO,SPI3_MISO,SPI2_NSS,I2S2_WS,SPI6_MISO,SDMMC2_D3,CAN3_TX,UART7_TX,EVENTOUT)
- net IRR2: now reaches U201.135 (PB5,UART5_RX,TIM3_CH2,I2C1_SMBA,SPI1_MOSI,I2S1_SD,SPI3_MOSI,I2S3_SD,SPI6_MOSI,CAN2_RX,OTG_HS_ULPI_D7,ETH_PPS_OUT,FMC_SDCKE1,DCMI_D10,LCD_G7,EVENTOUT)
- net IRR3: now reaches U201.136 (PB6,UART5_TX,TIM4_CH1,HDMI_CEC,I2C1_SCL,DFSDM1_DATIN5,USART1_TX,CAN2_TX,QUADSPI_BK1_NCS,I2C4_SCL,FMC_SDNE1,DCMI_D5,EVENTOUT)
- net IRR4: now reaches U201.137 (PB7,TIM4_CH2,I2C1_SDA,DFSDM1_CKIN5,USART1_RX,I2C4_SDA,FMC_NL,DCMI_VSYNC,EVENTOUT)
- net IDIFF0: now reaches U201.139 (PB8,I2C4_SCL,TIM4_CH3,TIM10_CH1,I2C1_SCL,DFSDM1_CKIN7,UART5_RX,CAN1_RX,SDMMC2_D4,ETH_MII_TXD3,SDMMC1_D4,DCMI_D6,LCD_B6,EVENTOUT)
- net IDIFF1: now reaches U201.140 (PB9,I2C4_SDA,TIM4_CH4,TIM11_CH1,I2C1_SDA,SPI2_NSS,I2S2_WS,DFSDM1_DATIN7,UART5_TX,CAN1_TX,SDMMC2_D5,I2C4_SMBA,SDMMC1_D5,DCMI_D7,LCD_B7,EVENTOUT)
- net VDIFF0: now reaches U201.46 (PB0,TIM1_CH2N,TIM3_CH3,TIM8_CH2N,DFSDM1_CKOUT,UART4_CTS,_LCD_R3,OTG_HS_ULPI_D1,ETH_MII_RXD2,LCD_G1,EVENTOUT,ADC1_IN8,ADC2_IN8)
- net VDIFF1: now reaches U201.47 (PB1,TIM1_CH3N,TIM3_CH4,TIM8_CH3N,DFSDM1_DATIN1,LCD_R6,OTG_HS_ULPI_D2,ETH_MII_RXD3,LCD_G0,EVENTOUT,ADC1_IN9,ADC2_IN9)
- net VDIFF2: now reaches U201.48 (PB2,SAI1_SD_A,SPI3_MOSI,I2S3_SD,QUADSPI_CLK,DFSDM1_CKIN1,EVENTOUT)
- net DDS_FGEN_FSELECT: now reaches U201.68 (PE15,TIM1_BKIN,FMC_D12,LCD_R7,EVENTOUT)
- net DDS_FGEN_PSEL0: now reaches U201.69 (PB10,TIM2_CH3,I2C2_SCL,SPI2_SCK,I2S2_CK,DFSDM1_DATIN7,USART3_TX,QUADSPI_BK1_NCS,OTG_HS_ULPI_D3,ETH_MII_RX_ER,LCD_G4,EVENTOUT)
- net DDS_FGEN_PSEL1: now reaches U201.70 (PB11,TIM2_CH4,I2C2_SDA,DFSDM1_CKIN7,USART3_RX,OTG_HS_ULPI_D4,ETH_MII_TX_EN,ETH_RMII_TX_EN,_DSI_TE,LCD_G5,EVENTOUT)
- no-connect marks 26 -> 53
Changed lines of the file:
@@
 $Descr A3 16535 11693
 encoding utf-8
-Sheet 9 10
+Sheet 11 12
 Title "MCU"
 Date "2020-03-07"
@@
 	15050 1900 15100 1900
 NoConn ~ 15050 2400
-NoConn ~ 15050 6700
-NoConn ~ 15050 7000
-NoConn ~ 15050 7100
 $Comp
 L Device:C C221
@@
 NoConn ~ 8850 10450
 NoConn ~ 8850 10550
-NoConn ~ 15050 6600
 Wire Wire Line
 	6150 10200 6150 10100
@@
 	1850 9400 2050 9400
 Connection ~ 1850 9400
-NoConn ~ 15050 7200
 NoConn ~ 15050 2200
 NoConn ~ 15050 2100
 NoConn ~ 15050 4900
-$Comp
-L ETH1CLCR2:STM32H743ZI U201
-U 1 1 60365EFD
-P 9350 4950
-F 0 "U201" H 14050 8850 50  0000 C CNN
-F 1 "STM32H743ZI" H 14550 8850 50  0000 C CNN
-F 2 "ETH1CLCR2:TQFP-144_20x20mm_P0.5mm" H 25250 6450 50  0001 C CNN
-F 3 "" H 25250 6450 50  0001 C CNN
-	1    9350 4950
-	1    0    0    -1
-$EndComp
 $Comp
 L power:+3.3V #PWR0218
@@
 Wire Wire Line
 	3600 4700 3650 4700
-NoConn ~ 15050 7300
-NoConn ~ 15050 6400
-NoConn ~ 15050 6500
-NoConn ~ 15050 3100
-NoConn ~ 15050 3200
-NoConn ~ 15050 3300
-NoConn ~ 15050 3400
-NoConn ~ 15050 3500
 NoConn ~ 3650 2500
-NoConn ~ 15050 6300
 NoConn ~ 3650 3200
 NoConn ~ 3650 5100
 NoConn ~ 3650 5200
+Text HLabel 15100 3100 2    50   Output ~ 0
+CXN_REL5
+Text HLabel 15100 3200 2    50   Output ~ 0
+CXN_REL4
+Text HLabel 15100 3300 2    50   Output ~ 0
+CXN_REL3
+Text HLabel 15100 3400 2    50   Output ~ 0
+CXN_REL2
+Text HLabel 15100 3500 2    50   Output ~ 0
+CXN_REL1
+Wire Wire Line
+	15100 3100 15050 3100
+Wire Wire Line
+	15050 3200 15100 3200
+Wire Wire Line
+	15100 3300 15050 3300
+Wire Wire Line
+	15050 3400 15100 3400
+Wire Wire Line
+	15100 3500 15050 3500
+Text HLabel 15100 6700 2    50   Output ~ 0
+IRR1
+Text HLabel 15100 6800 2    50   Output ~ 0
+IRR2
+Text HLabel 15100 6900 2    50   Output ~ 0
+IRR3
+Text HLabel 15100 7000 2    50   Output ~ 0
+IRR4
+Wire Wire Line
+	15100 6900 15050 6900
+Wire Wire Line
+	15100 6800 15050 6800
+Wire Wire Line
+	15050 6700 15100 6700
+Wire Wire Line
+	15100 7000 15050 7000
+Text HLabel 15100 6600 2    50   Output ~ 0
+IRR0
+Wire Wire Line
+	15050 6600 15100 6600
+Text HLabel 15100 6500 2    50   Output ~ 0
+VDIFF2
+Text HLabel 15100 6400 2    50   Output ~ 0
+VDIFF1
+Wire Wire Line
+	15050 6500 15100 6500
+Wire Wire Line
+	15050 6400 15100 6400
+Text HLabel 15100 6300 2    50   Output ~ 0
+VDIFF0
+Wire Wire Line
+	15050 6300 15100 6300
+$Comp
+L ETH1CLCR2:STM32H743ZI U201
+U 1 1 60365EFD
+P 9350 4950
+F 0 "U201" H 14050 8850 50  0000 C CNN
+F 1 "STM32H743ZI" H 14550 8850 50  0000 C CNN
+F 2 "ETH1CLCR2:TQFP-144_20x20mm_P0.5mm" H 25250 6450 50  0001 C CNN
+F 3 "" H 25250 6450 50  0001 C CNN
+	1    9350 4950
+	1    0    0    -1
+$EndComp
+Text HLabel 15100 7200 2    50   Output ~ 0
+IDIFF1
+Text HLabel 15100 7100 2    50   Output ~ 0
+IDIFF0
+Wire Wire Line
+	15050 7100 15100 7100
+Wire Wire Line
+	15100 7200 15050 7200
+Text HLabel 15100 7300 2    50   Output ~ 0
+DDS_FGEN_PSEL0
+Text HLabel 15100 7400 2    50   Output ~ 0
+DDS_FGEN_PSEL1
+Text HLabel 15100 6100 2    50   Output ~ 0
+DDS_FGEN_FSELECT
+Wire Wire Line
+	15100 7400 15050 7400
+Wire Wire Line
+	15050 7300 15100 7300
+Wire Wire Line
+	15100 6100 15050 6100
+NoConn ~ 15050 5300
+NoConn ~ 15050 5400
+NoConn ~ 15050 5500
+NoConn ~ 15050 5600
+NoConn ~ 15050 5700
+NoConn ~ 15050 5800
+NoConn ~ 15050 5900
+NoConn ~ 15050 6000
+NoConn ~ 15050 4700
+NoConn ~ 15050 4600
+NoConn ~ 15050 4400
+NoConn ~ 15050 4300
+NoConn ~ 15050 3900
+NoConn ~ 15050 3800
+NoConn ~ 15050 3700
+NoConn ~ 15050 2700
+NoConn ~ 15050 2000
+NoConn ~ 15050 1700
+NoConn ~ 15050 1600
+NoConn ~ 15050 1400
+NoConn ~ 15050 1300
+NoConn ~ 15050 1200
+NoConn ~ 3650 3000
+NoConn ~ 3650 2900
+NoConn ~ 3650 2800
+NoConn ~ 3650 2700
+NoConn ~ 3650 2600
+NoConn ~ 3650 2000
+NoConn ~ 3650 1900
+NoConn ~ 3650 1700
+NoConn ~ 3650 1800
+NoConn ~ 3650 1600
+NoConn ~ 3650 1500
+NoConn ~ 3650 4100
+NoConn ~ 3650 4200
+NoConn ~ 3650 4300
+NoConn ~ 3650 4400
+NoConn ~ 3650 4900
+NoConn ~ 3650 5500
+NoConn ~ 3650 5600
+NoConn ~ 3650 5700
+Text HLabel 15100 2900 2    50   Input ~ 0
+ADC_RVS1
+Text HLabel 15100 3000 2    50   Input ~ 0
+ADC_RVS2
+Wire Wire Line
+	15100 3000 15050 3000
+Wire Wire Line
+	15050 2900 15100 2900
 $EndSCHEMATC

Commit message: Footprints assigned.
Parts:
- renumbered C201 to C1101, C202 to C1102, C203 to C1103, C204 to C1104, C205 to C1105, C206 to C1106, C207 to C1107, C208 to C1108, C209 to C1109, C210 to C1110, C211 to C1111, C212 to C1112, C213 to C1113, C214 to C1114, C215 to C1115, C216 to C1116, C217 to C1117, C218 to C1118, C219 to C1119, C220 to C1120, C221 to C1121, C222 to C1122, D201 to D1101, D202 to D1102, D203 to D1103, FB201 to FB1101, J201 to J1101, J202 to J1102, R201 to R1101, R202 to R1102, R203 to R1103, R204 to R1104, R205 to R1105, R206 to R1106, R207 to R1107, R208 to R1108, R209 to R1109, R210 to R1110, U201 to U1101, U202 to U1102, U203 to U1103, Y201 to Y1101
Connections:
- net FGEN_SEL: now reaches U1101.77 (PD8,DFSDM1_CKIN3,USART3_TX,SPDIF_RX1,FMC_D13,EVENTOUT)
- net SPI1_MISO: no longer names the net of U1101.42 (PA6,TIM1_BKIN,TIM3_CH1,TIM8_BKIN,SPI1_MISO,SPI6_MISO,TIM13_CH1,MDIOS_MDC,DCMI_PIXCLK,LCD_G2,EVENTOUT,ADC1_IN6,ADC2_IN6)
- net SPI2_MISO: no longer names the net of U1101.75 (PB14,TIM1_CH2N,TIM8_CH2N,USART1_TX,SPI2_MISO,DFSDM1_DATIN2,USART3_RTS,UART4_RTS,TIM12_CH1,SDMMC2_D0,OTG_HS_DM,EVENTOUT)
- net SPI4_MISO: no longer names the net of U1101.4 (PE5,TRACED2,TIM9_CH1,SPI4_MISO,SAI1_SCK_A,DFSDM1_CKIN3,FMC_A21,DCMI_D6,LCD_G0,EVENTOUT)
- net SPI4_MOSI: no longer names the net of U1101.5 (PE6,TRACED3,TIM1_BKIN2,TIM9_CH2,SPI4_MOSI,SAI1_SD_A,SAI2_MCLK_B,FMC_A22,DCMI_D7,LCD_G1,EVENTOUT)
- net SPI4_NSS: no longer names the net of U1101.3 (PE4,TRACED1,SPI4_NSS,SAI1_FS_A,DFSDM1_DATIN3,FMC_A20,DCMI_D4,LCD_B0,EVENTOUT)
- net SPI4_SCK: no longer names the net of U1101.1 (PE2,TRACECLK,SPI4_SCK,SAI1_MCLK_A,QUADSPI_BK1_IO2,ETH_MII_TXD3,FMC_A23,EVENTOUT)
- net SPI5_MISO: no longer names the net of U1101.20 (PF8,SPI5_MISO,SAI1_SCK_B,UART7_RTS,TIM13_CH1,QUADSPI_BK1_IO0,EVENTOUT,ADC3_IN6)
- net SPI5_MOSI: no longer names the net of U1101.21 (PF9,SPI5_MOSI,SAI1_FS_B,UART7_CTS,TIM14_CH1,QUADSPI_BK1_IO1,EVENTOUT,ADC3_IN7)
- net SPI5_NSS: no longer names the net of U1101.18 (PF6,TIM10_CH1,SPI5_NSS,SAI1_SD_B,UART7_RX,QUADSPI_BK1_IO3,EVENTOUT,ADC3_IN4)
- net SPI5_SCK: no longer names the net of U1101.19 (PF7,TIM11_CH1,SPI5_SCK,SAI1_MCLK_B,UART7_TX,QUADSPI_BK1_IO2,EVENTOUT,ADC3_IN5)
- no-connect marks 53 -> 62

Commit message: Schematic
Connections:
- net SPI1_MISO: now reaches U1101.42 (PA6,TIM1_BKIN,TIM3_CH1,TIM8_BKIN,SPI1_MISO,SPI6_MISO,TIM13_CH1,MDIOS_MDC,DCMI_PIXCLK,LCD_G2,EVENTOUT,ADC1_IN6,ADC2_IN6)
- net DDS_DIV2: now reaches U1101.50 (PF12,FMC_A6,EVENTOUT)
- net DDS_DIV4: now reaches U1101.53 (PF13,I2C4_SMBA,DFSDM1_DATIN6,FMC_A7,EVENTOUT)
- net DDS_DIV8: now reaches U1101.54 (PF14,I2C4_SCL,DFSDM1_CKIN6,FMC_A8,EVENTOUT)
- net ~DDS_DIV10: now reaches U1101.55 (PF15,I2C4_SDA,FMC_A9,EVENTOUT)
- net ADC_RVS1 renamed ADC1_RVS1
- net ADC_RVS2 renamed ADC1_RVS2
- net DDS_FGEN_FSELECT: no longer names the net of U1101.68 (PE15,TIM1_BKIN,FMC_D12,LCD_R7,EVENTOUT)
- net DDS_FGEN_PSEL0: no longer names the net of U1101.69 (PB10,TIM2_CH3,I2C2_SCL,SPI2_SCK,I2S2_CK,DFSDM1_DATIN7,USART3_TX,QUADSPI_BK1_NCS,OTG_HS_ULPI_D3,ETH_MII_RX_ER,LCD_G4,EVENTOUT)
- net DDS_FGEN_PSEL1: no longer names the net of U1101.70 (PB11,TIM2_CH4,I2C2_SDA,DFSDM1_CKIN7,USART3_RX,OTG_HS_ULPI_D4,ETH_MII_TX_EN,ETH_RMII_TX_EN,_DSI_TE,LCD_G5,EVENTOUT)
- no-connect marks 62 -> 60
Changed lines of the file:
@@
 $Descr A3 16535 11693
 encoding utf-8
-Sheet 11 13
+Sheet 11 12
 Title "MCU"
 Date "2020-03-07"
@@
 Wire Wire Line
 	15100 7200 15050 7200
-Text HLabel 15100 7300 2    50   Output ~ 0
-DDS_FGEN_PSEL0
-Text HLabel 15100 7400 2    50   Output ~ 0
-DDS_FGEN_PSEL1
-Text HLabel 15100 6100 2    50   Output ~ 0
-DDS_FGEN_FSELECT
-Wire Wire Line
-	15100 7400 15050 7400
-Wire Wire Line
-	15050 7300 15100 7300
-Wire Wire Line
-	15100 6100 15050 6100
 NoConn ~ 15050 5300
 NoConn ~ 15050 5400
@@
 NoConn ~ 15050 1300
 NoConn ~ 15050 1200
-NoConn ~ 3650 3000
-NoConn ~ 3650 2900
-NoConn ~ 3650 2800
-NoConn ~ 3650 2700
 NoConn ~ 3650 2600
 NoConn ~ 3650 2000
@@
 NoConn ~ 3650 5700
 Text HLabel 15100 2900 2    50   Input ~ 0
-ADC_RVS1
+ADC1_RVS1
 Text HLabel 15100 3000 2    50   Input ~ 0
-ADC_RVS2
+ADC1_RVS2
 Wire Wire Line
 	15100 3000 15050 3000
@@
 NoConn ~ 15050 5100
 NoConn ~ 15050 5200
-NoConn ~ 3650 3800
 NoConn ~ 15050 7700
 Text HLabel 15100 3700 2    50   Output ~ 0
@@
 Wire Wire Line
 	15100 3700 15050 3700
+Text HLabel 3600 3800 0    50   Input ~ 0
+SPI1_MISO
+Wire Wire Line
+	3650 3800 3600 3800
+NoConn ~ 15050 7400
+NoConn ~ 15050 7300
+NoConn ~ 15050 6100
+Text HLabel 3600 2700 0    50   Output ~ 0
+DDS_DIV2
+Text HLabel 3600 2800 0    50   Output ~ 0
+DDS_DIV4
+Text HLabel 3600 2900 0    50   Output ~ 0
+DDS_DIV8
+Text HLabel 3600 3000 0    50   Output ~ 0
+~DDS_DIV10
+Wire Wire Line
+	3650 2700 3600 2700
+Wire Wire Line
+	3600 2800 3650 2800
+Wire Wire Line
+	3650 2900 3600 2900
+Wire Wire Line
+	3600 3000 3650 3000
 $EndSCHEMATC
