File: hardware/ETH1CLCR2/MCU.sch (KiCad schematic (older format))
At the start: 42 parts, among them J1101 Conn_02x01, J1102 20021111-00010T4LF, U1101 STM32H743ZI, U1102 HDC1080, U1103 24LC08B-E/MS, Y1101 NX3225GD-8MHZ

Commit message: PCB
Connections:
- net IRR0: now also U1101.93 (PG8,SPI6_NSS,SPDIF_RX2,USART6_RTS,ETH_PPS_OUT,FMC_SDCLK,LCD_G7,EVENTOUT); no longer U1101.133 (PB3,JTDO,TRACESWO,TIM2_CH2,SPI1_SCK,I2S1_CK,SPI3_SCK,I2S3_CK,SPI6_SCK,SDMMC2_D2,CAN3_RX,UART7_RX,EVENTOUT)
- net IRR1: now also U1101.103 (PA11,TIM1_CH4,SPI2_NSS,I2S2_WS,UART4_RX,USART1_CTS,CAN1_RX,OTG_FS_DM,LCD_R4,EVENTOUT); no longer U1101.134 (PB4,NJTRST,TIM3_CH1,SPI1_MISO,SPI3_MISO,SPI2_NSS,I2S2_WS,SPI6_MISO,SDMMC2_D3,CAN3_TX,UART7_TX,EVENTOUT)
- net IRR2: now also U1101.102 (PA10,TIM1_CH3,USART1_RX,LCD_B4,OTG_FS_ID,MDIOS_MDIO,DCMI_D1,LCD_B1,EVENTOUT); no longer U1101.135 (PB5,UART5_RX,TIM3_CH2,I2C1_SMBA,SPI1_MOSI,I2S1_SD,SPI3_MOSI,I2S3_SD,SPI6_MOSI,CAN2_RX,OTG_HS_ULPI_D7,ETH_PPS_OUT,FMC_SDCKE1,DCMI_D10,LCD_G7,EVENTOUT)
- net IRR3: now also U1101.104 (PA12,TIM1_ETR,SPI2_SCK,I2S2_CK,UART4_TX,USART1_RTS,SAI2_FS_B,CAN1_TX,OTG_FS_DP,LCD_R5,EVENTOUT); no longer U1101.136 (PB6,UART5_TX,TIM4_CH1,HDMI_CEC,I2C1_SCL,DFSDM1_DATIN5,USART1_TX,CAN2_TX,QUADSPI_BK1_NCS,I2C4_SCL,FMC_SDNE1,DCMI_D5,EVENTOUT)
- net IRR4: now also U1101.101 (PA9,TIM1_CH2,I2C3_SMBA,SPI2_SCK,I2S2_CK,USART1_TX,DCMI_D0,LCD_R5,EVENTOUT,OTG_FS_VBUS); no longer U1101.137 (PB7,TIM4_CH2,I2C1_SDA,DFSDM1_CKIN5,USART1_RX,I2C4_SDA,FMC_NL,DCMI_VSYNC,EVENTOUT)
- net MCU_DEFAULT: now also U1101.116 (PD2,TRACED2,TIM3_ETR,UART5_RX,SDMMC1_CMD,DCMI_D11,EVENTOUT); no longer U1101.37 (PA3,TIM2_CH4,TIM5_CH4,TIM9_CH2,USART2_RX,LCD_B2,OTG_HS_ULPI_D0,ETH_MII_COL,LCD_B5,EVENTOUT,ADC1_IN3,ADC2_IN3,ADC3_IN3)
- net TRIG_EN: now also U1101.63 (PE10,TIM1_CH2N,DFSDM1_DATIN4,UART7_CTS,QUADSPI_BK2_IO3,FMC_D7,EVENTOUT); no longer U1101.92 (PG7,SAI1_MCLK_A,USART6_CK,FMC_INT,DCMI_D13,LCD_CLK,EVENTOUT)
- net TRIG_IN: now also U1101.65 (PE12,TIM1_CH3N,SPI4_SCK,DFSDM1_DATIN5,SAI2_SCK_B,FMC_D9,LCD_B4,EVENTOUT); no longer U1101.88 (PG3,FMC_A13,EVENTOUT)
- net TRIG_OUT: now also U1101.64 (PE11,TIM1_CH2,SPI4_NSS,DFSDM1_CKIN4,SAI2_SD_B,FMC_D8,LCD_G3,EVENTOUT); no longer U1101.91 (PG6,FMC_NE3,DCMI_D12,LCD_R7,EVENTOUT)
- net VDIFF0: now also U1101.96 (PC6,TIM3_CH1,TIM8_CH1,I2S2_MCK,DFSDM1_CKIN3,USART6_TX,FMC_NWAIT,SDMMC2_D6,SDMMC1_D6,DCMI_D0,LCD_HSYNC,EVENTOUT); no longer U1101.46 (PB0,TIM1_CH2N,TIM3_CH3,TIM8_CH2N,DFSDM1_CKOUT,UART4_CTS,_LCD_R3,OTG_HS_ULPI_D1,ETH_MII_RXD2,LCD_G1,EVENTOUT,ADC1_IN8,ADC2_IN8)
- net VDIFF1: now also U1101.98 (PC8,TRACED1,TIM3_CH3,TIM8_CH3,UART5_RTS,USART6_CK,FMC_NE2,FMC_NCE,SDMMC1_D0,DCMI_D2,EVENTOUT); no longer U1101.47 (PB1,TIM1_CH3N,TIM3_CH4,TIM8_CH3N,DFSDM1_DATIN1,LCD_R6,OTG_HS_ULPI_D2,ETH_MII_RXD3,LCD_G0,EVENTOUT,ADC1_IN9,ADC2_IN9)
- net VDIFF2: now also U1101.97 (PC7,TIM3_CH2,TIM8_CH2,I2S3_MCK,DFSDM1_DATIN3,USART6_RX,FMC_NE1,SDMMC2_D7,SDMMC1_D7,DCMI_D1,LCD_G6,EVENTOUT); no longer U1101.48 (PB2,SAI1_SD_A,SPI3_MOSI,I2S3_SD,QUADSPI_CLK,DFSDM1_CKIN1,EVENTOUT)
- net SPI4_SCK: now reaches U1101.1 (PE2,TRACECLK,SPI4_SCK,SAI1_MCLK_A,QUADSPI_BK1_IO2,ETH_MII_TXD3,FMC_A23,EVENTOUT)
- net SPI4_NSS: now reaches U1101.3 (PE4,TRACED1,SPI4_NSS,SAI1_FS_A,DFSDM1_DATIN3,FMC_A20,DCMI_D4,LCD_B0,EVENTOUT)
- net SPI4_MOSI: now reaches U1101.5 (PE6,TRACED3,TIM1_BKIN2,TIM9_CH2,SPI4_MOSI,SAI1_SD_A,SAI2_MCLK_B,FMC_A22,DCMI_D7,LCD_G1,EVENTOUT)
- net SPI2_MISO: now reaches U1101.75 (PB14,TIM1_CH2N,TIM8_CH2N,USART1_TX,SPI2_MISO,DFSDM1_DATIN2,USART3_RTS,UART4_RTS,TIM12_CH1,SDMMC2_D0,OTG_HS_DM,EVENTOUT)
- net ~ADC2_HPF: now reaches U1101.78 (PD9,DFSDM1_DATIN3,USART3_RX,FMC_D14,EVENTOUT)
- net ADC2_M0: now reaches U1101.79 (PD10,DFSDM1_CKOUT,USART3_CK,FMC_D15,LCD_B3,EVENTOUT)
- net ADC2_M1: now reaches U1101.85 (PD14,TIM4_CH3,UART8_CTS,FMC_D0,EVENTOUT)
- net FGEN_SEL renamed ADC2_MDIV
- net SPI2_MOSI renamed ~ADC2_RST
- no-connect marks 60 -> 52
Changed lines of the file:
@@
 Text HLabel 15750 8700 2    50   BiDi ~ 0
 NRST
-Text HLabel 15100 1900 2    50   Output ~ 0
+Text HLabel 15100 5600 2    50   Output ~ 0
 TRIG_EN
-Text HLabel 15100 1800 2    50   Output ~ 0
+Text HLabel 15100 5700 2    50   Output ~ 0
 TRIG_OUT
-Text HLabel 15100 1500 2    50   Input ~ 0
+Text HLabel 15100 5800 2    50   Input ~ 0
 TRIG_IN
 Wire Wire Line
-	15100 1500 15050 1500
-Wire Wire Line
-	15100 1800 15050 1800
-Wire Wire Line
-	15050 1900 15100 1900
+	15100 5600 15050 5600
+Wire Wire Line
+	15100 5700 15050 5700
+Wire Wire Line
+	15050 5800 15100 5800
 NoConn ~ 15050 2400
 $Comp
@@
 	3650 10900 4150 10900
 Wire Wire Line
-	3650 3500 3100 3500
-Text Label 3100 3500 0    50   ~ 0
+	15050 3100 15600 3100
+Text Label 15600 3100 2    50   ~ 0
 MCU_DEFAULT
 Connection ~ 11350 9950
@@
 	3600 900  2750 900
 Connection ~ 2750 900
-Text HLabel 15100 7800 2    50   Output ~ 0
-SPI2_MOSI
-Wire Wire Line
-	15100 7800 15050 7800
+Text HLabel 15100 7700 2    50   Input ~ 0
+SPI2_MISO
 Text HLabel 15100 7500 2    50   Output ~ 0
 SPI2_NSS
@@
 Wire Wire Line
 	15100 5900 15050 5900
-Text HLabel 15100 6700 2    50   Output ~ 0
+Text HLabel 3600 4300 0    50   Output ~ 0
 IRR1
-Text HLabel 15100 6800 2    50   Output ~ 0
+Text HLabel 3600 4200 0    50   Output ~ 0
 IRR2
-Text HLabel 15100 6900 2    50   Output ~ 0
+Text HLabel 3600 4400 0    50   Output ~ 0
 IRR3
-Text HLabel 15100 7000 2    50   Output ~ 0
+Text HLabel 3600 4100 0    50   Output ~ 0
 IRR4
-Wire Wire Line
-	15100 6900 15050 6900
-Wire Wire Line
-	15100 6800 15050 6800
-Wire Wire Line
-	15050 6700 15100 6700
-Wire Wire Line
-	15100 7000 15050 7000
-Text HLabel 15100 6600 2    50   Output ~ 0
+Text HLabel 15100 2000 2    50   Output ~ 0
 IRR0
 Wire Wire Line
-	15050 6600 15100 6600
-Text HLabel 15100 6500 2    50   Output ~ 0
+	15050 2000 15100 2000
+Text HLabel 3600 5600 0    50   Output ~ 0
 VDIFF2
-Text HLabel 15100 6400 2    50   Output ~ 0
+Text HLabel 3600 5700 0    50   Output ~ 0
 VDIFF1
 Wire Wire Line
-	15050 6500 15100 6500
-Wire Wire Line
-	15050 6400 15100 6400
-Text HLabel 15100 6300 2    50   Output ~ 0
+	3650 5600 3600 5600
+Wire Wire Line
+	3650 5700 3600 5700
+Text HLabel 3600 5500 0    50   Output ~ 0
 VDIFF0
 Wire Wire Line
-	15050 6300 15100 6300
-$Comp
-L ETH1CLCR2:STM32H743ZI U1101
-U 1 1 60365EFD
-P 9350 4950
-F 0 "U1101" H 14050 8850 50  0000 C CNN
-F 1 "STM32H743ZI" H 14550 8850 50  0000 C CNN
-F 2 "ETH1CLCR2:TQFP-144_20x20mm_P0.5mm" H 25250 6450 50  0001 C CNN
-F 3 "" H 25250 6450 50  0001 C CNN
-	1    9350 4950
-	1    0    0    -1
-$EndComp
+	3650 5500 3600 5500
 Text HLabel 15100 7200 2    50   Output ~ 0
 IDIFF1
@@
 NoConn ~ 15050 5400
 NoConn ~ 15050 5500
-NoConn ~ 15050 5600
-NoConn ~ 15050 5700
-NoConn ~ 15050 5800
 NoConn ~ 15050 4700
 NoConn ~ 15050 4600
 NoConn ~ 15050 4400
-NoConn ~ 15050 4300
-NoConn ~ 15050 3900
-NoConn ~ 15050 3800
 NoConn ~ 15050 2700
-NoConn ~ 15050 2000
 NoConn ~ 15050 1700
 NoConn ~ 15050 1600
@@
 NoConn ~ 3650 1600
 NoConn ~ 3650 1500
-NoConn ~ 3650 4100
-NoConn ~ 3650 4200
-NoConn ~ 3650 4300
-NoConn ~ 3650 4400
 NoConn ~ 3650 4900
-NoConn ~ 3650 5500
-NoConn ~ 3650 5600
-NoConn ~ 3650 5700
 Text HLabel 15100 2900 2    50   Input ~ 0
 ADC1_RVS1
@@
 NoConn ~ 3650 2300
 NoConn ~ 3650 2400
-NoConn ~ 15050 5000
-NoConn ~ 15050 4800
-NoConn ~ 15050 5100
-NoConn ~ 15050 5200
-NoConn ~ 15050 7700
-Text HLabel 15100 3700 2    50   Output ~ 0
-FGEN_SEL
-Wire Wire Line
-	15100 3700 15050 3700
 Text HLabel 3600 3800 0    50   Input ~ 0
 SPI1_MISO
@@
 Wire Wire Line
 	3600 3000 3650 3000
-NoConn ~ 15050 3100
 NoConn ~ 15050 3200
 NoConn ~ 15050 3300
 NoConn ~ 15050 3400
 NoConn ~ 15050 3500
+Wire Wire Line
+	15050 7700 15100 7700
+Text HLabel 15100 7800 2    50   Output ~ 0
+~ADC2_RST
+Wire Wire Line
+	15100 7800 15050 7800
+Text HLabel 15100 3900 2    50   Output ~ 0
+ADC2_M0
+Wire Wire Line
+	15100 3900 15050 3900
+Text HLabel 15100 4300 2    50   Output ~ 0
+ADC2_M1
+Wire Wire Line
+	15100 4300 15050 4300
+Text HLabel 15100 3700 2    50   Output ~ 0
+ADC2_MDIV
+Wire Wire Line
+	15100 3700 15050 3700
+Text HLabel 15100 3800 2    50   Output ~ 0
+~ADC2_HPF
+Wire Wire Line
+	15100 3800 15050 3800
+Text HLabel 15100 5000 2    50   Output ~ 0
+SPI4_NSS
+Text HLabel 15100 5200 2    50   Output ~ 0
+SPI4_MOSI
+Text HLabel 15100 4800 2    50   Output ~ 0
+SPI4_SCK
+Wire Wire Line
+	15050 4800 15100 4800
+Wire Wire Line
+	15100 5200 15050 5200
+Wire Wire Line
+	15100 5000 15050 5000
+NoConn ~ 15050 5100
+NoConn ~ 3650 3500
+$Comp
+L ETH1CLCR2:STM32H743ZI U1101
+U 1 1 60365EFD
+P 9350 4950
+F 0 "U1101" H 14050 8850 50  0000 C CNN
+F 1 "STM32H743ZI" H 14550 8850 50  0000 C CNN
+F 2 "ETH1CLCR2:TQFP-144_20x20mm_P0.5mm" H 25250 6450 50  0001 C CNN
+F 3 "" H 25250 6450 50  0001 C CNN
+	1    9350 4950
+	1    0    0    -1
+$EndComp
+Wire Wire Line
+	3650 4400 3600 4400
+Wire Wire Line
+	3650 4300 3600 4300
+Wire Wire Line
+	3600 4200 3650 4200
+Wire Wire Line
+	3650 4100 3600 4100
+NoConn ~ 15050 7000
+NoConn ~ 15050 6900
+NoConn ~ 15050 6800
+NoConn ~ 15050 6700
+NoConn ~ 15050 6400
+NoConn ~ 15050 6500
+NoConn ~ 15050 6300
+NoConn ~ 15050 6600
+NoConn ~ 15050 1900
+NoConn ~ 15050 1800
 $EndSCHEMATC

Commit message: PCB
Connections:
- net DDS_DIV2: now also U1101.141 (PE0,TIM4_ETR,LPTIM1_ETR,UART8_RX,SAI2_MCLK_A,FMC_NBL0,DCMI_D2,EVENTOUT); no longer U1101.50 (PF12,FMC_A6,EVENTOUT)
- net DDS_DIV4: now also U1101.140 (PB9,I2C4_SDA,TIM4_CH4,TIM11_CH1,I2C1_SDA,SPI2_NSS,I2S2_WS,DFSDM1_DATIN7,UART5_TX,CAN1_TX,SDMMC2_D5,I2C4_SMBA,SDMMC1_D5,DCMI_D7,LCD_B7,EVENTOUT); no longer U1101.53 (PF13,I2C4_SMBA,DFSDM1_DATIN6,FMC_A7,EVENTOUT)
- net DDS_DIV8: now also U1101.139 (PB8,I2C4_SCL,TIM4_CH3,TIM10_CH1,I2C1_SCL,DFSDM1_CKIN7,UART5_RX,CAN1_RX,SDMMC2_D4,ETH_MII_TXD3,SDMMC1_D4,DCMI_D6,LCD_B6,EVENTOUT); no longer U1101.54 (PF14,I2C4_SCL,DFSDM1_CKIN6,FMC_A8,EVENTOUT)
- net IDIFF0: now also U1101.2 (PE3,TRACED0,SAI1_SD_B,FMC_A19,EVENTOUT); no longer U1101.139 (PB8,I2C4_SCL,TIM4_CH3,TIM10_CH1,I2C1_SCL,DFSDM1_CKIN7,UART5_RX,CAN1_RX,SDMMC2_D4,ETH_MII_TXD3,SDMMC1_D4,DCMI_D6,LCD_B6,EVENTOUT)
- net IDIFF1: now also U1101.4 (PE5,TRACED2,TIM9_CH1,SPI4_MISO,SAI1_SCK_A,DFSDM1_CKIN3,FMC_A21,DCMI_D6,LCD_G0,EVENTOUT); no longer U1101.140 (PB9,I2C4_SDA,TIM4_CH4,TIM11_CH1,I2C1_SDA,SPI2_NSS,I2S2_WS,DFSDM1_DATIN7,UART5_TX,CAN1_TX,SDMMC2_D5,I2C4_SMBA,SDMMC1_D5,DCMI_D7,LCD_B7,EVENTOUT)
- net ~DDS_DIV10: now also U1101.142 (PE1,LPTIM1_IN2,UART8_TX,FMC_NBL1,DCMI_D3,EVENTOUT); no longer U1101.55 (PF15,I2C4_SDA,FMC_A9,EVENTOUT)
- net at U1101.7 (PC13,EVENTOUT,RTC_TAMP2,RTC_TS,WKUP5): no longer R1101.1
- net at U1101.8 (PC14,EVENTOUT,OSC32_IN): no longer R1102.1
- net at U1101.9 (PC15,EVENTOUT,OSC32_OUT): no longer R1103.1
- net LED_GREEN: now reaches U1101.124 (PG9,SPI1_MISO,SPDIF_RX3,USART6_RX,QUADSPI_BK2_IO2,SAI2_FS_B,SDMMC2_D0,FMC_NE2,FMC_NCE,DCMI_VSYNC,EVENTOUT)
- net LED_GREEN: now also R1102.1
- net LED_RED: now reaches U1101.125 (PG10,SPI1_NSS,I2S1_WS,LCD_G3,SAI2_SD_B,SDMMC2_D1,FMC_NE3,DCMI_D2,LCD_B2,EVENTOUT)
- net LED_RED: now also R1101.1
- net SPI5_NSS: now reaches U1101.18 (PF6,TIM10_CH1,SPI5_NSS,SAI1_SD_B,UART7_RX,QUADSPI_BK1_IO3,EVENTOUT,ADC3_IN4)
- net SPI5_SCK: now reaches U1101.19 (PF7,TIM11_CH1,SPI5_SCK,SAI1_MCLK_B,UART7_TX,QUADSPI_BK1_IO2,EVENTOUT,ADC3_IN5)
- net SPI5_MISO: now reaches U1101.20 (PF8,SPI5_MISO,SAI1_SCK_B,UART7_RTS,TIM13_CH1,QUADSPI_BK1_IO0,EVENTOUT,ADC3_IN6)
- net SPI5_MOSI: now reaches U1101.21 (PF9,SPI5_MOSI,SAI1_FS_B,UART7_CTS,TIM14_CH1,QUADSPI_BK1_IO1,EVENTOUT,ADC3_IN7)
- net SPI1_MISO: no longer names the net of U1101.42 (PA6,TIM1_BKIN,TIM3_CH1,TIM8_BKIN,SPI1_MISO,SPI6_MISO,TIM13_CH1,MDIOS_MDC,DCMI_PIXCLK,LCD_G2,EVENTOUT,ADC1_IN6,ADC2_IN6)
- net SPI1_MOSI renamed LED_BLUE
- net LED_BLUE: now also R1103.1
- net SPI1_NSS: no longer names the net of U1101.40 (PA4,SPI1_NSS,I2S1_WS,SPI3_NSS,I2S3_WS,USART2_CK,SPI6_NSS,OTG_HS_SOF,DCMI_HSYNC,LCD_VSYNC,EVENTOUT,ADC1_IN4,ADC2_IN4,DAC_OUT1)
- net SPI1_SCK: no longer names the net of U1101.41 (PA5,TIM2_CH1,TIM2_ETR,TIM8_CH1N,SPI1_SCK,I2S1_CK,SPI6_SCK,OTG_HS_ULPI_CK,LCD_R4,EVENTOUT,ADC1_IN5,ADC2_IN5,DAC_OUT2)
Other:
- moved on the sheet: D1101, D1102, D1103, R1101, R1102, R1103
Changed lines of the file:
@@
 L Device:R R1101
 U 1 1 5E648C3B
-P 3250 6550
-F 0 "R1101" V 3043 6550 50  0000 C CNN
-F 1 "680" V 3134 6550 50  0000 C CNN
-F 2 "Resistor_SMD:R_0603_1608Metric_Pad0.98x0.95mm_HandSolder" V 3180 6550 50  0001 C CNN
-F 3 "~" H 3250 6550 50  0001 C CNN
-	1    3250 6550
+P 2500 6500
+F 0 "R1101" V 2293 6500 50  0000 C CNN
+F 1 "680" V 2384 6500 50  0000 C CNN
+F 2 "Resistor_SMD:R_0603_1608Metric_Pad0.98x0.95mm_HandSolder" V 2430 6500 50  0001 C CNN
+F 3 "~" H 2500 6500 50  0001 C CNN
+	1    2500 6500
 	0    1    1    0
 $EndComp
@@
 L Device:R R1102
 U 1 1 5E64A32E
-P 3250 6950
-F 0 "R1102" V 3043 6950 50  0000 C CNN
-F 1 "560" V 3134 6950 50  0000 C CNN
-F 2 "Resistor_SMD:R_0603_1608Metric_Pad0.98x0.95mm_HandSolder" V 3180 6950 50  0001 C CNN
-F 3 "~" H 3250 6950 50  0001 C CNN
-	1    3250 6950
+P 2500 6900
+F 0 "R1102" V 2293 6900 50  0000 C CNN
+F 1 "560" V 2384 6900 50  0000 C CNN
+F 2 "Resistor_SMD:R_0603_1608Metric_Pad0.98x0.95mm_HandSolder" V 2430 6900 50  0001 C CNN
+F 3 "~" H 2500 6900 50  0001 C CNN
+	1    2500 6900
 	0    1    1    0
 $EndComp
@@
 L Device:R R1103
 U 1 1 5E64A698
-P 3250 7350
-F 0 "R1103" V 3043 7350 50  0000 C CNN
-F 1 "680" V 3134 7350 50  0000 C CNN
-F 2 "Resistor_SMD:R_0603_1608Metric_Pad0.98x0.95mm_HandSolder" V 3180 7350 50  0001 C CNN
-F 3 "~" H 3250 7350 50  0001 C CNN
-	1    3250 7350
+P 2500 7300
+F 0 "R1103" V 2293 7300 50  0000 C CNN
+F 1 "680" V 2384 7300 50  0000 C CNN
+F 2 "Resistor_SMD:R_0603_1608Metric_Pad0.98x0.95mm_HandSolder" V 2430 7300 50  0001 C CNN
+F 3 "~" H 2500 7300 50  0001 C CNN
+	1    2500 7300
 	0    1    1    0
 $EndComp
@@
 L Device:LED D1101
 U 1 1 5E66EF29
-P 2900 6550
-F 0 "D1101" H 2893 6295 50  0000 C CNN
-F 1 "RED" H 2893 6386 50  0000 C CNN
-F 2 "LED_SMD:LED_0603_1608Metric_Pad1.05x0.95mm_HandSolder" H 2900 6550 50  0001 C CNN
-F 3 "~" H 2900 6550 50  0001 C CNN
-	1    2900 6550
+P 2150 6500
+F 0 "D1101" H 2143 6245 50  0000 C CNN
+F 1 "RED" H 2143 6336 50  0000 C CNN
+F 2 "LED_SMD:LED_0603_1608Metric_Pad1.05x0.95mm_HandSolder" H 2150 6500 50  0001 C CNN
+F 3 "~" H 2150 6500 50  0001 C CNN
+	1    2150 6500
 	-1   0    0    1
 $EndComp
@@
 L Device:LED D1102
 U 1 1 5E66FC1B
-P 2900 6950
-F 0 "D1102" H 2893 6695 50  0000 C CNN
-F 1 "GREEN" H 2893 6786 50  0000 C CNN
-F 2 "LED_SMD:LED_0603_1608Metric_Pad1.05x0.95mm_HandSolder" H 2900 6950 50  0001 C CNN
-F 3 "~" H 2900 6950 50  0001 C CNN
-	1    2900 6950
+P 2150 6900
+F 0 "D1102" H 2143 6645 50  0000 C CNN
+F 1 "GREEN" H 2143 6736 50  0000 C CNN
+F 2 "LED_SMD:LED_0603_1608Metric_Pad1.05x0.95mm_HandSolder" H 2150 6900 50  0001 C CNN
+F 3 "~" H 2150 6900 50  0001 C CNN
+	1    2150 6900
 	-1   0    0    1
 $EndComp
@@
 L Device:LED D1103
 U 1 1 5E69BE69
-P 2900 7350
-F 0 "D1103" H 2893 7095 50  0000 C CNN
-F 1 "BLUE" H 2893 7186 50  0000 C CNN
-F 2 "LED_SMD:LED_0603_1608Metric_Pad1.05x0.95mm_HandSolder" H 2900 7350 50  0001 C CNN
-F 3 "~" H 2900 7350 50  0001 C CNN
-	1    2900 7350
+P 2150 7300
+F 0 "D1103" H 2143 7045 50  0000 C CNN
+F 1 "BLUE" H 2143 7136 50  0000 C CNN
+F 2 "LED_SMD:LED_0603_1608Metric_Pad1.05x0.95mm_HandSolder" H 2150 7300 50  0001 C CNN
+F 3 "~" H 2150 7300 50  0001 C CNN
+	1    2150 7300
 	-1   0    0    1
 $EndComp
 Wire Wire Line
-	3100 7350 3050 7350
-Wire Wire Line
-	2700 7350 2700 6950
-Wire Wire Line
-	2700 6550 2750 6550
-Wire Wire Line
-	2750 7350 2700 7350
-Wire Wire Line
-	2700 6950 2750 6950
-Connection ~ 2700 6950
-Wire Wire Line
-	2700 6950 2700 6550
-Wire Wire Line
-	3050 6950 3100 6950
-Wire Wire Line
-	3050 6550 3100 6550
-Wire Wire Line
-	2650 6950 2700 6950
+	2350 7300 2300 7300
+Wire Wire Line
+	1950 7300 1950 6900
+Wire Wire Line
+	1950 6500 2000 6500
+Wire Wire Line
+	2000 7300 1950 7300
+Wire Wire Line
+	1950 6900 2000 6900
+Connection ~ 1950 6900
+Wire Wire Line
+	1950 6900 1950 6500
+Wire Wire Line
+	2300 6900 2350 6900
+Wire Wire Line
+	2300 6500 2350 6500
+Wire Wire Line
+	1900 6900 1950 6900
 $Comp
 L Sensor_Humidity:HDC1080 U1102
@@
 $EndComp
 Wire Wire Line
-	3400 6550 3450 6550
-Wire Wire Line
-	3450 6550 3450 6200
-Wire Wire Line
-	3450 6200 3650 6200
-Wire Wire Line
-	3400 6950 3500 6950
-Wire Wire Line
-	3500 6950 3500 6300
-Wire Wire Line
-	3500 6300 3650 6300
-Wire Wire Line
-	3550 7350 3550 6400
-Wire Wire Line
-	3550 6400 3650 6400
-Wire Wire Line
-	3400 7350 3550 7350
-Wire Wire Line
 	10350 10350 10950 10350
 Wire Wire Line
@@
 	1850 9400 2050 9400
 Connection ~ 1850 9400
-NoConn ~ 15050 2200
-NoConn ~ 15050 2100
-NoConn ~ 15050 4900
 $Comp
 L power:+3.3V #PWR01118
@@
 L power:+3.3V #PWR01103
 U 1 1 6057A4C1
-P 2650 6950
-F 0 "#PWR01103" H 2650 6800 50  0001 C CNN
-F 1 "+3.3V" V 2650 7100 50  0000 L CNN
-F 2 "" H 2650 6950 50  0001 C CNN
-F 3 "" H 2650 6950 50  0001 C CNN
-	1    2650 6950
+P 1900 6900
+F 0 "#PWR01103" H 1900 6750 50  0001 C CNN
+F 1 "+3.3V" V 1900 7050 50  0000 L CNN
+F 2 "" H 1900 6900 50  0001 C CNN
+F 3 "" H 1900 6900 50  0001 C CNN
+	1    1900 6900
 	0    -1   -1   0
 $EndComp
@@
 Wire Wire Line
 	15050 7600 15100 7600
-Text HLabel 3600 3600 0    50   Output ~ 0
-SPI1_NSS
-Wire Wire Line
-	3600 3600 3650 3600
-Text HLabel 3600 3700 0    50   Output ~ 0
-SPI1_SCK
-Wire Wire Line
-	3600 3700 3650 3700
-Text HLabel 15100 3600 2    50   Output ~ 0
-SPI1_MOSI
-Wire Wire Line
-	15100 3600 15050 3600
+Text HLabel 3600 2400 0    50   Output ~ 0
+SPI5_MOSI
+Wire Wire Line
+	3600 2400 3650 2400
 Text HLabel 3600 6100 0    50   Output ~ 0
 SPI3_MOSI
@@
 Wire Wire Line
 	3650 5500 3600 5500
-Text HLabel 15100 7200 2    50   Output ~ 0
+Text HLabel 15100 5100 2    50   Output ~ 0
 IDIFF1
-Text HLabel 15100 7100 2    50   Output ~ 0
+Text HLabel 15100 4900 2    50   Output ~ 0
 IDIFF0
 Wire Wire Line
-	15050 7100 15100 7100
-Wire Wire Line
-	15100 7200 15050 7200
+	15050 4900 15100 4900
+Wire Wire Line
+	15100 5100 15050 5100
 NoConn ~ 15050 5300
 NoConn ~ 15050 5400
 NoConn ~ 15050 5500
-NoConn ~ 15050 4700
-NoConn ~ 15050 4600
 NoConn ~ 15050 4400
 NoConn ~ 15050 2700
@@
 Wire Wire Line
 	15050 2900 15100 2900
-NoConn ~ 3650 2100
-NoConn ~ 3650 2200
-NoConn ~ 3650 2300
-NoConn ~ 3650 2400
-Text HLabel 3600 3800 0    50   Input ~ 0
-SPI1_MISO
-Wire Wire Line
-	3650 3800 3600 3800
-Text HLabel 3600 2700 0    50   Output ~ 0
+Text HLabel 15100 4600 2    50   Output ~ 0
 DDS_DIV2
-Text HLabel 3600 2800 0    50   Output ~ 0
+Text HLabel 15100 7200 2    50   Output ~ 0
 DDS_DIV4
-Text HLabel 3600 2900 0    50   Output ~ 0
+Text HLabel 15100 7100 2    50   Output ~ 0
 DDS_DIV8
-Text HLabel 3600 3000 0    50   Output ~ 0
+Text HLabel 15100 4700 2    50   Output ~ 0
 ~DDS_DIV10
 Wire Wire Line
-	3650 2700 3600 2700
-Wire Wire Line
-	3600 2800 3650 2800
-Wire Wire Line
-	3650 2900 3600 2900
-Wire Wire Line
-	3600 3000 3650 3000
+	15050 4600 15100 4600
+Wire Wire Line
+	15100 7200 15050 7200
+Wire Wire Line
+	15050 7100 15100 7100
+Wire Wire Line
+	15100 4700 15050 4700
 NoConn ~ 15050 3200
 NoConn ~ 15050 3300
@@
 Wire Wire Line
 	15100 5000 15050 5000
-NoConn ~ 15050 5100
 NoConn ~ 3650 3500
 $Comp
@@
 NoConn ~ 15050 1900
 NoConn ~ 15050 1800
+Text HLabel 3600 2300 0    50   Input ~ 0
+SPI5_MISO
+Text HLabel 3600 2200 0    50   Output ~ 0
+SPI5_SCK
+Text HLabel 3600 2100 0    50   Output ~ 0
+SPI5_NSS
+Wire Wire Line
+	3600 2100 3650 2100
+Wire Wire Line
+	3600 2200 3650 2200
+Wire Wire Line
+	3600 2300 3650 2300
+NoConn ~ 3650 3000
+NoConn ~ 3650 3600
+NoConn ~ 3650 3700
+NoConn ~ 3650 3800
+NoConn ~ 3650 2900
+NoConn ~ 3650 2800
+NoConn ~ 3650 2700
+NoConn ~ 3650 6200
+NoConn ~ 3650 6300
+NoConn ~ 3650 6400
+Wire Wire Line
+	15050 2100 15550 2100
+Wire Wire Line
+	15050 2200 15550 2200
+Wire Wire Line
+	15050 3600 15550 3600
+Wire Wire Line
+	2650 7300 3100 7300
+Text Label 3100 7300 2    50   ~ 0
+LED_BLUE
+Text Label 15550 3600 2    50   ~ 0
+LED_BLUE
+Wire Wire Line
+	2650 6900 3100 6900
+Text Label 3100 6900 2    50   ~ 0
+LED_GREEN
+Text Label 15550 2100 2    50   ~ 0
+LED_GREEN
+Wire Wire Line
+	2650 6500 3100 6500
+Text Label 3100 6500 2    50   ~ 0
+LED_RED
+Text Label 15550 2200 2    50   ~ 0
+LED_RED
 $EndSCHEMATC

Commit message: PCB
Connections:
- net ADC_SEL: now reaches U1101.117 (PD3,DFSDM1_CKOUT,SPI2_SCK,I2S2_CK,DFSDM1_DATIN0,USART2_CTS,FMC_CLK,DCMI_D5,LCD_G7,EVENTOUT)
- net DDS_LPF: now reaches U1101.135 (PB5,UART5_RX,TIM3_CH2,I2C1_SMBA,SPI1_MOSI,I2S1_SD,SPI3_MOSI,I2S3_SD,SPI6_MOSI,CAN2_RX,OTG_HS_ULPI_D7,ETH_PPS_OUT,FMC_SDCKE1,DCMI_D10,LCD_G7,EVENTOUT)
- net MUX_A0: now reaches U1101.136 (PB6,UART5_TX,TIM4_CH1,HDMI_CEC,I2C1_SCL,DFSDM1_DATIN5,USART1_TX,CAN2_TX,QUADSPI_BK1_NCS,I2C4_SCL,FMC_SDNE1,DCMI_D5,EVENTOUT)
- net MUX_A1: now reaches U1101.137 (PB7,TIM4_CH2,I2C1_SDA,DFSDM1_CKIN5,USART1_RX,I2C4_SDA,FMC_NL,DCMI_VSYNC,EVENTOUT)
- no-connect marks 52 -> 49
Changed lines of the file:
@@
 Wire Wire Line
 	15100 4700 15050 4700
-NoConn ~ 15050 3200
 NoConn ~ 15050 3300
 NoConn ~ 15050 3400
@@
 Wire Wire Line
 	3650 4100 3600 4100
-NoConn ~ 15050 7000
-NoConn ~ 15050 6900
-NoConn ~ 15050 6800
 NoConn ~ 15050 6700
 NoConn ~ 15050 6400
@@
 Text Label 15550 2200 2    50   ~ 0
 LED_RED
+Text HLabel 15100 3200 2    50   Output ~ 0
+ADC_SEL
+Wire Wire Line
+	15100 3200 15050 3200
+NoConn ~ 15050 1500
+Text HLabel 15100 6900 2    50   Output ~ 0
+MUX_A0
+Text HLabel 15100 7000 2    50   Output ~ 0
+MUX_A1
+Text HLabel 15100 6800 2    50   Output ~ 0
+DDS_LPF
+Wire Wire Line
+	15100 7000 15050 7000
+Wire Wire Line
+	15050 6900 15100 6900
+Wire Wire Line
+	15100 6800 15050 6800
 $EndSCHEMATC
