File: hardware/ETH1CLCR2/ETH1CLCR2.kicad_pcb (KiCad board)
At the start: 2 copper layers, 487 parts, among them J1101 Conn_02x01, J1102 20021111-00010T4LF, J401 C64AC, K401 HE3621A0510, K402 HE3621A0510, K403 HE3621A0510, K404 HE3621A0510, K405 HE3621A0510, K601 TQ2SA-5V, K801 TQ2SA-5V, Q1201 BC847, Q1202 BC847, Q1203 BC857, Q1204 BC847, Q1205 BC857, Q1206 BC857, Q601 MMBFJ309LT1G, Q602 MMBFJ309LT1G, Q603 BC847, Q604 BC857, Q605 MMBFJ309LT1G, Q606 MMBFJ309LT1G, Q607 BC847, Q608 BC857, Q609 MMBFJ309LT1G, Q610 MMBFJ309LT1G, Q611 BC847, Q612 BC857, Q613 MMBFJ309LT1G, Q614 MMBFJ309LT1G, Q615 BC847, Q616 BC857, Q617 BC847, Q801 BC847, Q901 IRFR5410, U1001 MCP6L91RT-ESN, U1002 MCP661, U1003 SN74LVC1G3157, U1004 SN74LVC1G3157, U1005 MCP661, U1006 MCP6L91RT-ESN, U1007 SN74LVC1T45DBV, U1008 SN74LVC1G3157, U1009 SN74LVC1G3157, U1010 MCP661, U1011 MCP6L91RT-ESN, U1012 SN74LVC1T45DBV, U1101 STM32H743ZI, U1102 HDC1080, U1103 24LC08B-E/MS, U1201 LM318, U1202 AD5452YRMZ, U1203 LT1468, U1204 MC33078, U1205 AD9835, U1206 ECS-3225SMV-500-GP-TR, U1207 74AHCT1G08, U1208 DG419LDY, U1209 SN74LVC1T45DBV, U1210 REF192, U201 LC03-3.3, U202 LAN8742A, U203 LC03-3.3, U301 74AC125, U302 TXB0104PW, U303 ADuM5402, U401 ULN2003A, U501 ADS8681PWR, U502 ADS8681PWR, U601 SN74LVC1T45DBV, U602 SN74LVC1T45DBV, U603 SN74LVC1T45DBV, U604 SN74LVC1T45DBV, U605 ADA4817-1ARDZ, U701 REF5040ID, U702 TL431BCDE4, U703 MCP6L91RT-EMS, U801 MCP6L91RT-ESN, U802 MCP661, U803 MCP661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

Commit message: PCB layout
Parts:
- added C905: 4u7/50V, Capacitor_SMD:C_1206_3216Metric_Pad1.33x1.80mm_HandSolder, F.Cu at (201.2, 112.4)
- added C906: 4u7/50V, Capacitor_SMD:C_1206_3216Metric_Pad1.33x1.80mm_HandSolder, F.Cu at (203.7, 112.4)
- added J101: RF_Shield_One_Piece, ETH1CLCR2:36107406S, F.Cu at (181.5, -73.0)
- F901: moved to B.Cu
- U605: footprint Package_SO:SOIC-8_3.9x4.9mm_P1.27mm -> Package_SO:SOIC-8-1EP_3.9x4.9mm_P1.27mm_EP2.29x3mm
- moved C303 257.2 mm to (407.4, -73.8)
- moved C304 257.2 mm to (398.7, -72.8)
- moved C1001 257.2 mm to (401.9, -98.4)
- moved C1002 257.2 mm to (412.2, -97.1)
- moved C1003 257.2 mm to (427.1, -112.7)
- moved C1006 257.2 mm to (434.1, -102.3)
- moved C1007 257.2 mm to (439.7, -107.3)
- moved C1009 257.2 mm to (426.6, -117.7)
- moved C1010 257.2 mm to (417.9, -106.6)
- moved C1011 257.2 mm to (426.6, -115.2)
- moved C1012 257.2 mm to (412.4, -102.1)
- moved C1014 257.2 mm to (430.2, -122.4)
- moved C1015 257.2 mm to (430.9, -119.9)
- moved C1017 257.2 mm to (412.2, -99.6)
- moved C1018 257.2 mm to (417.9, -104.1)
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- renumbered C905 to C907, C906 to C908, C907 to C909, C908 to C910, C909 to C911, C910 to C912, C911 to C913, C912 to C914, C913 to C915, C914 to C916, C915 to C917, C916 to C918
Other:
- board outline added: 160 x 100 mm
- copper layers 2 -> 4

Commit message: PCB layout
Parts:
- C1101, C1102, C1103, C1104, C1105, C1106, C1107, C1108, C1109, C1110, C1111, C1112, C1113, C1114, C1115, C1116, C1117, C1118, C1119, C1120, C1121, C1122, C202, C203, C204, C205, C207, C208, C210, C211, C212, C213, C214, C301, C302, C303, C304, C305, C306, C307, C308, C401, C503, C504, C505, C506, C507, C508, C701, C702, FB1101, FB201, R1104, R1105, R1109, R1110, R201, R202, R203, R204, R209, R210, R211, R213, R214, R215, R216, R217, R218, R219, R220, R301, R302, R306, R507, R508, R701, R901, U1103, Y1101: moved to B.Cu
- moved C506 322.2 mm to (114.4, 99.6), turned to 270 degrees
- moved R506 321.9 mm to (112.6, 100.8), turned to 270 degrees
- moved R508 319.8 mm to (117.0, 99.6), turned to 90 degrees
- moved C501 317.8 mm to (112.6, 90.2), turned to 90 degrees
- moved C502 315.7 mm to (112.6, 97.4), turned to 90 degrees
- moved C507 314.8 mm to (118.2, 88.5)
- moved C508 313.3 mm to (118.2, 96.1)
- moved R501 312.1 mm to (124.5, 94.2), turned to 180 degrees
- moved C505 311.1 mm to (119.6, 99.6), turned to 270 degrees
- moved R504 310.8 mm to (124.5, 101.7), turned to 180 degrees
- moved C510 310.8 mm to (124.5, 89.4)
- moved R507 310.4 mm to (117.0, 91.8), turned to 90 degrees
- moved R503 310.0 mm to (112.6, 93.6), turned to 270 degrees
- moved C509 309.3 mm to (124.5, 96.9)
- moved C302 306.4 mm to (169.0, 87.0)
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Routing:
- net Net-(D302-Pad3): track 0.00 -> 19.1 mm
- net Net-(D902-Pad1): track 0.00 -> 18.0 mm, vias 0 -> 7
- net GND_TRIG: track 0.00 -> 14.7 mm, vias 0 -> 6
- net /Trigger/EXT_TRIG_SIGN: track 0.00 -> 13.6 mm
- net /Trigger/TRIG_OUT_SIGN: track 0.00 -> 12.3 mm
- net /Connector/EXT_TRIG: track 0.00 -> 11.1 mm
- net Net-(R303-Pad2): track 0.00 -> 9.70 mm, vias 0 -> 2
- net Net-(D301-Pad1): track 0.00 -> 9.18 mm, vias 0 -> 1
- net GNDPWR: track 0.00 -> 8.70 mm, vias 0 -> 7
- net Net-(C905-Pad1): track 0.00 -> 8.67 mm, vias 0 -> 9
- net +5V_TRIG: track 0.00 -> 7.77 mm, vias 0 -> 3
- net +24V: track 0.00 -> 7.48 mm, vias 0 -> 5
- net /Trigger/TRIG_OUT_EN: track 0.00 -> 6.76 mm, vias 0 -> 2
- net Net-(Q901-Pad1): track 0.00 -> 5.61 mm
- net Net-(L201-Pad14): track 0.00 -> 3.70 mm
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- added copper zone on B.Cu, net +24V
- added copper zone on F.Cu, net +24V
- added copper zone on In2.Cu, net +24V
- added copper zone on In2.Cu, net +5V_TRIG
- added copper zone on B.Cu, net Earth
- added copper zone on B.Cu, net GNDPWR
- added copper zone on F.Cu, net GNDPWR
- added copper zone on In1.Cu, net GNDPWR
- added copper zone on B.Cu, net GND_TRIG
- added copper zone on F.Cu, net GND_TRIG
- added copper zone on In1.Cu, net GND_TRIG
- added copper zone on B.Cu, net Net-(C905-Pad1)
- added copper zone on F.Cu, net Net-(C905-Pad1)
- added copper zone on In2.Cu, net Net-(C905-Pad1)
- added copper zone on B.Cu, net Net-(D902-Pad1)
- added copper zone on F.Cu, net Net-(D902-Pad1)
- added copper zone on F.Cu, net Net-(Q901-Pad1)
Other:
- net class Default: clearance 0.2 -> 0.127; trace_width 0.25 -> 0.127; via_dia 0.8 -> 0.5; via_drill 0.4 -> 0.2
- rule trace_clearance: 0.2 -> 0.127
- rule trace_min: 0.2 -> 0.127
- rule via_min_drill: 0.3 -> 0.2
- rule via_min_size: 0.4 -> 0.5

Commit message: PCB layout
Parts:
- C807, C808, C809, C810, D802, Q801, R808, R810, R820, R824: moved to B.Cu
- moved R807 206.6 mm to (116.5, 62.7)
- moved R806 198.2 mm to (120.5, 62.7)
- moved R824 196.8 mm to (127.5, 72.0), turned to 270 degrees
- moved R810 192.0 mm to (139.2, 65.2)
- moved U804 191.8 mm to (102.6, 61.3)
- moved R812 189.8 mm to (120.5, 72.3)
- moved C809 186.7 mm to (125.1, 62.9), turned to 90 degrees
- moved R813 182.2 mm to (116.5, 72.3)
- moved D802 179.9 mm to (139.2, 72.5), turned to 180 degrees
- moved C808 179.6 mm to (151.0, 62.2), turned to 180 degrees
- moved Q801 177.2 mm to (139.2, 68.6), turned to 270 degrees
- moved C810 177.1 mm to (125.0, 72.0), turned to 90 degrees
- moved U802 168.0 mm to (127.5, 62.9), turned to 180 degrees
- moved C807 167.2 mm to (151.0, 72.6)
- moved R808 166.0 mm to (127.5, 62.9), turned to 270 degrees
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Routing:
- added copper zone on F.Cu, net Earth
- added copper zone on In1.Cu, net Earth
- added copper zone on In2.Cu, net Earth

Commit message: Modification of the function generator schematic.
Parts:
- removed C1201: 1p5, Capacitor_SMD:C_0603_1608Metric_Pad1.08x0.95mm_HandSolder
- removed C1202, C1213: 10n, Capacitor_SMD:C_0603_1608Metric_Pad1.08x0.95mm_HandSolder
- removed C1203: 4p7, Capacitor_SMD:C_0603_1608Metric_Pad1.08x0.95mm_HandSolder
- removed C1204: 18p, Capacitor_SMD:C_0603_1608Metric_Pad1.08x0.95mm_HandSolder
- removed C1205: 12p, Capacitor_SMD:C_0603_1608Metric_Pad1.08x0.95mm_HandSolder
- removed C1206: 10u, Capacitor_SMD:C_1206_3216Metric_Pad1.33x1.80mm_HandSolder
- removed C1207, C1218: 1u, Capacitor_SMD:C_0603_1608Metric_Pad1.08x0.95mm_HandSolder
- removed C1208, C1211: 22p, Capacitor_SMD:C_0603_1608Metric_Pad1.08x0.95mm_HandSolder
- removed C1209, C1210: 56p, Capacitor_SMD:C_0603_1608Metric_Pad1.08x0.95mm_HandSolder
- removed C1212, C1214, C1216, C1219: 100n, Capacitor_SMD:C_0603_1608Metric_Pad1.08x0.95mm_HandSolder
- removed C1215: 5p, Capacitor_SMD:C_0603_1608Metric_Pad1.08x0.95mm_HandSolder
- removed C1217: 10u, Capacitor_SMD:C_0805_2012Metric_Pad1.18x1.45mm_HandSolder
- removed D1201: SD103ATW, Package_TO_SOT_SMD:SOT-363_SC-70-6
- removed L1201, L1202, L1203: 4u7, Inductor_SMD:L_0603_1608Metric_Pad1.05x0.95mm_HandSolder
- removed Q1201, Q1202, Q1204: BC847, Package_TO_SOT_SMD:SOT-23
- removed Q1203, Q1205, Q1206: BC857, Package_TO_SOT_SMD:SOT-23
- removed R1201: 10k, Resistor_SMD:R_0603_1608Metric_Pad0.98x0.95mm_HandSolder
- removed R1202, R1203: 1k, Resistor_SMD:R_0603_1608Metric_Pad0.98x0.95mm_HandSolder
- removed R1204, R1210: 0, Resistor_SMD:R_0603_1608Metric_Pad0.98x0.95mm_HandSolder
- removed R1205, R1206: 300, Resistor_SMD:R_0603_1608Metric_Pad0.98x0.95mm_HandSolder
- removed R1207: 1k/.1%, Resistor_SMD:R_0805_2012Metric_Pad1.20x1.40mm_HandSolder
- removed R1208: xxk/.1%, Resistor_SMD:R_0805_2012Metric_Pad1.20x1.40mm_HandSolder
- removed R1209: 3k9, Resistor_SMD:R_0603_1608Metric_Pad0.98x0.95mm_HandSolder
- removed R1211, R1223: 1k/.1%, Resistor_SMD:R_0603_1608Metric_Pad0.98x0.95mm_HandSolder
- removed R1212: 4k22/.1%, Resistor_SMD:R_0603_1608Metric_Pad0.98x0.95mm_HandSolder
- removed R1213, R1222: 22k/.1%, Resistor_SMD:R_0603_1608Metric_Pad0.98x0.95mm_HandSolder
- removed R1214: 3k9/.1%, Resistor_SMD:R_0603_1608Metric_Pad0.98x0.95mm_HandSolder
- removed R1215, R1216, R1220, R1221: 22/0.5W, Resistor_SMD:R_1206_3216Metric_Pad1.30x1.75mm_HandSolder
- removed R1217, R1219: 470/.1%, Resistor_SMD:R_0603_1608Metric_Pad0.98x0.95mm_HandSolder
- removed R1218: 10/0.5W, Resistor_SMD:R_1206_3216Metric_Pad1.30x1.75mm_HandSolder
- removed TP1201, TP1202, TP1203: TestPoint, TestPoint:TestPoint_Plated_Hole_D2.0mm
- removed U1202: AD5452YRMZ, Package_SO:MSOP-8_3x3mm_P0.65mm
- removed U1203: LT1468, Package_SO:SOIC-8_3.9x4.9mm_P1.27mm
- removed U1204: MC33078, Package_SO:SOIC-8_3.9x4.9mm_P1.27mm
- removed U1205: AD9835, Package_SO:TSSOP-16_4.4x5mm_P0.65mm
- removed U1206: ECS-3225SMV-500-GP-TR, ETH1CLCR2:ECS
- removed U1207: 74AHCT1G08, Package_TO_SOT_SMD:SOT-353_SC-70-5
- removed U1208: DG419LDY, Package_SO:SOIC-8_3.9x4.9mm_P1.27mm
- removed U1209: SN74LVC1T45DBV, Package_TO_SOT_SMD:SOT-23-6
- removed U1210: REF192, Package_SO:SSOP-8_3.9x5.05mm_P1.27mm
- added U909: NCP1117-5.0_TO252, Package_TO_SOT_SMD:TO-252-2, F.Cu at (141.4, 127.6)
- added U910: NCP1117-5.0_SOT223, Package_TO_SOT_SMD:SOT-223-3_TabPin2, F.Cu at (126.7, 127.6)
- added U911: LT1175-5_SOT223, Package_TO_SOT_SMD:SOT-223-3_TabPin2, F.Cu at (110.9, 127.3)
- U1201: value LM318 -> AD9834; footprint Package_SO:SOIC-8_3.9x4.9mm_P1.27mm -> Package_SO:TSSOP-20_4.4x6.5mm_P0.65mm
- U901: value NCP1117-3.3_SOT223 -> NMK0509SC; footprint Package_TO_SOT_SMD:SOT-223-3_TabPin2 -> ETH1CLCR2:NMK_DUAL
- U906: value NCP1117-5.0_SOT223 -> LT1175-5_SOT223
- U908: value LT1175-5_SOT223 -> NCP1117-3.3_TO252; footprint Package_TO_SOT_SMD:SOT-223-3_TabPin2 -> Package_TO_SOT_SMD:TO-252-2
- moved U1201 284.9 mm to (75.7, 109.2), turned to 90 degrees
- moved U901 85.7 mm to (77.7, 134.7), turned to 180 degrees
- moved U904 62.1 mm to (90.0, 122.0)
- moved U908 56.4 mm to (163.2, 127.5), turned to 180 degrees
- moved U906 47.8 mm to (70.0, 122.2)
- moved J1101 29.9 mm to (138.2, 90.8)
- moved K601 24.3 mm to (160.7, 49.7), turned to 90 degrees
- moved C807 21.7 mm to (172.5, 69.7)
- moved C808 21.7 mm to (172.5, 59.3)
- moved U801 21.7 mm to (172.5, 59.9)
- moved U807 21.7 mm to (172.5, 69.1)
- moved C810 21.7 mm to (146.4, 69.1)
- moved R808 21.7 mm to (149.0, 59.9)
- moved R824 21.7 mm to (149.0, 69.1)
- moved U802 21.7 mm to (149.0, 59.9)
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- renumbered C915 to C916, C916 to C917, C917 to C918, C918 to C919
Connections:
- C911 pad 2: GND -> GNDA
- C912 pad 2: GND -> GNDA
- C913 pad 2: GND -> GNDA
- C914 pad 2: GND -> GNDA
- C916 pad 1: GND -> GNDA
- C916 pad 2: Net-(C915-Pad2) -> Net-(C916-Pad2)
- C917 pad 1: GND -> GNDA
- C918 pad 1: GND -> GNDA
- C919 pad 1: GND -> GNDA
- K401 pad 1: /Connector/H_CUR -> (no net)
- U1101 pad 123: /FGEN/DDS_MDAC_DIN -> (no net)
- U1101 pad 40: /FGEN/DDS_MDAC_~SYNC -> (no net)
- U1101 pad 41: /FGEN/DDS_MDAC_SCLK -> (no net)
- U1101 pad 68: /FGEN/DDS_FGEN_FSELECT -> (no net)
- U1101 pad 69: /FGEN/DDS_FGEN_PSEL0 -> (no net)
- U1101 pad 70: /FGEN/DDS_FGEN_PSEL1 -> (no net)
- U1101 pad 73: /FGEN/DDS_FGEN_~FSYNC -> (no net)
- U1101 pad 74: /FGEN/DDS_FGEN_SCLK -> (no net)
- U1101 pad 76: /FGEN/DDS_FGEN_SDATA -> (no net)
- U1101 pad 77: /FGEN/FGEN_SEL -> (no net)
- U1201 pad 2: Net-(C1215-Pad2) -> (no net)
- U1201 pad 3: GND -> (no net)
- U1201 pad 4: -5VA -> +5VF
- U1201 pad 5: (no net) -> +5VF
- U1201 pad 6: Net-(C1215-Pad1) -> (no net)
- U1201 pad 7: +5VA -> AGNDF
- U901 pad 1: GND -> +5V
- U901 pad 2: +3V3 -> GND
- U904 pad 1: GND -> AGNDF
- U904 pad 2: +5V -> +5VF
- U904 pad 3: Net-(C907-Pad1) -> Net-(C921-Pad1)
- U906 pad 1: GND -> (no net)
- U906 pad 2: +5VA -> Net-(C922-Pad2)
- U906 pad 3: Net-(C911-Pad1) -> AGNDF
- U907 pad 5: Net-(C915-Pad2) -> Net-(C916-Pad2)
- U907 pad 6: GND -> GNDA
- U908 pad 1: -5VA -> GND
- U908 pad 2: Net-(C915-Pad2) -> +3V3
- U908 pad 3: GND -> Net-(C901-Pad1)
Routing:
- net GND_TRIG: track 14.7 -> 5.69 mm
- net /Connector/EXT_TRIG: track 11.1 -> 6.76 mm
- removed copper zone on B.Cu, net Earth
- removed copper zone on F.Cu, net Earth
- removed copper zone on In1.Cu, net Earth
- removed copper zone on In2.Cu, net Earth
Other:
- copper layers 4 -> 6

Commit message: Schematic
Parts:
- moved C1101 4.12 mm to (155.3, 111.7)
- moved C1102 4.12 mm to (157.4, 111.7)
- moved C1103 4.12 mm to (164.5, 100.5)
- moved C1104 4.12 mm to (147.2, 96.8)
- moved C1105 4.12 mm to (156.1, 118.3)
- moved C1106 4.12 mm to (164.5, 109.7)
- moved C1108 4.12 mm to (149.4, 103.2)
- moved C1109 4.12 mm to (148.5, 118.3)
- moved C1110 4.12 mm to (152.2, 96.8)
- moved C1111 4.12 mm to (152.2, 118.3)
- moved C1112 4.12 mm to (143.1, 115.8)
- moved C1113 4.12 mm to (144.8, 115.8)
- moved C1114 4.12 mm to (143.1, 103.9)
- moved C1115 4.12 mm to (164.5, 104.7)
- moved C1116 4.12 mm to (160.9, 119.4)
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
Commit message: Schematic
Parts:
- moved U904 9.91 mm to (80.1, 122.2)
- moved U906 1.14 mm to (71.1, 122.2)

Commit message: Schematic
Parts:
- removed U901: NMK0509SC, ETH1CLCR2:NMK_DUAL
- removed U902: NMK2405SAC, ETH1CLCR2:NMK_SINGLE
- removed U904: NCP1117-5.0_SOT223, Package_TO_SOT_SMD:SOT-223-3_TabPin2
- removed U906: LT1175-5_SOT223, Package_TO_SOT_SMD:SOT-223-3_TabPin2
- added D501: 1N4148W, Diode_SMD:D_SOD-123, F.Cu at (100.2, 111.8)
- added Q501: BC847, Package_TO_SOT_SMD:SOT-23, F.Cu at (105.3, 112.4)
- added R509: 10k, Resistor_SMD:R_0603_1608Metric_Pad0.98x0.95mm_HandSolder, F.Cu at (109.7, 111.3)
- added U503: OP1177AR, Package_SO:SOIC-8_3.9x4.9mm_P1.27mm, F.Cu at (101.6, 106.9)
- added U505: OP1177AR, Package_SO:SOIC-8_3.9x4.9mm_P1.27mm, F.Cu at (110.0, 106.9)
- moved D802 6.02 mm to (164.8, 65.3), turned to 270 degrees
- moved R810 4.40 mm to (157.5, 65.3), turned to 90 degrees
- moved R808 2.25 mm to (147.3, 61.5)
- moved U802 2.25 mm to (147.3, 61.5)
- moved C809 2.25 mm to (144.9, 61.5)
- moved R813 1.77 mm to (136.3, 70.0)
- moved U803 1.77 mm to (138.3, 65.0)
- moved R807 1.77 mm to (136.3, 60.5)
- moved U812 1.77 mm to (129.5, 69.8)
- moved U804 1.77 mm to (122.4, 59.1)
- moved R812 1.77 mm to (140.3, 70.0)
- moved R806 1.77 mm to (140.3, 60.5)
- moved U806 1.77 mm to (129.4, 60.6)
- moved C810 1.66 mm to (144.8, 69.2)
- moved R824 1.66 mm to (147.3, 69.2)
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Connections:
- net /ADC/ADC_MISO renamed /ADC/ADC1_MISO
- net /ADC/ADC_MOSI renamed /ADC/ADC1_MOSI
- net /ADC/ADC_RVS1 renamed /ADC/ADC1_RVS1
- net /ADC/ADC_RVS2 renamed /ADC/ADC1_RVS2
- net /ADC/ADC_SCLK renamed /ADC/ADC1_SCLK
- net /ADC/ADC_~CS renamed /ADC/ADC1_~CS
- K801 pad 7: Net-(K801-Pad7) -> (no net)
- K801 pad 8: Net-(K801-Pad8) -> (no net)
- R503 pad 2: /ADC/ADC_IIN -> (no net)
- R506 pad 2: /ADC/ADC_VIN -> (no net)
- R808 pad 2: Net-(K801-Pad8) -> Net-(R808-Pad2)
- R824 pad 2: Net-(K801-Pad7) -> Net-(R824-Pad2)
- U1101 pad 73: (no net) -> /DDS/DDS_CS
- U1101 pad 74: (no net) -> /DDS/DDS_SCLK
- U1101 pad 76: (no net) -> /DDS/DDS_SDATA
- U1201 pad 10: AGNDF -> GND
- U1201 pad 11: AGNDF -> GND
- U1201 pad 12: AGNDF -> GND
- U1201 pad 13: (no net) -> /DDS/DDS_SDATA
- U1201 pad 14: (no net) -> /DDS/DDS_SCLK
- U1201 pad 15: (no net) -> /DDS/DDS_CS
- U1201 pad 17: AGNDF -> GND
- U1201 pad 18: AGNDF -> GND
- U1201 pad 4: +5VF -> +5VA
- U1201 pad 5: +5VF -> +3V3
- U1201 pad 7: AGNDF -> GND
- U1201 pad 9: AGNDF -> GND
- U802 pad 2: Net-(K801-Pad8) -> Net-(R808-Pad2)
- U808 pad 2: Net-(K801-Pad7) -> Net-(R824-Pad2)

Commit message: Footprints
Parts:
- removed J101: RF_Shield_One_Piece, ETH1CLCR2:36107406S
- removed U909: NCP1117-5.0_TO252, Package_TO_SOT_SMD:TO-252-2
- removed U910: NCP1117-5.0_SOT223, Package_TO_SOT_SMD:SOT-223-3_TabPin2
- removed U911: LT1175-5_SOT223, Package_TO_SOT_SMD:SOT-223-3_TabPin2
- added C1201: 4u7, Capacitor_SMD:C_0603_1608Metric_Pad1.08x0.95mm_HandSolder, F.Cu at (121.8, -73.2)
- added C1202: 100n, Capacitor_SMD:C_0603_1608Metric_Pad1.08x0.95mm_HandSolder, F.Cu at (107.8, -55.1)
- added C1203: 100p, Capacitor_SMD:C_0603_1608Metric_Pad1.08x0.95mm_HandSolder, F.Cu at (126.2, -73.2)
- added C1204: 4u7, Capacitor_SMD:C_0603_1608Metric_Pad1.08x0.95mm_HandSolder, F.Cu at (113.4, -67.6)
- added C1205: 68p, Capacitor_SMD:C_0603_1608Metric_Pad1.08x0.95mm_HandSolder, F.Cu at (112.0, -60.1)
- added C1206: 100p, Capacitor_SMD:C_0603_1608Metric_Pad1.08x0.95mm_HandSolder, F.Cu at (117.7, -66.0)
- added C1207: 4u7, Capacitor_SMD:C_0603_1608Metric_Pad1.08x0.95mm_HandSolder, F.Cu at (133.2, -80.7)
- added C1208: 3p3/COG, Capacitor_SMD:C_0603_1608Metric_Pad1.08x0.95mm_HandSolder, F.Cu at (117.7, -68.5)
- added C1209: 100n, Capacitor_SMD:C_0603_1608Metric_Pad1.08x0.95mm_HandSolder, F.Cu at (122.1, -65.6)
- added C1210: 100n, Capacitor_SMD:C_0603_1608Metric_Pad1.08x0.95mm_HandSolder, F.Cu at (103.4, -55.6)
- added C1211: 100n, Capacitor_SMD:C_0603_1608Metric_Pad1.08x0.95mm_HandSolder, F.Cu at (121.8, -75.7)
- added C1212: 100n, Capacitor_SMD:C_0603_1608Metric_Pad1.08x0.95mm_HandSolder, F.Cu at (124.5, -80.7)
- added C1213: 10n, Capacitor_SMD:C_0603_1608Metric_Pad1.08x0.95mm_HandSolder, F.Cu at (117.5, -76.0)
- added C1214: 100n, Capacitor_SMD:C_0603_1608Metric_Pad1.08x0.95mm_HandSolder, F.Cu at (102.2, -58.1)
- added C1215: 100n, Capacitor_SMD:C_0603_1608Metric_Pad1.08x0.95mm_HandSolder, F.Cu at (117.5, -73.5)
- added C1216: 100n, Capacitor_SMD:C_0603_1608Metric_Pad1.08x0.95mm_HandSolder, F.Cu at (109.0, -67.6)
- added C1217: 100n, Capacitor_SMD:C_0603_1608Metric_Pad1.08x0.95mm_HandSolder, F.Cu at (109.0, -65.1)
- added C1218: 100n, Capacitor_SMD:C_0603_1608Metric_Pad1.08x0.95mm_HandSolder, F.Cu at (99.1, -53.7)
- added C1219: 100n, Capacitor_SMD:C_0603_1608Metric_Pad1.08x0.95mm_HandSolder, F.Cu at (124.5, -78.2)
- added C1220: 100n, Capacitor_SMD:C_0603_1608Metric_Pad1.08x0.95mm_HandSolder, F.Cu at (120.7, -60.6)
- added C1221: 100n, Capacitor_SMD:C_0603_1608Metric_Pad1.08x0.95mm_HandSolder, F.Cu at (128.9, -80.7)
- added C1222: 100n, Capacitor_SMD:C_0603_1608Metric_Pad1.08x0.95mm_HandSolder, F.Cu at (107.6, -62.6)
- added C1223: 100n, Capacitor_SMD:C_0603_1608Metric_Pad1.08x0.95mm_HandSolder, F.Cu at (107.6, -60.1)
- added C1224: 100n, Capacitor_SMD:C_0603_1608Metric_Pad1.08x0.95mm_HandSolder, F.Cu at (116.5, -71.0)
- added C1225: 100n, Capacitor_SMD:C_0603_1608Metric_Pad1.08x0.95mm_HandSolder, F.Cu at (113.4, -65.1)
- added C1226: 100n, Capacitor_SMD:C_0603_1608Metric_Pad1.08x0.95mm_HandSolder, F.Cu at (112.1, -57.6)
- added C1227: 100n, Capacitor_SMD:C_0603_1608Metric_Pad1.08x0.95mm_HandSolder, F.Cu at (112.1, -52.6)
- added C1228: 100n, Capacitor_SMD:C_0603_1608Metric_Pad1.08x0.95mm_HandSolder, F.Cu at (130.8, -70.6)
- added C1229: 100n, Capacitor_SMD:C_0603_1608Metric_Pad1.08x0.95mm_HandSolder, F.Cu at (134.9, -73.2)
- added C1230: 100n, Capacitor_SMD:C_0603_1608Metric_Pad1.08x0.95mm_HandSolder, F.Cu at (116.5, -55.1)
- added C511: 10n, Capacitor_SMD:C_0603_1608Metric_Pad1.08x0.95mm_HandSolder, F.Cu at (118.1, -30.5)
- added C512: 1u, Capacitor_SMD:C_0603_1608Metric_Pad1.08x0.95mm_HandSolder, F.Cu at (121.2, -25.2)
- added C513: 47u, Capacitor_SMD:C_1206_3216Metric_Pad1.33x1.80mm_HandSolder, F.Cu at (115.8, -39.3)
- added C514: 470p/COG, Capacitor_SMD:C_0603_1608Metric_Pad1.08x0.95mm_HandSolder, F.Cu at (108.4, -22.4)
- added C515: 10u, Capacitor_SMD:C_1206_3216Metric_Pad1.33x1.80mm_HandSolder, F.Cu at (94.5, -20.6)
- added C516: 2700p/COG, Capacitor_SMD:C_0603_1608Metric_Pad1.08x0.95mm_HandSolder, F.Cu at (104.1, -19.7)
- added C517: 470p/COG, Capacitor_SMD:C_0603_1608Metric_Pad1.08x0.95mm_HandSolder, F.Cu at (112.5, -27.5)
- added C518: 10u, Capacitor_SMD:C_1206_3216Metric_Pad1.33x1.80mm_HandSolder, F.Cu at (103.0, -25.1)
- added C519: 10u, Capacitor_SMD:C_1206_3216Metric_Pad1.33x1.80mm_HandSolder, F.Cu at (124.2, -45.7)
- added C520: 470p/COG, Capacitor_SMD:C_0603_1608Metric_Pad1.08x0.95mm_HandSolder, F.Cu at (108.4, -19.9)
- added C521: 2700p/COG, Capacitor_SMD:C_0603_1608Metric_Pad1.08x0.95mm_HandSolder, F.Cu at (125.3, -40.3)
- added C522: 10u, Capacitor_SMD:C_1206_3216Metric_Pad1.33x1.80mm_HandSolder, F.Cu at (108.5, -31.6)
- added C523: 470p/COG, Capacitor_SMD:C_0603_1608Metric_Pad1.08x0.95mm_HandSolder, F.Cu at (120.7, -36.3)
- added C524: 100n, Capacitor_SMD:C_0603_1608Metric_Pad1.08x0.95mm_HandSolder, F.Cu at (108.2, -26.2)
- added C525: 100n, Capacitor_SMD:C_0603_1608Metric_Pad1.08x0.95mm_HandSolder, F.Cu at (104.1, -22.2)
- added C526: 100n, Capacitor_SMD:C_0603_1608Metric_Pad1.08x0.95mm_HandSolder, F.Cu at (129.4, -46.1)
- added C527: 100n, Capacitor_SMD:C_0603_1608Metric_Pad1.08x0.95mm_HandSolder, F.Cu at (120.9, -39.7)
- added C528: 100n, Capacitor_SMD:C_0603_1608Metric_Pad1.08x0.95mm_HandSolder, F.Cu at (123.4, -42.8)
- added C529: 100n, Capacitor_SMD:C_0603_1608Metric_Pad1.08x0.95mm_HandSolder, F.Cu at (99.7, -21.0)
- added C530: 100n, Capacitor_SMD:C_0603_1608Metric_Pad1.08x0.95mm_HandSolder, F.Cu at (112.5, -25.0)
- added C531: 100n, Capacitor_SMD:C_0603_1608Metric_Pad1.08x0.95mm_HandSolder, F.Cu at (125.3, -37.8)
- added C532: 100n, Capacitor_SMD:C_0603_1608Metric_Pad1.08x0.95mm_HandSolder, F.Cu at (133.7, -46.1)
- added C533: 100n, Capacitor_SMD:C_0603_1608Metric_Pad1.08x0.95mm_HandSolder, F.Cu at (118.1, -33.0)
- added C534: 100n, Capacitor_SMD:C_0603_1608Metric_Pad1.08x0.95mm_HandSolder, F.Cu at (94.7, -29.2)
- added C535: 100n, Capacitor_SMD:C_0603_1608Metric_Pad1.08x0.95mm_HandSolder, F.Cu at (129.4, -43.6)
- added C915: T521V107M016ATE050, Capacitor_Tantalum_SMD:CP_EIA-7343-20_Kemet-V_Pad2.25x2.55mm_HandSolder, F.Cu at (102.2, 21.5)
- added C920: T521V107M016ATE050, Capacitor_Tantalum_SMD:CP_EIA-7343-20_Kemet-V_Pad2.25x2.55mm_HandSolder, F.Cu at (102.2, 27.3)
- added C921: 4u7, Capacitor_SMD:C_1206_3216Metric_Pad1.33x1.80mm_HandSolder, F.Cu at (195.3, 113.4)
- added D1201: BYG20J, Diode_SMD:D_SMA, F.Cu at (113.5, -79.7)
- added D1202: BYG20J, Diode_SMD:D_SMA, F.Cu at (96.6, -61.8)
- added D1204: BZX584C5V6, Diode_SMD:D_SOD-523, F.Cu at (124.8, -55.6)
- added D1205: BZX584C5V6, Diode_SMD:D_SOD-523, F.Cu at (120.4, -53.1)
- added D1206: BZX584C5V6, Diode_SMD:D_SOD-523, F.Cu at (129.0, -60.6)
- added D1207: BZX584C5V6, Diode_SMD:D_SOD-523, F.Cu at (134.7, -65.7)
- added FB1201: BLM18SP601SZ1D, Inductor_SMD:L_0603_1608Metric_Pad1.05x0.95mm_HandSolder, F.Cu at (94.7, -53.7)
- added FB1202: BLM18SP601SZ1D, Inductor_SMD:L_0603_1608Metric_Pad1.05x0.95mm_HandSolder, F.Cu at (126.2, -75.7)
- added K501: TQ2SA-5V, ETH1CLCR2:SA, F.Cu at (122.7, 86.1)
- added L1201: CBMF1608T100K, Inductor_SMD:L_0603_1608Metric_Pad1.05x0.95mm_HandSolder, F.Cu at (79.7, 6.17)
- added L1202: CBMF1608T100K, Inductor_SMD:L_0603_1608Metric_Pad1.05x0.95mm_HandSolder, F.Cu at (84.2, 1.62)
- added L1203: CBMF1608T100K, Inductor_SMD:L_0603_1608Metric_Pad1.05x0.95mm_HandSolder, F.Cu at (84.2, 4.13)
- added L1204: CBMF1608T100K, Inductor_SMD:L_0603_1608Metric_Pad1.05x0.95mm_HandSolder, F.Cu at (88.5, 1.62)
- added L901: PM1608S-100M-RC, ETH1CLCR2:PM1608S, F.Cu at (196.1, 122.7)
- added Q1201: FDV301N, Package_TO_SOT_SMD:SOT-23, F.Cu at (79.8, 2.64)
- added R1201: 6k8, Resistor_SMD:R_0603_1608Metric_Pad0.98x0.95mm_HandSolder, F.Cu at (122.1, -70.6)
- added R1202: 2k, Resistor_SMD:R_0603_1608Metric_Pad0.98x0.95mm_HandSolder, F.Cu at (116.3, -62.6)
- added R1203: 200, Resistor_SMD:R_0603_1608Metric_Pad0.98x0.95mm_HandSolder, F.Cu at (103.4, -53.1)
- added R1204: 330, Resistor_SMD:R_0603_1608Metric_Pad0.98x0.95mm_HandSolder, F.Cu at (128.9, -78.2)
- added R1205: 200, Resistor_SMD:R_0603_1608Metric_Pad0.98x0.95mm_HandSolder, F.Cu at (112.0, -62.6)
- added R1206: 200, Resistor_SMD:R_0603_1608Metric_Pad0.98x0.95mm_HandSolder, F.Cu at (107.8, -57.6)
- added R1207: 820, Resistor_SMD:R_0603_1608Metric_Pad0.98x0.95mm_HandSolder, F.Cu at (116.3, -60.1)
- added R1208: 200, Resistor_SMD:R_0603_1608Metric_Pad0.98x0.95mm_HandSolder, F.Cu at (107.8, -52.6)
- added R1209: 100k, Resistor_SMD:R_0603_1608Metric_Pad0.98x0.95mm_HandSolder, F.Cu at (133.2, -78.2)
- added R1210: 220, Resistor_SMD:R_0603_1608Metric_Pad0.98x0.95mm_HandSolder, F.Cu at (112.1, -55.1)
- added R1211: 680, Resistor_SMD:R_0603_1608Metric_Pad0.98x0.95mm_HandSolder, F.Cu at (120.7, -63.1)
- added R1212: 220, Resistor_SMD:R_0603_1608Metric_Pad0.98x0.95mm_HandSolder, F.Cu at (137.6, -78.2)
- added R1213: 68, Resistor_SMD:R_0603_1608Metric_Pad0.98x0.95mm_HandSolder, F.Cu at (126.4, -68.1)
- added R1214: 33, Resistor_SMD:R_0603_1608Metric_Pad0.98x0.95mm_HandSolder, F.Cu at (134.9, -75.7)
- added R1215: 100, Resistor_SMD:R_0603_1608Metric_Pad0.98x0.95mm_HandSolder, F.Cu at (126.4, -65.6)
- added R1216: 200, Resistor_SMD:R_0603_1608Metric_Pad0.98x0.95mm_HandSolder, F.Cu at (125.0, -63.1)
- added R1217: 330, Resistor_SMD:R_0603_1608Metric_Pad0.98x0.95mm_HandSolder, F.Cu at (130.5, -75.7)
- added R1218: 330, Resistor_SMD:R_0603_1608Metric_Pad0.98x0.95mm_HandSolder, F.Cu at (120.8, -58.1)
- added R1219: 680, Resistor_SMD:R_0603_1608Metric_Pad0.98x0.95mm_HandSolder, F.Cu at (130.8, -65.6)
- added R1220: 680, Resistor_SMD:R_0603_1608Metric_Pad0.98x0.95mm_HandSolder, F.Cu at (116.5, -57.6)
- added R1221: 100, Resistor_SMD:R_0603_1608Metric_Pad0.98x0.95mm_HandSolder, F.Cu at (125.0, -60.6)
- added R1222: 100, Resistor_SMD:R_0603_1608Metric_Pad0.98x0.95mm_HandSolder, F.Cu at (116.5, -52.6)
- added R1223: 150, Resistor_SMD:R_0603_1608Metric_Pad0.98x0.95mm_HandSolder, F.Cu at (135.1, -70.6)
- added R1224: 150, Resistor_SMD:R_0603_1608Metric_Pad0.98x0.95mm_HandSolder, F.Cu at (120.8, -55.6)
- added R1225: 150, Resistor_SMD:R_0603_1608Metric_Pad0.98x0.95mm_HandSolder, F.Cu at (129.4, -63.1)
- added R1226: 1k, Resistor_SMD:R_0603_1608Metric_Pad0.98x0.95mm_HandSolder, F.Cu at (135.1, -68.1)
- added R1227: 68, Resistor_SMD:R_0603_1608Metric_Pad0.98x0.95mm_HandSolder, F.Cu at (125.2, -58.1)
- added R1228: 68, Resistor_SMD:R_0603_1608Metric_Pad0.98x0.95mm_HandSolder, F.Cu at (130.8, -68.1)
- added R1229: 100k, Resistor_SMD:R_0603_1608Metric_Pad0.98x0.95mm_HandSolder, F.Cu at (122.1, -68.1)
- added R1230: 4k7, Resistor_SMD:R_0603_1608Metric_Pad0.98x0.95mm_HandSolder, F.Cu at (130.5, -73.2)
- added R1231: 68, Resistor_SMD:R_0603_1608Metric_Pad0.98x0.95mm_HandSolder, F.Cu at (126.4, -70.6)
- added R510: 10k/.1%, Resistor_SMD:R_0603_1608Metric_Pad0.98x0.95mm_HandSolder, F.Cu at (129.6, -36.1)
- added R511: 300, Resistor_SMD:R_0603_1608Metric_Pad0.98x0.95mm_HandSolder, F.Cu at (121.2, -27.7)
- added R512: 10k/.1%, Resistor_SMD:R_0603_1608Metric_Pad0.98x0.95mm_HandSolder, F.Cu at (122.5, -30.2)
- added R513: 634, Resistor_SMD:R_0603_1608Metric_Pad0.98x0.95mm_HandSolder, F.Cu at (125.6, -27.7)
- added R514: 91, Resistor_SMD:R_0603_1608Metric_Pad0.98x0.95mm_HandSolder, F.Cu at (112.8, -19.9)
- added R515: 100k, Resistor_SMD:R_0603_1608Metric_Pad0.98x0.95mm_HandSolder, F.Cu at (112.8, -22.4)
- added R516: 10k, Resistor_SMD:R_0603_1608Metric_Pad0.98x0.95mm_HandSolder, F.Cu at (116.9, -25.0)
- added R517: 634, Resistor_SMD:R_0603_1608Metric_Pad0.98x0.95mm_HandSolder, F.Cu at (129.6, -38.6)
- added R518: 10k, Resistor_SMD:R_0603_1608Metric_Pad0.98x0.95mm_HandSolder, F.Cu at (125.0, -35.3)
- added R519: 91, Resistor_SMD:R_0603_1608Metric_Pad0.98x0.95mm_HandSolder, F.Cu at (133.7, -43.6)
- added R520: 91, Resistor_SMD:R_0603_1608Metric_Pad0.98x0.95mm_HandSolder, F.Cu at (129.6, -41.1)
- added R521: 100k, Resistor_SMD:R_0603_1608Metric_Pad0.98x0.95mm_HandSolder, F.Cu at (122.5, -32.8)
- added R522: 10k/.1%, Resistor_SMD:R_0603_1608Metric_Pad0.98x0.95mm_HandSolder, F.Cu at (134.0, -41.1)
- added R523: 300, Resistor_SMD:R_0603_1608Metric_Pad0.98x0.95mm_HandSolder, F.Cu at (121.5, -22.7)
- added R524: 100k, Resistor_SMD:R_0603_1608Metric_Pad0.98x0.95mm_HandSolder, F.Cu at (131.2, -33.6)
- added R525: 10k, Resistor_SMD:R_0603_1608Metric_Pad0.98x0.95mm_HandSolder, F.Cu at (134.0, -36.1)
- added R526: 10k/.1%, Resistor_SMD:R_0603_1608Metric_Pad0.98x0.95mm_HandSolder, F.Cu at (107.7, -28.7)
- added R527: 634, Resistor_SMD:R_0603_1608Metric_Pad0.98x0.95mm_HandSolder, F.Cu at (126.8, -30.2)
- added R528: 10k, Resistor_SMD:R_0603_1608Metric_Pad0.98x0.95mm_HandSolder, F.Cu at (117.1, -19.9)
- added R529: 91, Resistor_SMD:R_0603_1608Metric_Pad0.98x0.95mm_HandSolder, F.Cu at (126.8, -32.8)
- added R530: 100k, Resistor_SMD:R_0603_1608Metric_Pad0.98x0.95mm_HandSolder, F.Cu at (117.1, -22.4)
- added R531: 634, Resistor_SMD:R_0603_1608Metric_Pad0.98x0.95mm_HandSolder, F.Cu at (134.0, -38.6)
- added R830: 200/.1%, Resistor_SMD:R_0603_1608Metric_Pad0.98x0.95mm_HandSolder, F.Cu at (145.4, -80.7)
- added R831: 200/.1%, Resistor_SMD:R_0603_1608Metric_Pad0.98x0.95mm_HandSolder, F.Cu at (145.4, -78.2)
- added RV1201: 3314J-1-104E, Potentiometer_SMD:Potentiometer_Bourns_3314J_Vertical, F.Cu at (141.2, -88.4)
- added U1202: AD8038, Package_SO:SOIC-8_3.9x4.9mm_P1.27mm, F.Cu at (88.3, -55.8)
- added U1203: DAC7811, Package_SO:VSSOP-10_3x3mm_P0.5mm, F.Cu at (96.3, -57.2)
- added U1204: AD8038, Package_SO:SOIC-8_3.9x4.9mm_P1.27mm, F.Cu at (105.2, -78.7)
- added U1205: LMH6639, Package_SO:SOIC-8_3.9x4.9mm_P1.27mm, F.Cu at (96.8, -67.3)
- added U1206: LMH6639, Package_SO:SOIC-8_3.9x4.9mm_P1.27mm, F.Cu at (105.2, -72.3)
- added U1207: DG409, Package_SO:SOIC-16_3.9x9.9mm_P1.27mm, F.Cu at (88.3, -76.2)
- added U1208: 74AHC1G14, Package_TO_SOT_SMD:SOT-353_SC-70-5_Handsoldering, F.Cu at (103.9, -67.1)
- added U1210: 74AUP1G79, Package_TO_SOT_SMD:SOT-353_SC-70-5_Handsoldering, F.Cu at (112.4, -75.5)
- added U1211: 74AC161, Package_SO:SOIC-16_3.9x9.9mm_P1.27mm, F.Cu at (88.3, -64.8)
- added U1212: 74AC161, Package_SO:SOIC-16_3.9x9.9mm_P1.27mm, F.Cu at (96.8, -76.2)
- added U1213: SN74LVC1T45DBV, Package_TO_SOT_SMD:SOT-23-6, F.Cu at (111.9, -71.2)
- added U1214: SN74LVC1T45DBV, Package_TO_SOT_SMD:SOT-23-6, F.Cu at (103.0, -61.7)
- added U1215: SN74LVC1T45DBV, Package_TO_SOT_SMD:SOT-23-6, F.Cu at (119.9, -79.6)
- added U504: CS5361, Package_SO:SOIC-24W_7.5x15.4mm_P1.27mm, F.Cu at (159.1, 87.0)
- added U506: AD8656, Package_SO:SOIC-8_3.9x4.9mm_P1.27mm, F.Cu at (148.1, 81.8)
- added U507: AD8656, Package_SO:SOIC-8_3.9x4.9mm_P1.27mm, F.Cu at (101.2, -30.1)
- added U508: OP1177AR, Package_SO:SOIC-8_3.9x4.9mm_P1.27mm, F.Cu at (117.0, -44.2)
- added U509: AD8476_MSOP, Package_SO:MSOP-8_3x3mm_P0.65mm, F.Cu at (96.3, -24.6)
- added U901: NCS3S1205SC, ETH1CLCR2:NCS3, F.Cu at (181.6, 117.0)
- added U902: TLV1117-33, Package_TO_SOT_SMD:TO-263-3_TabPin2, F.Cu at (154.2, 130.8)
- added U904: TLV1117-50, Package_TO_SOT_SMD:TO-263-3_TabPin2, F.Cu at (127.9, 130.8)
- added U906: TLV1117-50, Package_TO_SOT_SMD:TO-263-3_TabPin2, F.Cu at (79.9, 130.8)
- added X1201: 830208220601, ETH1CLCR2:IQXO-791, F.Cu at (123.8, 20.2)
- R509: value 10k -> 10K
- RV1001, RV801: value TS53YJ203MR10 -> 3314J-1-203E; footprint Potentiometer_SMD:Potentiometer_Vishay_TS53YJ_Vertical -> Potentiometer_SMD:Potentiometer_Bourns_3314J_Vertical
- U505: value OP1177AR -> AD8476_MSOP; footprint Package_SO:SOIC-8_3.9x4.9mm_P1.27mm -> Package_SO:MSOP-8_3x3mm_P0.65mm
- U908: value NCP1117-3.3_TO252 -> LM2990SX-5.0; footprint Package_TO_SOT_SMD:TO-252-2 -> Package_TO_SOT_SMD:TO-263-3_TabPin2
- moved D801 154.5 mm to (175.8, 62.7), turned to 90 degrees
- moved D501 148.5 mm to (115.6, -35.9)
- moved Q501 143.6 mm to (113.7, -31.0)
- moved R509 139.0 mm to (116.9, -27.5)
- moved U505 130.5 mm to (87.8, -21.7)
- moved U908 60.0 mm to (103.3, 130.8)
- moved J1101 6.27 mm to (138.6, 100.9), turned to 180 degrees
- moved J1102 4.07 mm to (138.1, 114.6)
- moved R1106 4.07 mm to (138.6, 105.7)
- moved D1101 4.07 mm to (138.7, 108.6)
- moved D1102 4.07 mm to (138.7, 111.3)
- moved U905 3.96 mm to (180.2, 127.4)
- moved K601 3.95 mm to (156.7, 49.9), turned to 180 degrees
- moved U907 3.94 mm to (180.2, 136.1)
- moved C801 3.56 mm to (180.5, 60.1)
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Connections:
- K401 pad 1: (no net) -> /Connector/H_CUR
- K801 pad 7: (no net) -> Net-(K801-Pad7)
- K801 pad 8: (no net) -> Net-(K801-Pad8)
- R503 pad 2: (no net) -> /ADC/ADC1_IIN
- R506 pad 2: (no net) -> /ADC/ADC1_VIN
- R509 pad 1: Net-(Q501-Pad1) -> (no net)
- R509 pad 2: (no net) -> Net-(Q501-Pad1)
- U1101 pad 123: (no net) -> /DDS/MDAC_SDIN
- U1101 pad 40: (no net) -> /DDS/MDAC_CS
- U1101 pad 41: (no net) -> /DDS/MDAC_SCK
- U1101 pad 42: (no net) -> /DDS/MDAC_SDO
- U1201 pad 1: (no net) -> Net-(R1202-Pad2)
- U1201 pad 19: (no net) -> Net-(C1203-Pad2)
- U1201 pad 2: (no net) -> Net-(C1204-Pad2)
- U1201 pad 20: (no net) -> Net-(C1203-Pad1)
- U1201 pad 3: (no net) -> Net-(C1202-Pad2)
- U1201 pad 6: (no net) -> Net-(C1201-Pad1)
- U1201 pad 8: (no net) -> /DDS/MCLK
- U503 pad 2: (no net) -> Net-(C515-Pad2)
- U503 pad 3: (no net) -> Net-(R511-Pad1)
- U503 pad 4: (no net) -> -5VA
- U503 pad 6: (no net) -> Net-(U503-Pad6)
- U503 pad 7: (no net) -> +5VA
- U505 pad 1: (no net) -> GND
- U505 pad 2: (no net) -> +5VA
- U505 pad 3: (no net) -> GND
- U505 pad 4: (no net) -> Net-(C515-Pad2)
- U505 pad 5: (no net) -> Net-(C518-Pad2)
- U505 pad 7: (no net) -> -5VA
- U505 pad 8: (no net) -> Net-(U503-Pad6)
- U908 pad 1: GND -> GNDA
- U908 pad 2: +3V3 -> Net-(C916-Pad2)
- U908 pad 3: Net-(C901-Pad1) -> -5VA
Routing:
- net Net-(D902-Pad1): track 18.0 -> 11.5 mm, vias 7 -> 4
- net Net-(L901-Pad2): track 0.00 -> 4.13 mm, vias 0 -> 3
- net GNDPWR: track 8.70 -> 12.3 mm, vias 7 -> 10
- net Net-(Q901-Pad1): track 5.61 -> 7.29 mm
- added copper zone on B.Cu, net Net-(L901-Pad2)
- added copper zone on F.Cu, net Net-(L901-Pad2)
- removed copper zone on F.Cu, net Net-(Q901-Pad1)
