File: hardware/ETH1CLCR2/Trigger.sch (KiCad schematic (older format))
At the start: 22 parts, among them U401 74AC125, U402 TXB0104PW, U403 ADuM5402

Commit message: Footprints assigned.
Parts:
- renumbered C401 to C301, C402 to C302, C403 to C303, C404 to C304, C405 to C305, C406 to C306, C407 to C307, C408 to C308, C409 to C309, D401 to D301, D402 to D302, D403 to D303, L401 to L301, R401 to R301, R402 to R302, R403 to R303, R404 to R304, R405 to R305, R406 to R306, U401 to U301, U402 to U302, U403 to U303
