File: hardware/ETH1CLCR2/ADC.sch (KiCad schematic (older format))
At the start: 20 parts, among them U501 ADS8681PWR, U502 ADS8681PWR

Commit message: Schematic
Parts:
- added C511: 10n, Capacitor_SMD:C_0603_1608Metric_Pad1.08x0.95mm_HandSolder, symbol Device:C
- added C512: 1u, Capacitor_SMD:C_0603_1608Metric_Pad1.08x0.95mm_HandSolder, symbol Device:C
- added C513: 47u, Capacitor_SMD:C_1206_3216Metric_Pad1.33x1.80mm_HandSolder, symbol Device:C
- added C514, C517, C520, C523: 470p/COG, Capacitor_SMD:C_0603_1608Metric_Pad1.08x0.95mm_HandSolder, symbol Device:C
- added C515, C518, C519, C522: 10u, Capacitor_SMD:C_1206_3216Metric_Pad1.33x1.80mm_HandSolder, symbol Device:C
- added C516, C521: 2700p/COG, Capacitor_SMD:C_0603_1608Metric_Pad1.08x0.95mm_HandSolder, symbol Device:C
- added C524, C525, C526, C527, C528, C529, C530, C531, C532, C533, C534, C535: 100n, Capacitor_SMD:C_0603_1608Metric_Pad1.08x0.95mm_HandSolder, symbol Device:C
- added D501: 1N4148W, Diode_SMD:D_SOD-123, symbol Device:D
- added K501: TQ2SA-5V, ETH1CLCR2:SA, symbol ETH1CLCR2:TQ2SA-5V
- added Q501: BC847, Package_TO_SOT_SMD:SOT-23, symbol Transistor_BJT:BC847
- added R509: 10K, Resistor_SMD:R_0603_1608Metric_Pad0.98x0.95mm_HandSolder, symbol Device:R
- added R510, R512, R522, R526: 10k/.1%, Resistor_SMD:R_0603_1608Metric_Pad0.98x0.95mm_HandSolder, symbol Device:R
- added R511, R523: 300, Resistor_SMD:R_0603_1608Metric_Pad0.98x0.95mm_HandSolder, symbol Device:R
- added R513, R517, R527, R531: 634, Resistor_SMD:R_0603_1608Metric_Pad0.98x0.95mm_HandSolder, symbol Device:R
- added R514, R519, R520, R529: 91, Resistor_SMD:R_0603_1608Metric_Pad0.98x0.95mm_HandSolder, symbol Device:R
- added R515, R521, R524, R530: 100k, Resistor_SMD:R_0603_1608Metric_Pad0.98x0.95mm_HandSolder, symbol Device:R
- added R516, R518, R525, R528: 10k, Resistor_SMD:R_0603_1608Metric_Pad0.98x0.95mm_HandSolder, symbol Device:R
- added U503, U508: OP1177AR, Package_SO:SOIC-8_3.9x4.9mm_P1.27mm, symbol Amplifier_Operational:OP1177AR
- added U504: CS5361, Package_SO:SOIC-24W_7.5x15.4mm_P1.27mm, symbol Audio:CS5361
- added U505, U509: AD8476_MSOP, Package_SO:MSOP-8_3x3mm_P0.65mm, symbol ETH1CLCR2:AD8476_MSOP
- added U506, U507: AD8656, Package_SO:SOIC-8_3.9x4.9mm_P1.27mm, symbol ETH1CLCR2:AD8656
Connections:
- net +3V3: now also U504.12 (I2S/~LJ), U504.2 (M/~S), U504.6 (VD), U504.8 (VL)
- net +5V: now also D501.1 (K), K501.1, U504.19 (VA)
- net ADC_IIN: now also K501.3; no longer R503.2
- net ADC_VIN: now also K501.8; no longer R506.2
- net GND: now also C511.2, C512.2, C513.2, C524.2, C525.2, C526.2, C527.2, C528.2, C529.2, C530.2, C531.2, C532.2, C533.2, C534.2, C535.2, Q501.2 (E), R512.1, R515.2, R521.2, R524.2, R526.1, R530.2, U504.18 (GND), U504.23 (REFGND), U504.7 (GND), U505.1 (-IN), U505.3 (VCOM), U506.4 (V-), U507.4 (V-), U509.1 (-IN), U509.3 (VCOM)
- net ADC_MISO renamed ADC1_MISO
- net ADC_MOSI renamed ADC1_MOSI
- net ADC_RVS1 renamed ADC1_RVS1
- net ADC_RVS2 renamed ADC1_RVS2
- net ADC_SCLK renamed ADC1_SCLK
- net ADC_~CS renamed ADC1_~CS
- new net: C516.1, R513.1, R514.1, U504.16 (AINL+)
- new net: C516.2, R519.1, R527.1, U504.17 (AINL-)
- new net: C521.2, R529.1, R531.1, U504.20 (AINR-)
- new net: C521.1, R517.1, R520.1, U504.21 (AINR+)
- new net: C513.1, U504.24 (FILT+)
- new net: C515.2, R515.1, U503.2 (-), U505.4 (+OUT)
- new net: R511.1, U503.3 (+)
- new net: U503.6, U505.8 (+IN)
- new net: D501.2 (A), K501.10, Q501.3 (C)
- new net: R510.1, R511.2, R512.2
- new net: C518.2, R521.1, U505.5 (-OUT)
- new net: C514.1, R514.2, U506.1
- new net: C514.2, R513.2, U506.2 (-)
- new net: C515.1, R516.1, U506.3 (+)
- new net: C518.1, R518.1, U506.5 (+)
- new net: C520.2, R527.2, U506.6 (-)
- new net: C520.1, R519.2, U506.7
- new net: C519.2, R524.1, U508.2 (-), U509.4 (+OUT)
- new net: R523.1, U508.3 (+)
- new net: U508.6, U509.8 (+IN)
- new net: R522.1, R523.2, R526.2
- new net: C522.2, R530.1, U509.5 (-OUT)
- new net: C517.1, R520.2, U507.1
- new net: C517.2, R517.2, U507.2 (-)
- new net: C519.1, R525.1, U507.3 (+)
- new net: C522.1, R528.1, U507.5 (+)
- new net: C523.1, R529.2, U507.7
- new net: C523.2, R531.2, U507.6 (-)
- new net: Q501.1 (B), R509.2
- new net +5VA: C524.1, C525.1, C526.1, C527.1, C528.1, C529.1, U503.7 (V+), U505.2 (+Vs), U506.8 (V+), U507.8 (V+), U508.7 (V+), U509.2 (+Vs)
- new net -5VA: C530.1, C531.1, C532.1, C533.1, C534.1, C535.1, U503.4 (V-), U505.7 (-Vs), U508.4 (V-), U509.7 (-Vs)
- new net ADC1_IIN: K501.2, R503.2
- new net ADC1_VIN: K501.9, R506.2
- new net ADC2_IIN: K501.4, R510.2
- new net ADC2_LRCK: U504.3 (LRCK)
- new net ADC2_M0: U504.13 (M0)
- new net ADC2_M1: U504.14 (M1)
- new net ADC2_MDIV: U504.10 (MDIV)
- new net ADC2_SCLK: U504.4 (SCLK)
- new net ADC2_SDOUT: U504.9 (SDOUT)
- new net ADC2_VIN: K501.7, R522.2
- new net ADC_SEL: R509.1
- new net DDS_CLK: U504.5 (MCLK)
- new net VQ: C511.1, C512.1, R516.2, R518.2, R525.2, R528.2, U504.22 (VQ)
- new net ~ADC2_HPF: U504.11 (~HPF)
- new net ~ADC2_RST: U504.1 (~RST)
- no-connect marks 2 -> 3
Other:
- moved on the sheet: C501, C502, C503, C504, C505, C506, C507, C508, C509, C510, R501, R502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

Commit message: PCB
Parts:
- removed C532, C534: 100n, Capacitor_SMD:C_0603_1608Metric_Pad1.08x0.95mm_HandSolder, symbol Device:C
- renumbered C514 to C501, C501 to C502, C515 to C503, C516 to C504, C518 to C505, C520 to C506, C502 to C507, C517 to C508, C511 to C509, C512 to C510, C513 to C511, C519 to C512, C503 to C513, C504 to C514, C505 to C515, C506 to C516, C521 to C517, C522 to C518, C523 to C519, C507 to C520, C508 to C521, C509 to C522, C510 to C523, C533 to C532, C535 to C533, R513 to R501, R501 to R502, R502 to R503, R503 to R504, R514 to R505, R510 to R506, R511 to R507, R515 to R508, R516 to R509, R512 to R510, R518 to R511, R504 to R512, R505 to R513, R519 to R514, R521 to R515, R506 to R516, R527 to R517, R517 to R518, R520 to R519, R507 to R520, R508 to R521, R528 to R527, R529 to R528, R530 to R529, R531 to R530, R509 to R531, U506 to U502, U505 to U504, U502 to U505, U504 to U506
Other:
- moved on the sheet: C532, C533
