File: hardware/ETH1CLCR2/ADC.sch (KiCad schematic (older format))
At the start: 86 parts, among them K501 TQ2SA-5V, Q501 BC847, U501 ADS8681IPWR, U502 AD8656, U503 OP1177AR, U504 AD8476_MSOP, U505 ADS8681IPWR, U506 CS5361, U507 AD8656, U508 OP1177AR, U509 AD8476_MSOP

Commit message: BOM
Parts:
- R531: value 10K -> 10k
Changed lines of the file:
@@
 P 9950 9800
 F 0 "R531" V 9743 9800 50  0000 C CNN
-F 1 "10K" V 9834 9800 50  0000 C CNN
+F 1 "10k" V 9834 9800 50  0000 C CNN
 F 2 "Resistor_SMD:R_0603_1608Metric_Pad0.98x0.95mm_HandSolder" V 9880 9800 50  0001 C CNN
 F 3 "~" H 9950 9800 50  0001 C CNN
