File: hardware/ETH1CLCR2/Power.sch (KiCad schematic (older format))
At the start: 38 parts, among them Q901 IRFR5410, U901 NCS3S1205SC, U902 TLV1117-33, U903 MAX5902, U904 TLV1117-50, U905 NMK2409SAC, U906 TLV1117-50, U907 NMK2409SC, U908 LM2990SX-5.0

Commit message: PCB
Parts:
- TP901: footprint TestPoint:TestPoint_Plated_Hole_D2.0mm -> TestPoint:TestPoint_Loop_D2.60mm_Drill1.6mm_Beaded
- renumbered C921 to C901, C901 to C902, C902 to C903, C903 to C904, C904 to C905, C905 to C906, C906 to C907, C907 to C908, C908 to C909, C909 to C910, C910 to C911, C911 to C912, C912 to C913, C913 to C914, C914 to C915, C915 to C916, C916 to C917, C917 to C918, C918 to C919, C919 to C920, C920 to C921, U902 to U901, U901 to U902
Connections:
- net GNDA is gone; now on net GND: C912.2, C913.2, C914.2, C915.2, C916.2, C917.1, C918.1, C919.1, C920.1, C921.1, U906.1 (GND), U907.6 (GND), U908.1 (GND)
Changed lines of the file:
@@
 $EndComp
 $Comp
-L Device:C C901
+L Device:C C902
 U 1 1 609E5909
 P 8300 3250
-F 0 "C901" H 8415 3296 50  0000 L CNN
+F 0 "C902" H 8415 3296 50  0000 L CNN
 F 1 "10u" H 8415 3205 50  0000 L CNN
 F 2 "Capacitor_SMD:C_1206_3216Metric_Pad1.33x1.80mm_HandSolder" H 8338 3100 50  0001 C CNN
@@
 Connection ~ 8300 3450
 $Comp
-L Device:C C902
+L Device:C C903
 U 1 1 609EC1FE
 P 9550 3250
-F 0 "C902" H 9665 3296 50  0000 L CNN
+F 0 "C903" H 9665 3296 50  0000 L CNN
 F 1 "10u" H 9665 3205 50  0000 L CNN
 F 2 "Capacitor_SMD:C_1206_3216Metric_Pad1.33x1.80mm_HandSolder" H 9588 3100 50  0001 C CNN
@@
 Connection ~ 9550 3050
 $Comp
-L Device:C C907
+L Device:C C908
 U 1 1 609FCF54
 P 7800 4350
-F 0 "C907" H 7915 4396 50  0000 L CNN
+F 0 "C908" H 7915 4396 50  0000 L CNN
 F 1 "10u" H 7915 4305 50  0000 L CNN
 F 2 "Capacitor_SMD:C_1206_3216Metric_Pad1.33x1.80mm_HandSolder" H 7838 4200 50  0001 C CNN
@@
 Connection ~ 7800 4550
 $Comp
-L Device:C C908
+L Device:C C909
 U 1 1 609FCF61
 P 9050 4350
-F 0 "C908" H 9165 4396 50  0000 L CNN
+F 0 "C909" H 9165 4396 50  0000 L CNN
 F 1 "10u" H 9165 4305 50  0000 L CNN
 F 2 "Capacitor_SMD:C_1206_3216Metric_Pad1.33x1.80mm_HandSolder" H 9088 4200 50  0001 C CNN
@@
 	7550 4550 7800 4550
 $Comp
-L Device:C C909
+L Device:C C910
 U 1 1 60F841C5
 P 9600 4350
-F 0 "C909" H 9715 4396 50  0000 L CNN
+F 0 "C910" H 9715 4396 50  0000 L CNN
 F 1 "1u" H 9715 4305 50  0000 L CNN
 F 2 "Capacitor_SMD:C_1206_3216Metric_Pad1.33x1.80mm_HandSolder" H 9638 4200 50  0001 C CNN
@@
 $EndComp
 $Comp
-L Device:C C910
+L Device:C C911
 U 1 1 60F841CB
 P 10100 4350
-F 0 "C910" H 10215 4396 50  0000 L CNN
+F 0 "C911" H 10215 4396 50  0000 L CNN
 F 1 "100n" H 10215 4305 50  0000 L CNN
 F 2 "Capacitor_SMD:C_1206_3216Metric_Pad1.33x1.80mm_HandSolder" H 10138 4200 50  0001 C CNN
@@
 $EndComp
 $Comp
-L Device:C C903
+L Device:C C904
 U 1 1 60F8D591
 P 10100 3250
-F 0 "C903" H 10215 3296 50  0000 L CNN
+F 0 "C904" H 10215 3296 50  0000 L CNN
 F 1 "1u" H 10215 3205 50  0000 L CNN
 F 2 "Capacitor_SMD:C_1206_3216Metric_Pad1.33x1.80mm_HandSolder" H 10138 3100 50  0001 C CNN
@@
 $EndComp
 $Comp
-L Device:C C904
+L Device:C C905
 U 1 1 60F8D597
 P 10600 3250
-F 0 "C904" H 10715 3296 50  0000 L CNN
+F 0 "C905" H 10715 3296 50  0000 L CNN
 F 1 "100n" H 10715 3205 50  0000 L CNN
 F 2 "Capacitor_SMD:C_1206_3216Metric_Pad1.33x1.80mm_HandSolder" H 10638 3100 50  0001 C CNN
@@
 F 0 "TP901" H 8992 4626 50  0000 R CNN
 F 1 "TestPoint" H 8992 4717 50  0000 R CNN
-F 2 "TestPoint:TestPoint_Plated_Hole_D2.0mm" H 9250 4600 50  0001 C CNN
+F 2 "TestPoint:TestPoint_Loop_D2.60mm_Drill1.6mm_Beaded" H 9250 4600 50  0001 C CNN
 F 3 "~" H 9250 4600 50  0001 C CNN
 	1    9050 4600
@@
 	9050 4600 9050 4550
 $Comp
-L Device:C C905
+L Device:C C906
 U 1 1 611D1D2A
 P 5050 3550
-F 0 "C905" H 5165 3596 50  0000 L CNN
+F 0 "C906" H 5165 3596 50  0000 L CNN
 F 1 "4u7/50V" H 5165 3505 50  0000 L CNN
 F 2 "Capacitor_SMD:C_1206_3216Metric_Pad1.33x1.80mm_HandSolder" H 5088 3400 50  0001 C CNN
@@
 Connection ~ 4300 4100
 $Comp
-L Device:C C906
+L Device:C C907
 U 1 1 611DDF1B
 P 5650 3550
-F 0 "C906" H 5765 3596 50  0000 L CNN
+F 0 "C907" H 5765 3596 50  0000 L CNN
 F 1 "4u7/50V" H 5765 3505 50  0000 L CNN
 F 2 "Capacitor_SMD:C_1206_3216Metric_Pad1.33x1.80mm_HandSolder" H 5688 3400 50  0001 C CNN
@@
 	8300 3050 8700 3050
 $Comp
-L ETH1CLCR2:NCS3 U901
+L ETH1CLCR2:NCS3 U902
 U 1 1 60B9EE6D
 P 7600 3250
-F 0 "U901" H 7600 3715 50  0000 C CNN
+F 0 "U902" H 7600 3715 50  0000 C CNN
 F 1 "NCS3S1205SC" H 7600 3624 50  0000 C CNN
 F 2 "ETH1CLCR2:NCS3" H 7600 3250 50  0001 C CNN
@@
 	6900 3050 7150 3050
 $Comp
-L Device:C C921
+L Device:C C901
 U 1 1 60BCC6E4
 P 6400 3250
-F 0 "C921" H 6515 3296 50  0000 L CNN
+F 0 "C901" H 6515 3296 50  0000 L CNN
 F 1 "4u7" H 6515 3205 50  0000 L CNN
 F 2 "Capacitor_SMD:C_1206_3216Metric_Pad1.33x1.80mm_HandSolder" H 6438 3100 50  0001 C CNN
@@
 	6400 3450 7150 3450
 $Comp
-L Regulator_Linear:TLV1117-33 U902
+L Regulator_Linear:TLV1117-33 U901
 U 1 1 611EE804
 P 9000 3050
-F 0 "U902" H 9000 3292 50  0000 C CNN
+F 0 "U901" H 9000 3292 50  0000 C CNN
 F 1 "TLV1117-33" H 9000 3201 50  0000 C CNN
 F 2 "Package_TO_SOT_SMD:TO-263-3_TabPin2" H 9000 3050 50  0001 C CNN
@@
 $EndComp
 $Comp
-L power:GNDA #PWR0919
+L power:GNDA #PWR0910
 U 1 1 60F40D30
 P 10350 5650
-F 0 "#PWR0919" H 10350 5400 50  0001 C CNN
+F 0 "#PWR0910" H 10350 5400 50  0001 C CNN
 F 1 "GNDA" V 10355 5522 50  0000 R CNN
 F 2 "" H 10350 5650 50  0001 C CNN
@@
 	9650 6000 10150 6000
 $Comp
-L Device:CP C920
+L Device:CP C921
 U 1 1 6094BAF0
 P 10150 5850
-F 0 "C920" H 10268 5896 50  0000 L CNN
+F 0 "C921" H 10268 5896 50  0000 L CNN
 F 1 "T521V107M016ATE050" H 10268 5805 50  0000 L CNN
 F 2 "Capacitor_Tantalum_SMD:CP_EIA-7343-20_Kemet-V_Pad2.25x2.55mm_HandSolder" H 10188 5700 50  0001 C CNN
@@
 	10150 5650 10150 5600
 $Comp
-L Device:CP C915
+L Device:CP C916
 U 1 1 6093A953
 P 10150 5450
-F 0 "C915" H 10268 5496 50  0000 L CNN
+F 0 "C916" H 10268 5496 50  0000 L CNN
 F 1 "T521V107M016ATE050" H 10268 5405 50  0000 L CNN
 F 2 "Capacitor_Tantalum_SMD:CP_EIA-7343-20_Kemet-V_Pad2.25x2.55mm_HandSolder" H 10188 5300 50  0001 C CNN
@@
 	8600 6000 9150 6000
 $Comp
-L Device:C C914
+L Device:C C915
 U 1 1 60F50B6C
 P 9650 5450
-F 0 "C914" H 9765 5496 50  0000 L CNN
+F 0 "C915" H 9765 5496 50  0000 L CNN
 F 1 "100n" H 9765 5405 50  0000 L CNN
 F 2 "Capacitor_SMD:C_1206_3216Metric_Pad1.33x1.80mm_HandSolder" H 9688 5300 50  0001 C CNN
@@
 $EndComp
 $Comp
-L Device:C C919
+L Device:C C920
 U 1 1 60F4EDE5
 P 9650 5850
-F 0 "C919" H 9765 5896 50  0000 L CNN
+F 0 "C920" H 9765 5896 50  0000 L CNN
 F 1 "100n" H 9765 5805 50  0000 L CNN
 F 2 "Capacitor_SMD:C_1206_3216Metric_Pad1.33x1.80mm_HandSolder" H 9688 5700 50  0001 C CNN
@@
 $EndComp
 $Comp
-L Device:C C918
+L Device:C C919
 U 1 1 60F4D101
 P 9150 5850
-F 0 "C918" H 9265 5896 50  0000 L CNN
+F 0 "C919" H 9265 5896 50  0000 L CNN
 F 1 "1u" H 9265 5805 50  0000 L CNN
 F 2 "Capacitor_SMD:C_1206_3216Metric_Pad1.33x1.80mm_HandSolder" H 9188 5700 50  0001 C CNN
@@
 $EndComp
 $Comp
-L Device:C C913
+L Device:C C914
 U 1 1 60F4B484
 P 9150 5450
-F 0 "C913" H 9265 5496 50  0000 L CNN
+F 0 "C914" H 9265 5496 50  0000 L CNN
 F 1 "1u" H 9265 5405 50  0000 L CNN
 F 2 "Capacitor_SMD:C_1206_3216Metric_Pad1.33x1.80mm_HandSolder" H 9188 5300 50  0001 C CNN
@@
 	7200 6000 7200 5850
 $Comp
-L Device:C C917
+L Device:C C918
 U 1 1 60A76326
 P 8600 5850
-F 0 "C917" H 8715 5896 50  0000 L CNN
+F 0 "C918" H 8715 5896 50  0000 L CNN
 F 1 "10u" H 8715 5805 50  0000 L CNN
 F 2 "Capacitor_SMD:C_1206_3216Metric_Pad1.33x1.80mm_HandSolder" H 8638 5700 50  0001 C CNN
@@
 $EndComp
 $Comp
-L Device:C C916
+L Device:C C917
 U 1 1 60A75F4C
 P 7350 5850
-F 0 "C916" H 7465 5896 50  0000 L CNN
+F 0 "C917" H 7465 5896 50  0000 L CNN
 F 1 "10u" H 7465 5805 50  0000 L CNN
 F 2 "Capacitor_SMD:C_1206_3216Metric_Pad1.33x1.80mm_HandSolder" H 7388 5700 50  0001 C CNN
@@
 	7150 5650 7350 5650
 $Comp
-L Device:C C912
+L Device:C C913
 U 1 1 60A6A7BE
 P 8600 5450
-F 0 "C912" H 8715 5496 50  0000 L CNN
+F 0 "C913" H 8715 5496 50  0000 L CNN
 F 1 "10u" H 8715 5405 50  0000 L CNN
 F 2 "Capacitor_SMD:C_1206_3216Metric_Pad1.33x1.80mm_HandSolder" H 8638 5300 50  0001 C CNN
@@
 $EndComp
 $Comp
-L Device:C C911
+L Device:C C912
 U 1 1 60A6652D
 P 7350 5450
-F 0 "C911" H 7465 5496 50  0000 L CNN
+F 0 "C912" H 7465 5496 50  0000 L CNN
 F 1 "10u" H 7465 5405 50  0000 L CNN
 F 2 "Capacitor_SMD:C_1206_3216Metric_Pad1.33x1.80mm_HandSolder" H 7388 5300 50  0001 C CNN
@@
 Wire Wire Line
 	6250 5450 6200 5450
+$Comp
+L power:GNDA #PWR0915
+U 1 1 60CF2DB9
+P 1800 7200
+F 0 "#PWR0915" H 1800 6950 50  0001 C CNN
+F 1 "GNDA" H 1805 7027 50  0000 C CNN
+F 2 "" H 1800 7200 50  0001 C CNN
+F 3 "" H 1800 7200 50  0001 C CNN
+	1    1800 7200
+	1    0    0    -1
+$EndComp
+$Comp
+L power:GND #PWR0916
+U 1 1 60CF31AD
+P 2100 7200
+F 0 "#PWR0916" H 2100 6950 50  0001 C CNN
+F 1 "GND" H 2105 7027 50  0000 C CNN
+F 2 "" H 2100 7200 50  0001 C CNN
+F 3 "" H 2100 7200 50  0001 C CNN
+	1    2100 7200
+	1    0    0    -1
+$EndComp
+Wire Wire Line
+	2100 7200 2100 7150
+Wire Wire Line
+	2100 7150 1800 7150
+Wire Wire Line
+	1800 7150 1800 7200
 $EndSCHEMATC
