File: hardware/ETH1CLCR2/Power.sch (KiCad schematic (older format))
At the start: 38 parts, among them Q901 IRFR5410, U901 LM1117SX-3.3/NOPB, U902 NCS3S1205SC, U903 MAX5902, U904 LM1117SX-5.0/NOPB, U905 NMK2409SAC, U906 LM1117SX-5.0/NOPB, U907 NMK2409SC, U908 LM2990SX-5.0

Commit message: BOM
Parts:
- C901: value 4u7 -> 4u7/50V
Changed lines of the file:
@@
 P 6400 3250
 F 0 "C901" H 6515 3296 50  0000 L CNN
-F 1 "4u7" H 6515 3205 50  0000 L CNN
+F 1 "4u7/50V" H 6515 3205 50  0000 L CNN
 F 2 "Capacitor_SMD:C_1206_3216Metric_Pad1.33x1.80mm_HandSolder" H 6438 3100 50  0001 C CNN
 F 3 "~" H 6400 3250 50  0001 C CNN
