File: hardware/ETH1CLCR2/V_Diff_Amp.sch (KiCad schematic (older format))
At the start: 31 parts, among them U1001 MCP6L91RT-EMS, U1002 MCP6L91RT-EMS

Commit message: Schematic design
Parts:
- removed U1001, U1002: MCP6L91RT-EMS, Package_SO:MSOP-8_3x3mm_P0.65mm, symbol Amplifier_Operational:MCP6L91RT-EMS
- added C1003, C1005: 1u, symbol Device:C
- added C1004, C1006: DNP, symbol Device:C
- added C1007, C1008, C1009, C1010, C1011, C1012, C1013, C1014, C1015, C1016, C1017, C1018: 100n, symbol Device:C
- added FB1001: Ferrite_Bead_Small, symbol Device:Ferrite_Bead_Small
- added R1019, R1026: 100k/.1%, symbol Device:R
- added R1020: 100, symbol Device:R
- added R1021, R1027: 2k/.1%, symbol Device:R
- added R1022, R1028: 18k/.1%, symbol Device:R
- added R1023, R1029: 1k, symbol Device:R
- added R1024: 3k3/.1%, symbol Device:R
- added R1025: DNP, symbol Device:R
- added TP1001: TestPoint, symbol Connector:TestPoint
- added U1001, U1008, U1009: MCP6L91RT-ESN, Package_SO:SOIC-8_3.9x4.9mm_P1.27mm, symbol Amplifier_Operational:MCP6L91RT-ESN
- added U1002, U1006, U1010, U1011: SN74LVC1G3157, symbol ETH1CLCR2:SN74LVC1G3157
- added U1007, U1012: MCP661, symbol ETH1CLCR2:MCP661
- added U804, U805, U806: SN74LVC1T45DBV, Package_TO_SOT_SMD:SOT-23-6, symbol Logic_LevelTranslator:SN74LVC1T45DBV
- R1010, R1015: renamed from R?; value R -> DNP
- RV1001: value R_POT -> 20k_POT
- gave numbers to parts that had none: 13
Connections:
- net labels added: +3.3V, +5VA, ADC_VIN, L_POT, VDIFF0, VDIFF1, VDIFF2
- net labels removed: +5VP
- wire segments 81 -> 251
Other:
- moved on the sheet: C1001, C1002, D1001, D1002, D1003, K1001, Q1001, R1001, R1002, R1003, R1004, R1005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

Commit message: Footprints assigned.
Parts:
- added C819, C820, C821, C822, C823, C824: 100n, Capacitor_SMD:C_0603_1608Metric_Pad1.08x0.95mm_HandSolder, symbol Device:C
- added TP801, TP802, TP803, TP804, TP805, TP806: TestPoint, TestPoint:TestPoint_Plated_Hole_D2.0mm, symbol Connector:TestPoint
- C801: renamed from C1001; footprint (none) -> Capacitor_SMD:C_0603_1608Metric_Pad1.08x0.95mm_HandSolder
- C802: renamed from C1002; footprint (none) -> Capacitor_SMD:C_0603_1608Metric_Pad1.08x0.95mm_HandSolder
- C803: renamed from C1004; footprint (none) -> Capacitor_SMD:C_0603_1608Metric_Pad1.08x0.95mm_HandSolder
- C804: renamed from C1003; footprint (none) -> Capacitor_SMD:C_0603_1608Metric_Pad1.08x0.95mm_HandSolder
- C805: renamed from C1005; footprint (none) -> Capacitor_SMD:C_0603_1608Metric_Pad1.08x0.95mm_HandSolder
- C806: renamed from C1006; footprint (none) -> Capacitor_SMD:C_0603_1608Metric_Pad1.08x0.95mm_HandSolder
- C807: renamed from C1007; footprint (none) -> Capacitor_SMD:C_0603_1608Metric_Pad1.08x0.95mm_HandSolder
- C808: renamed from C1008; footprint (none) -> Capacitor_SMD:C_0603_1608Metric_Pad1.08x0.95mm_HandSolder
- C809: renamed from C1009; footprint (none) -> Capacitor_SMD:C_0603_1608Metric_Pad1.08x0.95mm_HandSolder
- C810: renamed from C1010; footprint (none) -> Capacitor_SMD:C_0603_1608Metric_Pad1.08x0.95mm_HandSolder
- C811: renamed from C1011; footprint (none) -> Capacitor_SMD:C_0603_1608Metric_Pad1.08x0.95mm_HandSolder
- C812: renamed from C1012; footprint (none) -> Capacitor_SMD:C_0603_1608Metric_Pad1.08x0.95mm_HandSolder
- C813: renamed from C1013; footprint (none) -> Capacitor_SMD:C_0603_1608Metric_Pad1.08x0.95mm_HandSolder
- C814: renamed from C1014; footprint (none) -> Capacitor_SMD:C_0603_1608Metric_Pad1.08x0.95mm_HandSolder
- C815: renamed from C1015; footprint (none) -> Capacitor_SMD:C_0603_1608Metric_Pad1.08x0.95mm_HandSolder
- C816: renamed from C1016; footprint (none) -> Capacitor_SMD:C_0603_1608Metric_Pad1.08x0.95mm_HandSolder
- C817: renamed from C1017; footprint (none) -> Capacitor_SMD:C_0603_1608Metric_Pad1.08x0.95mm_HandSolder
- C818: renamed from C1018; footprint (none) -> Capacitor_SMD:C_0603_1608Metric_Pad1.08x0.95mm_HandSolder
- D802: renamed from D1003; value D -> 1N4148W; footprint (none) -> Diode_SMD:D_SOD-123
- FB801: renamed from FB1001; value Ferrite_Bead_Small -> BLM18TG102TN1D; footprint (none) -> Inductor_SMD:L_0603_1608Metric_Pad1.05x0.95mm_HandSolder
- K801: renamed from K1001; footprint (none) -> ETH1CLCR2:SA
- R801: renamed from R1010; footprint (none) -> Resistor_SMD:R_0603_1608Metric_Pad0.98x0.95mm_HandSolder
- R802: renamed from R1001; footprint (none) -> Resistor_SMD:R_0603_1608Metric_Pad0.98x0.95mm_HandSolder
- R803: renamed from R1002; footprint (none) -> Resistor_SMD:R_0603_1608Metric_Pad0.98x0.95mm_HandSolder
- R804: renamed from R1003; footprint (none) -> Resistor_SMD:R_0603_1608Metric_Pad0.98x0.95mm_HandSolder
- R805: renamed from R1004; footprint (none) -> Resistor_SMD:R_0603_1608Metric_Pad0.98x0.95mm_HandSolder
- R806: renamed from R1011; footprint (none) -> Resistor_SMD:R_0603_1608Metric_Pad0.98x0.95mm_HandSolder
- R807: renamed from R1012; footprint (none) -> Resistor_SMD:R_0603_1608Metric_Pad0.98x0.95mm_HandSolder
- R808: renamed from R1013; footprint (none) -> Resistor_SMD:R_0603_1608Metric_Pad0.98x0.95mm_HandSolder
- R809: renamed from R1019; footprint (none) -> Resistor_SMD:R_0603_1608Metric_Pad0.98x0.95mm_HandSolder
- R810: renamed from R1014; footprint (none) -> Resistor_SMD:R_0603_1608Metric_Pad0.98x0.95mm_HandSolder
- R811: renamed from R1015; footprint (none) -> Resistor_SMD:R_0603_1608Metric_Pad0.98x0.95mm_HandSolder
- R812: renamed from R1016; footprint (none) -> Resistor_SMD:R_0603_1608Metric_Pad0.98x0.95mm_HandSolder
- R813: renamed from R1017; footprint (none) -> Resistor_SMD:R_0603_1608Metric_Pad0.98x0.95mm_HandSolder
- R814: renamed from R1021; footprint (none) -> Resistor_SMD:R_0603_1608Metric_Pad0.98x0.95mm_HandSolder
- R815: renamed from R1022; footprint (none) -> Resistor_SMD:R_0603_1608Metric_Pad0.98x0.95mm_HandSolder
- R816: renamed from R1005; footprint (none) -> Resistor_SMD:R_0603_1608Metric_Pad0.98x0.95mm_HandSolder
- R817: renamed from R1020; footprint (none) -> Resistor_SMD:R_0603_1608Metric_Pad0.98x0.95mm_HandSolder
- R818: renamed from R1023; footprint (none) -> Resistor_SMD:R_0603_1608Metric_Pad0.98x0.95mm_HandSolder
- R819: renamed from R1006; footprint (none) -> Resistor_SMD:R_0603_1608Metric_Pad0.98x0.95mm_HandSolder
- R820: renamed from R1007; footprint (none) -> Resistor_SMD:R_0603_1608Metric_Pad0.98x0.95mm_HandSolder
- R821: renamed from R1008; footprint (none) -> Resistor_SMD:R_0603_1608Metric_Pad0.98x0.95mm_HandSolder
- R822: renamed from R1025; footprint (none) -> Resistor_SMD:R_0603_1608Metric_Pad0.98x0.95mm_HandSolder
- R823: renamed from R1009; footprint (none) -> Resistor_SMD:R_0603_1608Metric_Pad0.98x0.95mm_HandSolder
- R824: renamed from R1018; footprint (none) -> Resistor_SMD:R_0603_1608Metric_Pad0.98x0.95mm_HandSolder
- R825: renamed from R1024; footprint (none) -> Resistor_SMD:R_0603_1608Metric_Pad0.98x0.95mm_HandSolder
- R826: renamed from R1026; footprint (none) -> Resistor_SMD:R_0603_1608Metric_Pad0.98x0.95mm_HandSolder
- R827: renamed from R1027; footprint (none) -> Resistor_SMD:R_0603_1608Metric_Pad0.98x0.95mm_HandSolder
- R828: renamed from R1028; footprint (none) -> Resistor_SMD:R_0603_1608Metric_Pad0.98x0.95mm_HandSolder
- R829: renamed from R1029; footprint (none) -> Resistor_SMD:R_0603_1608Metric_Pad0.98x0.95mm_HandSolder
- RV801: renamed from RV1001; value 20k_POT -> TS53YJ203MR10; footprint (none) -> Potentiometer_SMD:Potentiometer_Vishay_TS53YJ_Vertical
- TP807: renamed from TP1001; footprint (none) -> TestPoint:TestPoint_Plated_Hole_D2.0mm
- U802: renamed from U1003; footprint (none) -> Package_SO:SOIC-8_3.9x4.9mm_P1.27mm
- U803: renamed from U1004; footprint (none) -> Package_SO:SOIC-8_3.9x4.9mm_P1.27mm
- U804: renamed from U1002; footprint (none) -> Package_TO_SOT_SMD:SOT-23-6_Handsoldering
- U805: renamed from U1006; footprint (none) -> Package_TO_SOT_SMD:SOT-23-6_Handsoldering
- U806: renamed from U1007; footprint (none) -> Package_SO:SOIC-8_3.9x4.9mm_P1.27mm
- U808: renamed from U1005; footprint (none) -> Package_SO:SOIC-8_3.9x4.9mm_P1.27mm
- U810: renamed from U1010; footprint (none) -> Package_TO_SOT_SMD:SOT-23-6_Handsoldering
- U811: renamed from U1011; footprint (none) -> Package_TO_SOT_SMD:SOT-23-6_Handsoldering
- U812: renamed from U1012; footprint (none) -> Package_SO:SOIC-8_3.9x4.9mm_P1.27mm
- renumbered D1001 to D801, D1002 to D803, Q1001 to Q801, U1001 to U801, U1008 to U807, U804 to U809, U1009 to U813, U805 to U814, U806 to U815
Connections:
- net +3V3: now also C822.1, C823.1, C824.1
- net +5VA: now also C819.1, C820.1, C821.1
- net GND: now also C819.2, C820.2, C821.2, C822.2, C823.2, C824.2
- net at R813.1, U803.6, U804.4 (COM): now also TP803.1
- net at R822.1, U805.4 (COM), U810.4 (COM): now also TP804.1
- net at R801.2, U801.2 (-), U801.6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: now also TP802.1
- net at R811.2, U807.2 (-), U807.6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: now also TP806.1
- net at R801.1, R806.2, R808.1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: now also TP801.1
- net at R811.1, R812.2, R824.1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: now also TP805.1

Commit message: Schematic
Parts:
- added R830, R831: 200/.1%, Resistor_SMD:R_0603_1608Metric_Pad0.98x0.95mm_HandSolder, symbol Device:R
Connections:
- net at R808.2, U802.2 (-): now also R830.1; no longer K801.8
- net at R824.2, U808.2 (-): now also R831.2; no longer K801.7
- new net: K801.7, R831.1
- new net: K801.8, R830.2
Other:
- moved on the sheet: R808, R811, R824
Changed lines of the file:
@@
 $Descr A3 16535 11693
 encoding utf-8
-Sheet 8 13
+Sheet 8 12
 Title ""
 Date ""
@@
 L Device:R R808
 U 1 1 621FAD95
-P 4550 3100
-F 0 "R808" V 4343 3100 50  0000 C CNN
-F 1 "1k8/.1%" V 4434 3100 50  0000 C CNN
-F 2 "Resistor_SMD:R_0603_1608Metric_Pad0.98x0.95mm_HandSolder" V 4480 3100 50  0001 C CNN
-F 3 "~" H 4550 3100 50  0001 C CNN
-	1    4550 3100
-	0    1    1    0
-$EndComp
-Wire Wire Line
-	4400 3100 4200 3100
-Wire Wire Line
-	4200 3100 4200 2400
+P 4750 2850
+F 0 "R808" V 4543 2850 50  0000 C CNN
+F 1 "1k8/.1%" V 4634 2850 50  0000 C CNN
+F 2 "Resistor_SMD:R_0603_1608Metric_Pad0.98x0.95mm_HandSolder" V 4680 2850 50  0001 C CNN
+F 3 "~" H 4750 2850 50  0001 C CNN
+	1    4750 2850
+	0    1    1    0
+$EndComp
+Wire Wire Line
+	4600 2850 4200 2850
+Wire Wire Line
+	4200 2850 4200 2400
 Wire Wire Line
 	4200 2400 4250 2400
 Wire Wire Line
-	4700 3100 5000 3100
-Wire Wire Line
-	5000 3100 5000 2300
+	4900 2850 5000 2850
+Wire Wire Line
+	5000 2850 5000 2300
 Connection ~ 5000 2300
 Wire Wire Line
@@
 $EndComp
 Wire Wire Line
-	4200 3350 4200 3100
-Connection ~ 4200 3100
+	4200 3350 4200 3300
+Connection ~ 4200 2850
 NoConn ~ 4600 3350
 NoConn ~ 4500 3950
@@
 L Device:R R811
 U 1 1 622462BE
-P 4550 4500
-F 0 "R811" V 4343 4500 50  0000 C CNN
-F 1 "DNP" V 4434 4500 50  0000 C CNN
-F 2 "Resistor_SMD:R_0603_1608Metric_Pad0.98x0.95mm_HandSolder" V 4480 4500 50  0001 C CNN
-F 3 "~" H 4550 4500 50  0001 C CNN
-	1    4550 4500
-	0    1    1    0
-$EndComp
-Wire Wire Line
-	4400 4500 4200 4500
-Wire Wire Line
-	4200 4500 4200 5050
+P 4750 4550
+F 0 "R811" V 4543 4550 50  0000 C CNN
+F 1 "DNP" V 4634 4550 50  0000 C CNN
+F 2 "Resistor_SMD:R_0603_1608Metric_Pad0.98x0.95mm_HandSolder" V 4680 4550 50  0001 C CNN
+F 3 "~" H 4750 4550 50  0001 C CNN
+	1    4750 4550
+	0    1    1    0
+$EndComp
+Wire Wire Line
+	4600 4550 4200 4550
+Wire Wire Line
+	4200 4550 4200 5050
 Wire Wire Line
 	4200 5050 4250 5050
 Wire Wire Line
-	4700 4500 5000 4500
-Wire Wire Line
-	5000 4500 5000 5150
+	4900 4550 5000 4550
+Wire Wire Line
+	5000 4550 5000 5150
 Wire Wire Line
 	5000 5150 4850 5150
@@
 L Device:R R824
 U 1 1 622462CA
-P 4550 5950
-F 0 "R824" V 4343 5950 50  0000 C CNN
-F 1 "1k8/.1%" V 4434 5950 50  0000 C CNN
-F 2 "Resistor_SMD:R_0603_1608Metric_Pad0.98x0.95mm_HandSolder" V 4480 5950 50  0001 C CNN
-F 3 "~" H 4550 5950 50  0001 C CNN
-	1    4550 5950
-	0    1    1    0
-$EndComp
-Wire Wire Line
-	4400 5950 4100 5950
-Wire Wire Line
-	4100 5950 4100 5250
+P 4750 5850
+F 0 "R824" V 4543 5850 50  0000 C CNN
+F 1 "1k8/.1%" V 4634 5850 50  0000 C CNN
+F 2 "Resistor_SMD:R_0603_1608Metric_Pad0.98x0.95mm_HandSolder" V 4680 5850 50  0001 C CNN
+F 3 "~" H 4750 5850 50  0001 C CNN
+	1    4750 5850
+	0    1    1    0
+$EndComp
+Wire Wire Line
+	4600 5850 4100 5850
+Wire Wire Line
+	4100 5850 4100 5250
 Wire Wire Line
 	4100 5250 4250 5250
 Wire Wire Line
-	4700 5950 5000 5950
-Wire Wire Line
-	5000 5950 5000 5150
+	4900 5850 5000 5850
+Wire Wire Line
+	5000 5850 5000 5150
 Connection ~ 5000 5150
 Wire Wire Line
@@
 Connection ~ 3750 5050
 Wire Wire Line
-	4100 5250 4100 3950
+	4100 5250 4100 4300
 Connection ~ 4100 5250
 $Comp
@@
 	12500 3750 12450 3750
 Connection ~ 12450 3750
+$Comp
+L Device:R R831
+U 1 1 60F43C5D
+P 4100 4150
+F 0 "R831" H 4170 4196 50  0000 L CNN
+F 1 "200/.1%" H 4170 4105 50  0000 L CNN
+F 2 "Resistor_SMD:R_0603_1608Metric_Pad0.98x0.95mm_HandSolder" V 4030 4150 50  0001 C CNN
+F 3 "~" H 4100 4150 50  0001 C CNN
+	1    4100 4150
+	1    0    0    -1
+$EndComp
+Wire Wire Line
+	4100 4000 4100 3950
+$Comp
+L Device:R R830
+U 1 1 60F4703B
+P 4200 3150
+F 0 "R830" H 4270 3196 50  0000 L CNN
+F 1 "200/.1%" H 4270 3105 50  0000 L CNN
+F 2 "Resistor_SMD:R_0603_1608Metric_Pad0.98x0.95mm_HandSolder" V 4130 3150 50  0001 C CNN
+F 3 "~" H 4200 3150 50  0001 C CNN
+	1    4200 3150
+	1    0    0    -1
+$EndComp
+Wire Wire Line
+	4200 3000 4200 2850
 $EndSCHEMATC

Commit message: Footprints
Parts:
- RV801: value TS53YJ203MR10 -> 3314J-1-203E; footprint Potentiometer_SMD:Potentiometer_Vishay_TS53YJ_Vertical -> Potentiometer_SMD:Potentiometer_Bourns_3314J_Vertical
Changed lines of the file:
@@
 P 1950 6200
 F 0 "RV801" V 1835 6200 50  0000 C CNN
-F 1 "TS53YJ203MR10" V 1744 6200 50  0000 C CNN
-F 2 "Potentiometer_SMD:Potentiometer_Vishay_TS53YJ_Vertical" H 1950 6200 50  0001 C CNN
+F 1 "3314J-1-203E" V 1744 6200 50  0000 C CNN
+F 2 "Potentiometer_SMD:Potentiometer_Bourns_3314J_Vertical" H 1950 6200 50  0001 C CNN
 F 3 "~" H 1950 6200 50  0001 C CNN
 	1    1950 6200

Commit message: PCB
Parts:
- removed C819: 100n, Capacitor_SMD:C_0603_1608Metric_Pad1.08x0.95mm_HandSolder, symbol Device:C
- TP801, TP802, TP803, TP804, TP805, TP806, TP807: footprint TestPoint:TestPoint_Plated_Hole_D2.0mm -> TestPoint:TestPoint_Pad_1.0x1.0mm
- U809, U814, U815: footprint Package_TO_SOT_SMD:SOT-23-6 -> Package_TO_SOT_SMD:SOT-23-6_Handsoldering
- renumbered C812 to C811, C820 to C812, C821 to C813, C815 to C814, C816 to C815, C817 to C816, C818 to C817, C822 to C818, C823 to C819, C824 to C820, C811 to C821, C814 to C822, C813 to C823, R808 to R806, R806 to R807, R807 to R808, R830 to R809, R831 to R810, R809 to R811, R810 to R812, R811 to R813, R812 to R814, R813 to R815, R814 to R816, R815 to R817, R816 to R818, R817 to R819, R818 to R820, R819 to R821, R820 to R822, R821 to R823, R822 to R824, R823 to R825, R824 to R826, R825 to R827, R826 to R828, R827 to R829, R828 to R830, R829 to R831
Connections:
- net +5V: now also C821.1, C822.1, C823.1
- net +5VA: no longer C821.1, C822.1, C823.1
Other:
- moved on the sheet: C807, C808, C809, C810, C812, C813, C818, C819, C820, C821, C822, C823
