File: hardware/ETH1CLCR2/V_Diff_Amp.sch (KiCad schematic (older format))
At the start: 83 parts, among them K801 TQ2SA-5V, Q801 BC847, U801 MCP6L91RT-ESN, U802 MCP661, U803 MCP661, U804 SN74LVC1G3157, U805 SN74LVC1G3157, U806 MCP661, U807 MCP6L91RT-ESN, U808 MCP661, U809 SN74LVC1T45DBV, U810 SN74LVC1G3157, U811 SN74LVC1G3157, U812 MCP661, U813 MCP6L91RT-ESN, U814 SN74LVC1T45DBV, U815 SN74LVC1T45DBV

Commit message: PCB
Changed lines of the file:
@@
 U 1 1 622462AC
 P 4500 5150
-F 0 "U808" H 4700 5400 50  0000 L CNN
+F 0 "U808" H 4650 5400 50  0000 L CNN
 F 1 "MCP661" H 4600 5300 50  0000 L CNN
 F 2 "Package_SO:SOIC-8_3.9x4.9mm_P1.27mm" H 4600 5200 50  0001 C CNN

Commit message: PCB
Parts:
- U801, U807, U813: value MCP6L91RT-ESN -> MCP6L91T-E/SN
- U802, U803, U806, U808, U812: value MCP661 -> MCP661-E/SN
- U804, U805, U810, U811: value SN74LVC1G3157 -> SN74LVC1G3157DBVR
Other:
- moved on the sheet: TP803
Changed lines of the file:
@@
 P 4500 2300
 F 0 "U802" H 4700 2550 50  0000 L CNN
-F 1 "MCP661" H 4600 2450 50  0000 L CNN
+F 1 "MCP661-E/SN" H 4600 2450 50  0000 L CNN
 F 2 "Package_SO:SOIC-8_3.9x4.9mm_P1.27mm" H 4600 2350 50  0001 C CNN
 F 3 "" H 4600 2450 50  0001 C CNN
@@
 	4200 2200 4250 2200
 Wire Wire Line
-	4700 1650 5000 1650
-Wire Wire Line
-	5000 1650 5000 2300
-Wire Wire Line
-	5000 2300 4850 2300
+	4700 1650 5200 1650
+Wire Wire Line
+	5200 1650 5200 2300
+Wire Wire Line
+	5200 2300 4850 2300
 $Comp
 L Device:R R806
@@
 	4200 2400 4250 2400
 Wire Wire Line
-	4900 2850 5000 2850
-Wire Wire Line
-	5000 2850 5000 2300
-Connection ~ 5000 2300
+	4900 2850 5200 2850
+Wire Wire Line
+	5200 2850 5200 2300
+Connection ~ 5200 2300
 Wire Wire Line
 	4200 2200 3750 2200
@@
 P 4500 5150
 F 0 "U808" H 4650 5400 50  0000 L CNN
-F 1 "MCP661" H 4600 5300 50  0000 L CNN
+F 1 "MCP661-E/SN" H 4600 5300 50  0000 L CNN
 F 2 "Package_SO:SOIC-8_3.9x4.9mm_P1.27mm" H 4600 5200 50  0001 C CNN
 F 3 "" H 4600 5300 50  0001 C CNN
@@
 	4200 5050 4250 5050
 Wire Wire Line
-	4900 4550 5000 4550
-Wire Wire Line
-	5000 4550 5000 5150
-Wire Wire Line
-	5000 5150 4850 5150
+	4900 4550 5200 4550
+Wire Wire Line
+	5200 4550 5200 5150
+Wire Wire Line
+	5200 5150 4850 5150
 $Comp
 L Device:R R826
@@
 	4100 5250 4250 5250
 Wire Wire Line
-	4900 5850 5000 5850
-Wire Wire Line
-	5000 5850 5000 5150
-Connection ~ 5000 5150
+	4900 5850 5200 5850
+Wire Wire Line
+	5200 5850 5200 5150
+Connection ~ 5200 5150
 Wire Wire Line
 	4200 5050 3750 5050
@@
 P 7000 3750
 F 0 "U803" H 7200 4000 50  0000 L CNN
-F 1 "MCP661" H 7100 3900 50  0000 L CNN
+F 1 "MCP661-E/SN" H 7100 3900 50  0000 L CNN
 F 2 "Package_SO:SOIC-8_3.9x4.9mm_P1.27mm" H 7100 3800 50  0001 C CNN
 F 3 "" H 7100 3900 50  0001 C CNN
@@
 	6300 3050 6300 2300
 Wire Wire Line
-	6300 2300 5000 2300
-Wire Wire Line
-	5000 5150 6300 5150
+	6300 2300 5200 2300
+Wire Wire Line
+	5200 5150 6300 5150
 Wire Wire Line
 	6300 5150 6300 5050
@@
 P 10450 3850
 F 0 "U806" H 10600 4100 50  0000 L CNN
-F 1 "MCP661" H 10500 4000 50  0000 L CNN
+F 1 "MCP661-E/SN" H 10500 4000 50  0000 L CNN
 F 2 "Package_SO:SOIC-8_3.9x4.9mm_P1.27mm" H 10550 3900 50  0001 C CNN
 F 3 "" H 10550 4000 50  0001 C CNN
@@
 P 8850 3750
 F 0 "U804" H 8850 4215 50  0000 C CNN
-F 1 "SN74LVC1G3157" H 8850 4124 50  0000 C CNN
+F 1 "SN74LVC1G3157DBVR" H 8850 4124 50  0000 C CNN
 F 2 "Package_TO_SOT_SMD:SOT-23-6_Handsoldering" H 8850 4100 50  0001 C CNN
 F 3 "" H 8850 4100 50  0001 C CNN
@@
 P 11650 3750
 F 0 "U805" H 11650 4215 50  0000 C CNN
-F 1 "SN74LVC1G3157" H 11650 4124 50  0000 C CNN
+F 1 "SN74LVC1G3157DBVR" H 11650 4124 50  0000 C CNN
 F 2 "Package_TO_SOT_SMD:SOT-23-6_Handsoldering" H 11650 4100 50  0001 C CNN
 F 3 "" H 11650 4100 50  0001 C CNN
@@
 	9250 3950 9200 3950
 Wire Wire Line
-	9200 3550 9250 3550
-Wire Wire Line
-	9250 3550 9250 3200
-Wire Wire Line
-	9250 3200 11250 3200
-Wire Wire Line
-	11250 3200 11250 3550
-Wire Wire Line
-	11250 3550 11300 3550
+	9200 3550 9350 3550
+Wire Wire Line
+	9350 3550 9350 3200
+Wire Wire Line
+	9350 3200 11150 3200
+Wire Wire Line
+	11150 3200 11150 3550
+Wire Wire Line
+	11150 3550 11300 3550
 $Comp
 L power:+5VA #PWR0814
@@
 P 10450 6250
 F 0 "U812" H 10600 6500 50  0000 L CNN
-F 1 "MCP661" H 10500 6400 50  0000 L CNN
+F 1 "MCP661-E/SN" H 10500 6400 50  0000 L CNN
 F 2 "Package_SO:SOIC-8_3.9x4.9mm_P1.27mm" H 10550 6300 50  0001 C CNN
 F 3 "" H 10550 6400 50  0001 C CNN
@@
 P 8850 6150
 F 0 "U810" H 8850 6615 50  0000 C CNN
-F 1 "SN74LVC1G3157" H 8850 6524 50  0000 C CNN
+F 1 "SN74LVC1G3157DBVR" H 8850 6524 50  0000 C CNN
 F 2 "Package_TO_SOT_SMD:SOT-23-6_Handsoldering" H 8850 6500 50  0001 C CNN
 F 3 "" H 8850 6500 50  0001 C CNN
@@
 P 11650 6150
 F 0 "U811" H 11650 6615 50  0000 C CNN
-F 1 "SN74LVC1G3157" H 11650 6524 50  0000 C CNN
+F 1 "SN74LVC1G3157DBVR" H 11650 6524 50  0000 C CNN
 F 2 "Package_TO_SOT_SMD:SOT-23-6_Handsoldering" H 11650 6500 50  0001 C CNN
 F 3 "" H 11650 6500 50  0001 C CNN
@@
 	9250 6350 9200 6350
 Wire Wire Line
-	9200 5950 9250 5950
-Wire Wire Line
-	9250 5950 9250 5600
-Wire Wire Line
-	9250 5600 11250 5600
-Wire Wire Line
-	11250 5600 11250 5950
-Wire Wire Line
-	11250 5950 11300 5950
+	9200 5950 9350 5950
+Wire Wire Line
+	9350 5950 9350 5600
+Wire Wire Line
+	9350 5600 11150 5600
+Wire Wire Line
+	11150 5600 11150 5950
+Wire Wire Line
+	11150 5950 11300 5950
 $Comp
 L power:+5VA #PWR0836
@@
 VDIFF1
 Wire Wire Line
-	8500 3750 7600 3750
+	8500 3750 7750 3750
 Connection ~ 7400 3750
 $Comp
@@
 P 3400 2200
 F 0 "U801" H 3650 2450 50  0000 L CNN
-F 1 "MCP6L91RT-ESN" H 3400 2350 50  0000 L CNN
+F 1 "MCP6L91T-E/SN" H 3400 2350 50  0000 L CNN
 F 2 "Package_SO:SOIC-8_3.9x4.9mm_P1.27mm" H 3300 2000 50  0001 L CNN
 F 3 "http://ww1.microchip.com/downloads/en/DeviceDoc/22141b.pdf" H 3550 2350 50  0001 C CNN
@@
 P 3400 5050
 F 0 "U807" H 3650 5300 50  0000 L CNN
-F 1 "MCP6L91RT-ESN" H 3400 5200 50  0000 L CNN
+F 1 "MCP6L91T-E/SN" H 3400 5200 50  0000 L CNN
 F 2 "Package_SO:SOIC-8_3.9x4.9mm_P1.27mm" H 3300 4850 50  0001 L CNN
 F 3 "http://ww1.microchip.com/downloads/en/DeviceDoc/22141b.pdf" H 3550 5200 50  0001 C CNN
@@
 P 13950 6250
 F 0 "U813" H 14200 6500 50  0000 L CNN
-F 1 "MCP6L91RT-ESN" H 13950 6400 50  0000 L CNN
+F 1 "MCP6L91T-E/SN" H 13950 6400 50  0000 L CNN
 F 2 "Package_SO:SOIC-8_3.9x4.9mm_P1.27mm" H 13850 6050 50  0001 L CNN
 F 3 "http://ww1.microchip.com/downloads/en/DeviceDoc/22141b.pdf" H 14100 6400 50  0001 C CNN
@@
 L Connector:TestPoint TP803
 U 1 1 61094A28
-P 7600 3700
-F 0 "TP803" H 7658 3818 50  0000 L CNN
-F 1 "TestPoint" H 7658 3727 50  0000 L CNN
-F 2 "TestPoint:TestPoint_Pad_1.0x1.0mm" H 7800 3700 50  0001 C CNN
-F 3 "~" H 7800 3700 50  0001 C CNN
-	1    7600 3700
-	1    0    0    -1
-$EndComp
-Wire Wire Line
-	7600 3700 7600 3750
-Connection ~ 7600 3750
-Wire Wire Line
-	7600 3750 7400 3750
+P 7750 3700
+F 0 "TP803" H 7808 3818 50  0000 L CNN
+F 1 "TestPoint" H 7808 3727 50  0000 L CNN
+F 2 "TestPoint:TestPoint_Pad_1.0x1.0mm" H 7950 3700 50  0001 C CNN
+F 3 "~" H 7950 3700 50  0001 C CNN
+	1    7750 3700
+	1    0    0    -1
+$EndComp
+Wire Wire Line
+	7750 3700 7750 3750
+Connection ~ 7750 3750
+Wire Wire Line
+	7750 3750 7400 3750
 $Comp
 L Connector:TestPoint TP804
