File: hardware/ETH1CLCR2/DDS.sch (KiCad schematic (older format))
At the start: 58 parts, among them Q1201 FDV301N, U1201 AD9834, U1202 AD8038, U1203 DAC7811, U1204 AD8038, U1205 LMH6639, U1206 LMH6639, U1207 DG409, U1209 LM393

Commit message: Schematic
Parts:
- added U? (x2): 74AC161, symbol ETH1CLCR2:74AC161
- added U?: 74AHC1G14, symbol 74xGxx:74AHC1G14
- added U?: 74AUP1G79, symbol 74xGxx:74AUP1G79
Connections:
- net labels added: DDS_CS, DDS_SCLK, DDS_SDATA, MDAC_CS, MDAC_SCK, MDAC_SDIN, MDAC_SDO
- wire segments 218 -> 258
- no-connect marks 3 -> 11
Other:
- moved on the sheet: C1202

Commit message: Schematic
Parts:
- removed U1209: LM393, symbol Comparator:LM393
- added C1209, C1210, C1211, C1212, C1214, C1215, C1216, C1217, C1218, C1219, C1220, C1221, C1222, C1223, C1224, C1225, C1226, C1227, C1228, C1229, C1230: 100n, Capacitor_SMD:C_0603_1608Metric_Pad1.08x0.95mm_HandSolder, symbol Device:C
- added R1226: 1k, Resistor_SMD:R_0603_1608Metric_Pad0.98x0.95mm_HandSolder, symbol Device:R
- added R1227, R1228, R1231: 68, Resistor_SMD:R_0603_1608Metric_Pad0.98x0.95mm_HandSolder, symbol Device:R
- added U1213, U1214, U1215: SN74LVC1T45DBV, Package_TO_SOT_SMD:SOT-23-6, symbol Logic_LevelTranslator:SN74LVC1T45DBV
- added X1201: 830208220601, symbol ETH1CLCR2:IQXO-791
- C1201, C1202, C1203, C1204, C1205, C1206, C1207, C1213: footprint (none) -> Capacitor_SMD:C_0603_1608Metric_Pad1.08x0.95mm_HandSolder
- C1208: value 3p3 -> 3p3/COG; footprint (none) -> Capacitor_SMD:C_0603_1608Metric_Pad1.08x0.95mm_HandSolder
- FB1201: value Ferrite_Bead_Small -> BLM18SP601SZ1D; footprint (none) -> Inductor_SMD:L_0603_1608Metric_Pad1.05x0.95mm_HandSolder
- FB1202: value Ferrite -> BLM18SP601SZ1D; footprint (none) -> Inductor_SMD:L_0603_1608Metric_Pad1.05x0.95mm_HandSolder
- R1201, R1202, R1203, R1204, R1205, R1206, R1207, R1208, R1209, R1210, R1211, R1212, R1213, R1214, R1215, R1216, R1217, R1218, R1219, R1220, R1221, R1222, R1223, R1224, R1225, R1229, R1230, RV1201: footprint (none) -> Resistor_SMD:R_0603_1608Metric_Pad0.98x0.95mm_HandSolder
- gave numbers to parts that had none: 4
Connections:
- net labels added: +5V, A0, A1, DDS_CLK, DDS_DIV2, DDS_DIV4, DDS_DIV8, DDS_LPF, LPF, MUX_A0, MUX_A1, ~DDS_DIV10
- net labels removed: +5VF, -5VF
- wire segments 258 -> 385
Other:
- moved on the sheet: C1201, C1202, C1203, C1204, C1205, C1206, C1207, C1208, C1213, D1201, D1202, D1204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

Commit message: Footprints
Parts:
- D1201, D1202: footprint (none) -> Diode_SMD:D_SMA
- D1204, D1205, D1206, D1207: value 5V6 -> BZX584C5V6; footprint (none) -> Diode_SMD:D_SOD-523
- L1201, L1202, L1203, L1204: value 10u -> CBMF1608T100K; footprint (none) -> Inductor_SMD:L_0603_1608Metric_Pad1.05x0.95mm_HandSolder
- Q1201: footprint (none) -> Package_TO_SOT_SMD:SOT-23
- RV1201: value 100k -> 3314J-1-104E; footprint Resistor_SMD:R_0603_1608Metric_Pad0.98x0.95mm_HandSolder -> Potentiometer_SMD:Potentiometer_Bourns_3314J_Vertical
- U1202, U1204, U1205, U1206: footprint (none) -> Package_SO:SOIC-8_3.9x4.9mm_P1.27mm
- U1203: footprint (none) -> Package_SO:VSSOP-10_3x3mm_P0.5mm
- U1207, U1211, U1212: footprint (none) -> Package_SO:SOIC-16_3.9x9.9mm_P1.27mm
- U1208, U1210: footprint (none) -> Package_TO_SOT_SMD:SOT-353_SC-70-5_Handsoldering
- X1201: footprint (none) -> ETH1CLCR2:IQXO-791
Connections:
- net -5VA: now also D1202.2 (A), D1205.2 (A), D1207.2 (A), FB1202.1
- net H_CUR: now reaches R1223.1, R1224.1, R1225.1
Other:
- moved on the sheet: C1201, C1202, C1203, C1204, C1205, C1206, C1207, C1208, C1213, D1201, D1202, D1204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

Commit message: PCB
Parts:
- removed C1218: 100n, Capacitor_SMD:C_0603_1608Metric_Pad1.08x0.95mm_HandSolder, symbol Device:C
- renumbered C1213 to C1201, C1201 to C1202, C1202 to C1203, C1208 to C1205, C1203 to C1206, C1205 to C1207, C1206 to C1208, C1207 to C1209, C1209 to C1210, C1210 to C1211, C1211 to C1212, C1212 to C1213, C1219 to C1218, C1220 to C1219, C1221 to C1220, C1222 to C1221, C1223 to C1222, C1224 to C1223, C1225 to C1224, C1226 to C1225, C1227 to C1226, C1228 to C1227, C1229 to C1228, C1230 to C1229, D1204 to D1202, D1206 to D1203, D1202 to D1204, D1207 to D1206, L1203 to L1202, L1202 to L1203, R1229 to R1201, R1230 to R1202, R1219 to R1203, R1201 to R1204, R1202 to R1205, R1221 to R1206, R1209 to R1208, R1217 to R1209, R1223 to R1210, R1203 to R1211, R1205 to R1212, R1224 to R1213, R1210 to R1214, R1208 to R1215, R1225 to R1216, R1220 to R1217, R1211 to R1218, R1204 to R1219, R1206 to R1220, R1212 to R1221, R1215 to R1222, R1222 to R1223, R1218 to R1224, R1213 to R1225, R1216 to R1226, R1214 to R1227, R1226 to R1228, R1227 to R1229, R1228 to R1230, U1205 to U1201, U1201 to U1202, U1202 to U1203, U1203 to U1204, U1204 to U1205, U1207 to U1206, U1206 to U1207, U1213 to U1208, U1208 to U1209, U1214 to U1211, U1211 to U1212, U1212 to U1213, U1215 to U1214
Other:
- moved on the sheet: C1218, C1219, C1220, C1221, C1222, C1223, C1224, C1225, C1226, C1227, C1228, C1229

Commit message: PCB
Connections:
- net AGNDF is gone; now on net GND: Q1201.2 (S)
Changed lines of the file:
@@
 Connection ~ 10350 1200
-$Comp
-L ETH1CLCR2:AGNDF #PWR01205
-U 1 1 611E3FE3
-P 10350 1650
-F 0 "#PWR01205" H 10350 1400 50  0001 C CNN
-F 1 "AGNDF" H 10355 1477 50  0000 C CNN
-F 2 "" H 10350 1650 50  0001 C CNN
-F 3 "" H 10350 1650 50  0001 C CNN
-	1    10350 1650
-	1    0    0    -1
-$EndComp
 $Comp
 L Device:R R1202
@@
 Wire Wire Line
 	4050 10800 4300 10800
+$Comp
+L power:GND #PWR?
+U 1 1 60A1C535
+P 10350 1650
+F 0 "#PWR?" H 10350 1400 50  0001 C CNN
+F 1 "GND" H 10355 1477 50  0000 C CNN
+F 2 "" H 10350 1650 50  0001 C CNN
+F 3 "" H 10350 1650 50  0001 C CNN
+	1    10350 1650
+	1    0    0    -1
+$EndComp
 $EndSCHEMATC

Commit message: PCB
Parts:
- added R1222: 1k, Resistor_SMD:R_0603_1608Metric_Pad0.98x0.95mm_HandSolder, symbol Device:R
- renumbered R1222 to R1223, R1223 to R1224, R1224 to R1225, R1225 to R1226, R1226 to R1227, R1227 to R1228, R1228 to R1229, R1229 to R1230, R1230 to R1231, R1231 to R1232
Connections:
- net GND: now also R1222.2; no longer U1206.9 (DB)
- new net: R1222.1, U1206.9 (DB)
Other:
- moved on the sheet: C1201, C1202, C1203, C1204, C1205, C1206, C1207, C1208, C1209, D1201, D1202, D1203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

Commit message: PCB
Parts:
- R1203, R1217: value 680 -> 680/.1%
- R1209, R1225: value 330 -> 330/.1%
- U1201, U1207: value LMH6639 -> LMH6639MA
- U1203, U1205: value AD8038 -> AD8038ARZ
- U1206: value DG409 -> DG409DY
Other:
- moved on the sheet: R1203, R1209, R1217, R1222, R1225, U1203, U1205
