File: hardware/ETH1CLCR2/DDS.sch (KiCad schematic (older format))
At the start: 101 parts, among them Q1201 FDV301N, Q1202 2SC3326B, Q1203 DTA144E, Q1204 DTC114E, U1201 LMH6639MA, U1202 AD9834, U1203 AD8038ARZ, U1204 DAC7811, U1205 AD8038ARZ, U1206 DG409DY, U1207 LMH6639MA, U1208 TL431DBZ, U1209 SN74LVC1T45DBV, U1210 SN74LVC1T45DBV, U1211 74AHC1G14, U1212 SN74LVC1T45DBV, U1213 74AUP1G79, U1214 74AC161, U1215 74AC161, U1216 SN74LVC1T45DBV, X1201 830208220601

Commit message: PCB done
Parts:
- added C1233, C1234, C1235, C1236: 100n, Capacitor_SMD:C_0603_1608Metric_Pad1.08x0.95mm_HandSolder, symbol Device:C
Connections:
- net GND: now also C1233.2, C1234.2, C1235.2, C1236.2
- net at FB1202.2, U1201.4 (V-), U1207.4 (V-): now also C1235.1, C1236.1
- net at FB1201.2, U1201.7 (V+), U1207.7 (V+): now also C1233.1, C1234.1
Changed lines of the file:
@@
 	13550 2150 13650 2150
-Wire Wire Line
-	12450 1350 12750 1350
 Wire Wire Line
 	13650 1400 13650 1350
@@
 	14500 1800 14500 1750
 Wire Wire Line
-	12450 1350 12450 1850
+	12450 1350 12450 1800
 Wire Wire Line
 	13650 1700 13650 2150
@@
 	12450 4400 12450 3900
 Wire Wire Line
-	12450 4400 11750 4400
+	12450 4400 12000 4400
 Wire Wire Line
 	11750 4400 11750 2800
@@
 Wire Wire Line
 	14850 4800 14850 4750
-Wire Wire Line
-	14100 2650 14800 2650
 Wire Wire Line
 	4750 3050 4750 3100
@@
 Wire Wire Line
 	14150 4800 14500 4800
-Text HLabel 14800 2650 2    50   Output ~ 0
-H_CUR
 Wire Wire Line
 	1850 3250 2400 3250
@@
 L power:PWR_FLAG #FLG01201
 U 1 1 60C70737
-P 12750 1300
-F 0 "#FLG01201" H 12750 1375 50  0001 C CNN
-F 1 "PWR_FLAG" H 12750 1473 50  0000 C CNN
-F 2 "" H 12750 1300 50  0001 C CNN
-F 3 "~" H 12750 1300 50  0001 C CNN
-	1    12750 1300
-	1    0    0    -1
-$EndComp
-Wire Wire Line
-	12750 1300 12750 1350
-Connection ~ 12750 1350
-Wire Wire Line
-	12750 1350 13100 1350
+P 12400 1800
+F 0 "#FLG01201" H 12400 1875 50  0001 C CNN
+F 1 "PWR_FLAG" V 12400 2100 50  0000 C CNN
+F 2 "" H 12400 1800 50  0001 C CNN
+F 3 "~" H 12400 1800 50  0001 C CNN
+	1    12400 1800
+	0    -1   -1   0
+$EndComp
+Wire Wire Line
+	12400 1800 12450 1800
 $Comp
 L power:PWR_FLAG #FLG01202
@@
 Wire Wire Line
 	5850 10800 6100 10800
+$Comp
+L Device:C C1236
+U 1 1 60BD99E4
+P 12450 4600
+F 0 "C1236" H 12565 4646 50  0000 L CNN
+F 1 "100n" H 12565 4555 50  0000 L CNN
+F 2 "Capacitor_SMD:C_0603_1608Metric_Pad1.08x0.95mm_HandSolder" H 12488 4450 50  0001 C CNN
+F 3 "~" H 12450 4600 50  0001 C CNN
+	1    12450 4600
+	1    0    0    -1
+$EndComp
+Wire Wire Line
+	12450 4450 12450 4400
+$Comp
+L power:GND #PWR01275
+U 1 1 60C100D0
+P 12450 4750
+F 0 "#PWR01275" H 12450 4500 50  0001 C CNN
+F 1 "GND" H 12455 4577 50  0000 C CNN
+F 2 "" H 12450 4750 50  0001 C CNN
+F 3 "" H 12450 4750 50  0001 C CNN
+	1    12450 4750
+	1    0    0    -1
+$EndComp
+$Comp
+L Device:C C1235
+U 1 1 60C14C4B
+P 12000 4600
+F 0 "C1235" H 12115 4646 50  0000 L CNN
+F 1 "100n" H 12115 4555 50  0000 L CNN
+F 2 "Capacitor_SMD:C_0603_1608Metric_Pad1.08x0.95mm_HandSolder" H 12038 4450 50  0001 C CNN
+F 3 "~" H 12000 4600 50  0001 C CNN
+	1    12000 4600
+	1    0    0    -1
+$EndComp
+$Comp
+L power:GND #PWR01274
+U 1 1 60C1512C
+P 12000 4750
+F 0 "#PWR01274" H 12000 4500 50  0001 C CNN
+F 1 "GND" H 12005 4577 50  0000 C CNN
+F 2 "" H 12000 4750 50  0001 C CNN
+F 3 "" H 12000 4750 50  0001 C CNN
+	1    12000 4750
+	1    0    0    -1
+$EndComp
+Wire Wire Line
+	12000 4450 12000 4400
+Connection ~ 12000 4400
+Wire Wire Line
+	12000 4400 11750 4400
+$Comp
+L Device:C C1233
+U 1 1 60C89F63
+P 12450 1150
+F 0 "C1233" H 12565 1196 50  0000 L CNN
+F 1 "100n" H 12565 1105 50  0000 L CNN
+F 2 "Capacitor_SMD:C_0603_1608Metric_Pad1.08x0.95mm_HandSolder" H 12488 1000 50  0001 C CNN
+F 3 "~" H 12450 1150 50  0001 C CNN
+	1    12450 1150
+	-1   0    0    1
+$EndComp
+Wire Wire Line
+	12450 1300 12450 1350
+$Comp
+L power:GND #PWR01272
+U 1 1 60C89F6A
+P 12450 1000
+F 0 "#PWR01272" H 12450 750 50  0001 C CNN
+F 1 "GND" H 12455 827 50  0000 C CNN
+F 2 "" H 12450 1000 50  0001 C CNN
+F 3 "" H 12450 1000 50  0001 C CNN
+	1    12450 1000
+	-1   0    0    1
+$EndComp
+Connection ~ 12450 1800
+Wire Wire Line
+	12450 1800 12450 1850
+Connection ~ 12450 1350
+Wire Wire Line
+	14100 2650 14800 2650
+Text HLabel 14800 2650 2    50   Output ~ 0
+H_CUR
+$Comp
+L Device:C C1234
+U 1 1 60C89F70
+P 12900 1150
+F 0 "C1234" H 13015 1196 50  0000 L CNN
+F 1 "100n" H 13015 1105 50  0000 L CNN
+F 2 "Capacitor_SMD:C_0603_1608Metric_Pad1.08x0.95mm_HandSolder" H 12938 1000 50  0001 C CNN
+F 3 "~" H 12900 1150 50  0001 C CNN
+	1    12900 1150
+	-1   0    0    1
+$EndComp
+$Comp
+L power:GND #PWR01273
+U 1 1 60C89F76
+P 12900 1000
+F 0 "#PWR01273" H 12900 750 50  0001 C CNN
+F 1 "GND" H 12905 827 50  0000 C CNN
+F 2 "" H 12900 1000 50  0001 C CNN
+F 3 "" H 12900 1000 50  0001 C CNN
+	1    12900 1000
+	-1   0    0    1
+$EndComp
+Wire Wire Line
+	12900 1300 12900 1350
+Wire Wire Line
+	12450 1350 12900 1350
+Wire Wire Line
+	12900 1350 13100 1350
+Connection ~ 12900 1350
 $EndSCHEMATC
