File: hardware/ETH1CLCR2/I_Diff_Amp.sch (KiCad schematic (older format))
At the start: 57 parts, among them U1013 MCP6L91RT-ESN, U1014 MCP661, U1015 SN74LVC1G3157, U1016 SN74LVC1G3157, U1017 MCP661, U1018 MCP6L91RT-ESN, U1019 MCP6L91RT-ESN, U1020 SN74LVC1T45DBV, U1021 SN74LVC1G3157, U1022 SN74LVC1G3157, U1023 MCP661, U1024 SN74LVC1T45DBV

Commit message: Footprints assigned.
Parts:
- added C1017, C1018, C1019, C1020: 100n, Capacitor_SMD:C_0603_1608Metric_Pad1.08x0.95mm_HandSolder, symbol Device:C
- added TP1001, TP1002, TP1003, TP1004: TestPoint, TestPoint:TestPoint_Plated_Hole_D2.0mm, symbol Connector:TestPoint
- C1001: renamed from C1019; footprint (none) -> Capacitor_SMD:C_0603_1608Metric_Pad1.08x0.95mm_HandSolder
- C1002: renamed from C1021; footprint (none) -> Capacitor_SMD:C_0603_1608Metric_Pad1.08x0.95mm_HandSolder
- C1003: renamed from C1020; footprint (none) -> Capacitor_SMD:C_0603_1608Metric_Pad1.08x0.95mm_HandSolder
- C1004: renamed from C1023; footprint (none) -> Capacitor_SMD:C_0603_1608Metric_Pad1.08x0.95mm_HandSolder
- C1005: renamed from C1022; footprint (none) -> Capacitor_SMD:C_0603_1608Metric_Pad1.08x0.95mm_HandSolder
- C1006: renamed from C1024; footprint (none) -> Capacitor_SMD:C_0603_1608Metric_Pad1.08x0.95mm_HandSolder
- C1007: renamed from C1025; footprint (none) -> Capacitor_SMD:C_0603_1608Metric_Pad1.08x0.95mm_HandSolder
- C1008: renamed from C1026; footprint (none) -> Capacitor_SMD:C_0603_1608Metric_Pad1.08x0.95mm_HandSolder
- C1009: renamed from C1027; footprint (none) -> Capacitor_SMD:C_0603_1608Metric_Pad1.08x0.95mm_HandSolder
- C1010: renamed from C1028; footprint (none) -> Capacitor_SMD:C_0603_1608Metric_Pad1.08x0.95mm_HandSolder
- C1011: renamed from C1029; footprint (none) -> Capacitor_SMD:C_0603_1608Metric_Pad1.08x0.95mm_HandSolder
- C1012: renamed from C1030; footprint (none) -> Capacitor_SMD:C_0603_1608Metric_Pad1.08x0.95mm_HandSolder
- C1013: renamed from C1031; footprint (none) -> Capacitor_SMD:C_0603_1608Metric_Pad1.08x0.95mm_HandSolder
- C1014: renamed from C1032; footprint (none) -> Capacitor_SMD:C_0603_1608Metric_Pad1.08x0.95mm_HandSolder
- C1015: renamed from C1033; footprint (none) -> Capacitor_SMD:C_0603_1608Metric_Pad1.08x0.95mm_HandSolder
- C1016: renamed from C1034; footprint (none) -> Capacitor_SMD:C_0603_1608Metric_Pad1.08x0.95mm_HandSolder
- FB1001: renamed from FB1002; value Ferrite_Bead_Small -> BLM18TG102TN1D; footprint (none) -> Inductor_SMD:L_0603_1608Metric_Pad1.05x0.95mm_HandSolder
- R1001: renamed from R1030; footprint (none) -> Resistor_SMD:R_0603_1608Metric_Pad0.98x0.95mm_HandSolder
- R1002: renamed from R1031; footprint (none) -> Resistor_SMD:R_0603_1608Metric_Pad0.98x0.95mm_HandSolder
- R1003: renamed from R1032; footprint (none) -> Resistor_SMD:R_0603_1608Metric_Pad0.98x0.95mm_HandSolder
- R1004: renamed from R1033; footprint (none) -> Resistor_SMD:R_0603_1608Metric_Pad0.98x0.95mm_HandSolder
- R1005: renamed from R1034; footprint (none) -> Resistor_SMD:R_0603_1608Metric_Pad0.98x0.95mm_HandSolder
- R1006: renamed from R1035; footprint (none) -> Resistor_SMD:R_0603_1608Metric_Pad0.98x0.95mm_HandSolder
- R1007: renamed from R1036; footprint (none) -> Resistor_SMD:R_0603_1608Metric_Pad0.98x0.95mm_HandSolder
- R1008: renamed from R1038; footprint (none) -> Resistor_SMD:R_0603_1608Metric_Pad0.98x0.95mm_HandSolder
- R1009: renamed from R1039; footprint (none) -> Resistor_SMD:R_0603_1608Metric_Pad0.98x0.95mm_HandSolder
- R1010: renamed from R1040; footprint (none) -> Resistor_SMD:R_0603_1608Metric_Pad0.98x0.95mm_HandSolder
- R1011: renamed from R1041; footprint (none) -> Resistor_SMD:R_0603_1608Metric_Pad0.98x0.95mm_HandSolder
- R1012: renamed from R1037; footprint (none) -> Resistor_SMD:R_0603_1608Metric_Pad0.98x0.95mm_HandSolder
- R1013: renamed from R1042; footprint (none) -> Resistor_SMD:R_0603_1608Metric_Pad0.98x0.95mm_HandSolder
- R1014: renamed from R1043; footprint (none) -> Resistor_SMD:R_0603_1608Metric_Pad0.98x0.95mm_HandSolder
- R1015: renamed from R1044; footprint (none) -> Resistor_SMD:R_0603_1608Metric_Pad0.98x0.95mm_HandSolder
- R1016: renamed from R1046; footprint (none) -> Resistor_SMD:R_0603_1608Metric_Pad0.98x0.95mm_HandSolder
- R1017: renamed from R1047; footprint (none) -> Resistor_SMD:R_0603_1608Metric_Pad0.98x0.95mm_HandSolder
- R1018: renamed from R1048; footprint (none) -> Resistor_SMD:R_0603_1608Metric_Pad0.98x0.95mm_HandSolder
- R1019: renamed from R1049; footprint (none) -> Resistor_SMD:R_0603_1608Metric_Pad0.98x0.95mm_HandSolder
- R1020: renamed from R1045; footprint (none) -> Resistor_SMD:R_0603_1608Metric_Pad0.98x0.95mm_HandSolder
- R1021: renamed from R1050; footprint (none) -> Resistor_SMD:R_0603_1608Metric_Pad0.98x0.95mm_HandSolder
- R1022: renamed from R1051; footprint (none) -> Resistor_SMD:R_0603_1608Metric_Pad0.98x0.95mm_HandSolder
- R1023: renamed from R1052; footprint (none) -> Resistor_SMD:R_0603_1608Metric_Pad0.98x0.95mm_HandSolder
- R1024: renamed from R1053; footprint (none) -> Resistor_SMD:R_0603_1608Metric_Pad0.98x0.95mm_HandSolder
- RV1001: renamed from RV1002; value 20k_POT -> TS53YJ203MR10; footprint (none) -> Potentiometer_SMD:Potentiometer_Vishay_TS53YJ_Vertical
- TP1005: renamed from TP1002; footprint (none) -> TestPoint:TestPoint_Plated_Hole_D2.0mm
- U1002: renamed from U1014; footprint (none) -> Package_SO:SOIC-8_3.9x4.9mm_P1.27mm
- U1003: renamed from U1015; footprint (none) -> Package_TO_SOT_SMD:SOT-23-6_Handsoldering
- U1004: renamed from U1016; footprint (none) -> Package_TO_SOT_SMD:SOT-23-6_Handsoldering
- U1005: renamed from U1017; footprint (none) -> Package_SO:SOIC-8_3.9x4.9mm_P1.27mm
- U1008: renamed from U1021; footprint (none) -> Package_TO_SOT_SMD:SOT-23-6_Handsoldering
- U1009: renamed from U1022; footprint (none) -> Package_TO_SOT_SMD:SOT-23-6_Handsoldering
- U1010: renamed from U1023; footprint (none) -> Package_SO:SOIC-8_3.9x4.9mm_P1.27mm
- renumbered D1004 to D1001, D1005 to D1002, U1013 to U1001, U1018 to U1006, U1020 to U1007, U1019 to U1011, U1024 to U1012
Connections:
- net +3V3: now also C1019.1, C1020.1
- net +5VA: now also C1017.1, C1018.1
- net GND: now also C1017.2, C1018.2, C1019.2, C1020.2
- net at R1009.1, U1002.6, U1003.4 (COM): now also TP1002.1
- net at R1005.2, U1001.2 (-), U1001.6: now also TP1001.1
- net at R1008.2, U1006.2 (-), U1006.6: now also TP1004.1
- net at R1016.1, U1004.4 (COM), U1008.4 (COM): now also TP1003.1

Commit message: Footprints
Parts:
- RV1001: value TS53YJ203MR10 -> 3314J-1-203E; footprint Potentiometer_SMD:Potentiometer_Vishay_TS53YJ_Vertical -> Potentiometer_SMD:Potentiometer_Bourns_3314J_Vertical
Changed lines of the file:
@@
 AR Path="/60FFA72B/61019063" Ref="RV1001"  Part="1"
 F 0 "RV1001" V 3385 6600 50  0000 C CNN
-F 1 "TS53YJ203MR10" V 3294 6600 50  0000 C CNN
-F 2 "Potentiometer_SMD:Potentiometer_Vishay_TS53YJ_Vertical" H 3500 6600 50  0001 C CNN
+F 1 "3314J-1-203E" V 3294 6600 50  0000 C CNN
+F 2 "Potentiometer_SMD:Potentiometer_Bourns_3314J_Vertical" H 3500 6600 50  0001 C CNN
 F 3 "~" H 3500 6600 50  0001 C CNN
 	1    3500 6600

Commit message: PCB
Parts:
- removed C1009: 100n, Capacitor_SMD:C_0603_1608Metric_Pad1.08x0.95mm_HandSolder, symbol Device:C
- TP1001, TP1002, TP1003, TP1004, TP1005: footprint TestPoint:TestPoint_Plated_Hole_D2.0mm -> TestPoint:TestPoint_Pad_1.0x1.0mm
- U1007, U1012: footprint Package_TO_SOT_SMD:SOT-23-6 -> Package_TO_SOT_SMD:SOT-23-6_Handsoldering
- renumbered C1010 to C1009, C1012 to C1010, C1014 to C1011, C1015 to C1012, C1016 to C1013, C1017 to C1014, C1018 to C1015, C1013 to C1016, C1011 to C1017, C1019 to C1018, C1020 to C1019
Connections:
- net +5V: now also C1016.1, C1017.1
- net +5VA: no longer C1016.1, C1017.1
Other:
- moved on the sheet: C1007, C1008, C1010, C1011, C1012, C1013, C1014, C1015, C1016, C1017

Commit message: PCB
Changed lines of the file:
@@
 AR Path="/621B52CA/610190E1" Ref="U?"  Part="1"
 AR Path="/60FFA72B/610190E1" Ref="U1002"  Part="1"
-F 0 "U1002" H 6850 4300 50  0000 L CNN
+F 0 "U1002" H 6800 4300 50  0000 L CNN
 F 1 "MCP661" H 6750 4200 50  0000 L CNN
 F 2 "Package_SO:SOIC-8_3.9x4.9mm_P1.27mm" H 6750 4100 50  0001 C CNN

Commit message: PCB
Parts:
- U1001, U1006, U1011: value MCP6L91RT-ESN -> MCP6L91T-E/SN
- U1002, U1005, U1010: value MCP661 -> MCP661-E/SN
- U1003, U1004, U1008, U1009: value SN74LVC1G3157 -> SN74LVC1G3157DBVR
Other:
- moved on the sheet: TP1002
Changed lines of the file:
@@
 AR Path="/60FFA72B/610190E1" Ref="U1002"  Part="1"
 F 0 "U1002" H 6800 4300 50  0000 L CNN
-F 1 "MCP661" H 6750 4200 50  0000 L CNN
+F 1 "MCP661-E/SN" H 6750 4200 50  0000 L CNN
 F 2 "Package_SO:SOIC-8_3.9x4.9mm_P1.27mm" H 6750 4100 50  0001 C CNN
 F 3 "" H 6750 4200 50  0001 C CNN
@@
 AR Path="/60FFA72B/61019191" Ref="U1005"  Part="1"
 F 0 "U1005" H 10250 4400 50  0000 L CNN
-F 1 "MCP661" H 10150 4300 50  0000 L CNN
+F 1 "MCP661-E/SN" H 10150 4300 50  0000 L CNN
 F 2 "Package_SO:SOIC-8_3.9x4.9mm_P1.27mm" H 10200 4200 50  0001 C CNN
 F 3 "" H 10200 4300 50  0001 C CNN
@@
 AR Path="/60FFA72B/610191D6" Ref="U1003"  Part="1"
 F 0 "U1003" H 8500 4515 50  0000 C CNN
-F 1 "SN74LVC1G3157" H 8500 4424 50  0000 C CNN
+F 1 "SN74LVC1G3157DBVR" H 8500 4424 50  0000 C CNN
 F 2 "Package_TO_SOT_SMD:SOT-23-6_Handsoldering" H 8500 4400 50  0001 C CNN
 F 3 "" H 8500 4400 50  0001 C CNN
@@
 AR Path="/60FFA72B/610191DE" Ref="U1004"  Part="1"
 F 0 "U1004" H 11300 4515 50  0000 C CNN
-F 1 "SN74LVC1G3157" H 11300 4424 50  0000 C CNN
+F 1 "SN74LVC1G3157DBVR" H 11300 4424 50  0000 C CNN
 F 2 "Package_TO_SOT_SMD:SOT-23-6_Handsoldering" H 11300 4400 50  0001 C CNN
 F 3 "" H 11300 4400 50  0001 C CNN
@@
 	8900 4250 8850 4250
 Wire Wire Line
-	8850 3850 8900 3850
-Wire Wire Line
-	8900 3850 8900 3500
-Wire Wire Line
-	8900 3500 10900 3500
-Wire Wire Line
-	10900 3500 10900 3850
-Wire Wire Line
-	10900 3850 10950 3850
+	8850 3850 9000 3850
+Wire Wire Line
+	9000 3850 9000 3500
+Wire Wire Line
+	9000 3500 10800 3500
+Wire Wire Line
+	10800 3500 10800 3850
+Wire Wire Line
+	10800 3850 10950 3850
 $Comp
 L power:+5VA #PWR?
@@
 AR Path="/621B52CA/61019215" Ref="U?"  Part="1"
 AR Path="/60FFA72B/61019215" Ref="U1010"  Part="1"
-F 0 "U1010" H 10250 6800 50  0000 L CNN
-F 1 "MCP661" H 10150 6700 50  0000 L CNN
+F 0 "U1010" H 10150 6800 50  0000 L CNN
+F 1 "MCP661-E/SN" H 10150 6700 50  0000 L CNN
 F 2 "Package_SO:SOIC-8_3.9x4.9mm_P1.27mm" H 10200 6600 50  0001 C CNN
 F 3 "" H 10200 6700 50  0001 C CNN
@@
 AR Path="/60FFA72B/6101925A" Ref="U1008"  Part="1"
 F 0 "U1008" H 8500 6915 50  0000 C CNN
-F 1 "SN74LVC1G3157" H 8500 6824 50  0000 C CNN
+F 1 "SN74LVC1G3157DBVR" H 8500 6824 50  0000 C CNN
 F 2 "Package_TO_SOT_SMD:SOT-23-6_Handsoldering" H 8500 6800 50  0001 C CNN
 F 3 "" H 8500 6800 50  0001 C CNN
@@
 AR Path="/60FFA72B/61019262" Ref="U1009"  Part="1"
 F 0 "U1009" H 11300 6915 50  0000 C CNN
-F 1 "SN74LVC1G3157" H 11300 6824 50  0000 C CNN
+F 1 "SN74LVC1G3157DBVR" H 11300 6824 50  0000 C CNN
 F 2 "Package_TO_SOT_SMD:SOT-23-6_Handsoldering" H 11300 6800 50  0001 C CNN
 F 3 "" H 11300 6800 50  0001 C CNN
@@
 	8900 6650 8850 6650
 Wire Wire Line
-	8850 6250 8900 6250
-Wire Wire Line
-	8900 6250 8900 5900
-Wire Wire Line
-	8900 5900 10900 5900
-Wire Wire Line
-	10900 5900 10900 6250
-Wire Wire Line
-	10900 6250 10950 6250
+	8850 6250 9000 6250
+Wire Wire Line
+	9000 6250 9000 5900
+Wire Wire Line
+	9000 5900 10800 5900
+Wire Wire Line
+	10800 5900 10800 6250
+Wire Wire Line
+	10800 6250 10950 6250
 $Comp
 L power:+5VA #PWR?
@@
 IDIFF0
 Wire Wire Line
-	8150 4050 7250 4050
+	8150 4050 7400 4050
 Connection ~ 7050 4050
 $Comp
@@
 AR Path="/60FFA72B/610192B4" Ref="U1001"  Part="1"
 F 0 "U1001" H 5200 2850 50  0000 L CNN
-F 1 "MCP6L91RT-ESN" H 4950 2750 50  0000 L CNN
+F 1 "MCP6L91T-E/SN" H 4950 2750 50  0000 L CNN
 F 2 "Package_SO:SOIC-8_3.9x4.9mm_P1.27mm" H 4850 2400 50  0001 L CNN
 F 3 "http://ww1.microchip.com/downloads/en/DeviceDoc/22141b.pdf" H 5100 2750 50  0001 C CNN
@@
 AR Path="/60FFA72B/610192BA" Ref="U1006"  Part="1"
 F 0 "U1006" H 5200 5700 50  0000 L CNN
-F 1 "MCP6L91RT-ESN" H 4950 5600 50  0000 L CNN
+F 1 "MCP6L91T-E/SN" H 4950 5600 50  0000 L CNN
 F 2 "Package_SO:SOIC-8_3.9x4.9mm_P1.27mm" H 4850 5250 50  0001 L CNN
 F 3 "http://ww1.microchip.com/downloads/en/DeviceDoc/22141b.pdf" H 5100 5600 50  0001 C CNN
@@
 AR Path="/60FFA72B/610192C0" Ref="U1011"  Part="1"
 F 0 "U1011" H 13750 6800 50  0000 L CNN
-F 1 "MCP6L91RT-ESN" H 13500 6700 50  0000 L CNN
+F 1 "MCP6L91T-E/SN" H 13500 6700 50  0000 L CNN
 F 2 "Package_SO:SOIC-8_3.9x4.9mm_P1.27mm" H 13400 6350 50  0001 L CNN
 F 3 "http://ww1.microchip.com/downloads/en/DeviceDoc/22141b.pdf" H 13650 6700 50  0001 C CNN
@@
 L Connector:TestPoint TP1002
 U 1 1 61006ACB
-P 7250 4000
-F 0 "TP1002" H 7308 4118 50  0000 L CNN
-F 1 "TestPoint" H 7308 4027 50  0000 L CNN
-F 2 "TestPoint:TestPoint_Pad_1.0x1.0mm" H 7450 4000 50  0001 C CNN
-F 3 "~" H 7450 4000 50  0001 C CNN
-	1    7250 4000
-	1    0    0    -1
-$EndComp
-Wire Wire Line
-	7250 4000 7250 4050
-Connection ~ 7250 4050
-Wire Wire Line
-	7250 4050 7050 4050
+P 7400 4000
+F 0 "TP1002" H 7458 4118 50  0000 L CNN
+F 1 "TestPoint" H 7458 4027 50  0000 L CNN
+F 2 "TestPoint:TestPoint_Pad_1.0x1.0mm" H 7600 4000 50  0001 C CNN
+F 3 "~" H 7600 4000 50  0001 C CNN
+	1    7400 4000
+	1    0    0    -1
+$EndComp
+Wire Wire Line
+	7400 4000 7400 4050
+Connection ~ 7400 4050
+Wire Wire Line
+	7400 4050 7050 4050
 $Comp
 L Connector:TestPoint TP1003
