File: hardware/ETH1CLCR2/Reference.sch (KiCad schematic (older format))
At the start: 16 parts, among them U801 REF5040ID, U802 TL431BCDE4, U803 MCP6L91RT-EMS

Commit message: Schematic design
Parts:
- C801: value C -> 1u
- C802: value C -> 10u
- R804: value 33/.1% -> 33/1W
Changed lines of the file:
@@
 $Descr A4 11693 8268
 encoding utf-8
-Sheet 8 10
+Sheet 7 12
 Title ""
 Date ""
@@
 AR Path="/610A8D82/610AB5A8" Ref="C801"  Part="1"
 F 0 "C801" H 2965 2596 50  0000 L CNN
-F 1 "C" H 2965 2505 50  0000 L CNN
+F 1 "1u" H 2965 2505 50  0000 L CNN
 F 2 "" H 2888 2400 50  0001 C CNN
 F 3 "~" H 2850 2550 50  0001 C CNN
@@
 AR Path="/610A8D82/610AB5AE" Ref="C802"  Part="1"
 F 0 "C802" H 3465 2596 50  0000 L CNN
-F 1 "C" H 3465 2505 50  0000 L CNN
+F 1 "10u" H 3465 2505 50  0000 L CNN
 F 2 "" H 3388 2400 50  0001 C CNN
 F 3 "~" H 3350 2550 50  0001 C CNN
@@
 P 3050 4450
 F 0 "R804" V 2843 4450 50  0000 C CNN
-F 1 "33/.1%" V 2934 4450 50  0000 C CNN
+F 1 "33/1W" V 2934 4450 50  0000 C CNN
 F 2 "" V 2980 4450 50  0001 C CNN
 F 3 "~" H 3050 4450 50  0001 C CNN
@@
 Wire Wire Line
 	5850 5000 5750 5000
+Wire Wire Line
+	4800 4150 4950 4150
+Wire Wire Line
+	5350 4150 5350 4700
+$Comp
+L Device:C C803
+U 1 1 610D4EC3
+P 4950 4350
+F 0 "C803" H 5065 4396 50  0000 L CNN
+F 1 "1u" H 5065 4305 50  0000 L CNN
+F 2 "" H 4988 4200 50  0001 C CNN
+F 3 "~" H 4950 4350 50  0001 C CNN
+	1    4950 4350
+	1    0    0    -1
+$EndComp
+$Comp
+L power:GND #PWR0808
+U 1 1 610D55F5
+P 4950 4500
+F 0 "#PWR0808" H 4950 4250 50  0001 C CNN
+F 1 "GND" H 4955 4327 50  0000 C CNN
+F 2 "" H 4950 4500 50  0001 C CNN
+F 3 "" H 4950 4500 50  0001 C CNN
+	1    4950 4500
+	1    0    0    -1
+$EndComp
+Wire Wire Line
+	4950 4200 4950 4150
+Connection ~ 4950 4150
+Wire Wire Line
+	4950 4150 5350 4150
+Connection ~ 3950 4450
+Wire Wire Line
+	3950 4450 3450 4450
+Wire Wire Line
+	3950 4450 4350 4450
+Wire Wire Line
+	3950 4450 3950 3850
+Wire Wire Line
+	3950 3850 6150 3850
+Wire Wire Line
+	5850 5000 6150 5000
+Connection ~ 5850 5000
+$Comp
+L power:+1V5 #PWR0809
+U 1 1 610E7D15
+P 6150 5000
+F 0 "#PWR0809" H 6150 4850 50  0001 C CNN
+F 1 "+1V5" V 6150 5150 50  0000 L CNN
+F 2 "" H 6150 5000 50  0001 C CNN
+F 3 "" H 6150 5000 50  0001 C CNN
+	1    6150 5000
+	0    1    1    0
+$EndComp
+$Comp
+L power:+3.3VP #PWR0727
+U 1 1 60C64194
+P 6150 3850
+F 0 "#PWR0727" H 6300 3800 50  0001 C CNN
+F 1 "+3.3VP" V 6150 4000 50  0000 L CNN
+F 2 "" H 6150 3850 50  0001 C CNN
+F 3 "" H 6150 3850 50  0001 C CNN
+	1    6150 3850
+	0    1    1    0
+$EndComp
 $Comp
 L Device:R R803
@@
 	0    1    1    0
 $EndComp
-Wire Wire Line
-	4800 4150 4950 4150
-Wire Wire Line
-	5350 4150 5350 4700
-$Comp
-L Device:C C803
-U 1 1 610D4EC3
-P 4950 4350
-F 0 "C803" H 5065 4396 50  0000 L CNN
-F 1 "1u" H 5065 4305 50  0000 L CNN
-F 2 "" H 4988 4200 50  0001 C CNN
-F 3 "~" H 4950 4350 50  0001 C CNN
-	1    4950 4350
-	1    0    0    -1
-$EndComp
-$Comp
-L power:GND #PWR0808
-U 1 1 610D55F5
-P 4950 4500
-F 0 "#PWR0808" H 4950 4250 50  0001 C CNN
-F 1 "GND" H 4955 4327 50  0000 C CNN
-F 2 "" H 4950 4500 50  0001 C CNN
-F 3 "" H 4950 4500 50  0001 C CNN
-	1    4950 4500
-	1    0    0    -1
-$EndComp
-Wire Wire Line
-	4950 4200 4950 4150
-Connection ~ 4950 4150
-Wire Wire Line
-	4950 4150 5350 4150
-Connection ~ 3950 4450
-Wire Wire Line
-	3950 4450 3450 4450
-Wire Wire Line
-	3950 4450 4350 4450
-Wire Wire Line
-	3950 4450 3950 3850
-Wire Wire Line
-	3950 3850 6150 3850
-Wire Wire Line
-	5850 5000 6150 5000
-Connection ~ 5850 5000
-$Comp
-L power:+1V5 #PWR0809
-U 1 1 610E7D15
-P 6150 5000
-F 0 "#PWR0809" H 6150 4850 50  0001 C CNN
-F 1 "+1V5" V 6150 5150 50  0000 L CNN
-F 2 "" H 6150 5000 50  0001 C CNN
-F 3 "" H 6150 5000 50  0001 C CNN
-	1    6150 5000
-	0    1    1    0
-$EndComp
-$Comp
-L power:+3.3VP #PWR0807
-U 1 1 610E8785
-P 6150 3850
-F 0 "#PWR0807" H 6300 3800 50  0001 C CNN
-F 1 "+3.3VP" V 6150 4000 50  0000 L CNN
-F 2 "" H 6150 3850 50  0001 C CNN
-F 3 "" H 6150 3850 50  0001 C CNN
-	1    6150 3850
-	0    1    1    0
-$EndComp
+$Comp
+L power:PWR_FLAG #FLG0101
+U 1 1 61EFACEA
+P 5350 4100
+F 0 "#FLG0101" H 5350 4175 50  0001 C CNN
+F 1 "PWR_FLAG" H 5350 4273 50  0000 C CNN
+F 2 "" H 5350 4100 50  0001 C CNN
+F 3 "~" H 5350 4100 50  0001 C CNN
+	1    5350 4100
+	1    0    0    -1
+$EndComp
+Wire Wire Line
+	5350 4100 5350 4150
+Connection ~ 5350 4150
+$Comp
+L power:PWR_FLAG #FLG0701
+U 1 1 61F28C49
+P 3900 3850
+F 0 "#FLG0701" H 3900 3925 50  0001 C CNN
+F 1 "PWR_FLAG" V 3900 3977 50  0000 L CNN
+F 2 "" H 3900 3850 50  0001 C CNN
+F 3 "~" H 3900 3850 50  0001 C CNN
+	1    3900 3850
+	0    -1   -1   0
+$EndComp
+Wire Wire Line
+	3900 3850 3950 3850
+Connection ~ 3950 3850
 $EndSCHEMATC

Commit message: Footprints assigned.
Parts:
- C701: renamed from C801; footprint (none) -> Capacitor_SMD:C_0603_1608Metric_Pad1.08x0.95mm_HandSolder
- C702: renamed from C802; footprint (none) -> Capacitor_SMD:C_0805_2012Metric_Pad1.18x1.45mm_HandSolder
- C703: renamed from C803; footprint (none) -> Capacitor_SMD:C_0603_1608Metric_Pad1.08x0.95mm_HandSolder
- C704: renamed from C804; footprint (none) -> Capacitor_SMD:C_0603_1608Metric_Pad1.08x0.95mm_HandSolder
- C705: renamed from C805; footprint (none) -> Capacitor_SMD:C_0805_2012Metric_Pad1.18x1.45mm_HandSolder
- R701: renamed from R801; footprint (none) -> Resistor_SMD:R_0603_1608Metric_Pad0.98x0.95mm_HandSolder
- R702: renamed from R802; value 3R3 -> 3R3/.5W; footprint (none) -> Resistor_SMD:R_1206_3216Metric_Pad1.30x1.75mm_HandSolder
- R703: renamed from R803; footprint (none) -> Resistor_SMD:R_0603_1608Metric_Pad0.98x0.95mm_HandSolder
- R704: renamed from R804; value 33/1W -> 33/.5W; footprint (none) -> Resistor_SMD:R_1206_3216Metric_Pad1.30x1.75mm_HandSolder
- R705: renamed from R805; footprint (none) -> Resistor_SMD:R_0603_1608Metric_Pad0.98x0.95mm_HandSolder
- R706: renamed from R806; footprint (none) -> Resistor_SMD:R_0603_1608Metric_Pad0.98x0.95mm_HandSolder
- R707: renamed from R807; footprint (none) -> Resistor_SMD:R_0603_1608Metric_Pad0.98x0.95mm_HandSolder
- R708: renamed from R808; footprint (none) -> Resistor_SMD:R_0603_1608Metric_Pad0.98x0.95mm_HandSolder
- renumbered U801 to U701, U802 to U702, U803 to U703

Commit message: PCB
Parts:
- removed U703: MCP6L91RT-EMS, Package_SO:MSOP-8_3x3mm_P0.65mm, symbol Amplifier_Operational:MCP6L91RT-EMS
- added U703: MCP661, Package_SO:SOIC-8_3.9x4.9mm_P1.27mm, symbol ETH1CLCR2:MCP661
Connections:
- net +1V5: now also U703.2 (-), U703.6
- net GND: now also U703.4 (V-)
- net at R706.2, R708.1: now also U703.3 (+)
- net at C703.1, R703.1: now also U703.7 (V+)
Changed lines of the file:
@@
 Wire Wire Line
 	2300 3700 2300 3750
-$Comp
-L Amplifier_Operational:MCP6L91RT-EMS U703
-U 1 1 610D03DA
-P 5450 5000
-F 0 "U703" H 5700 5250 50  0000 L CNN
-F 1 "MCP6L91RT-EMS" H 5450 5150 50  0000 L CNN
-F 2 "Package_SO:MSOP-8_3x3mm_P0.65mm" H 5350 4800 50  0001 L CNN
-F 3 "http://ww1.microchip.com/downloads/en/DeviceDoc/22141b.pdf" H 5600 5150 50  0001 C CNN
-	1    5450 5000
-	1    0    0    -1
-$EndComp
 Wire Wire Line
 	5150 4900 4350 4900
@@
 	3900 3850 3950 3850
 Connection ~ 3950 3850
+$Comp
+L ETH1CLCR2:MCP661 U703
+U 1 1 60E57A4C
+P 5400 5000
+F 0 "U703" H 5550 5250 50  0000 L CNN
+F 1 "MCP661" H 5500 5150 50  0000 L CNN
+F 2 "Package_SO:SOIC-8_3.9x4.9mm_P1.27mm" H 5500 5050 50  0001 C CNN
+F 3 "" H 5500 5150 50  0001 C CNN
+	1    5400 5000
+	1    0    0    -1
+$EndComp
 $EndSCHEMATC

Commit message: PCB
Parts:
- U703: value MCP661 -> MCP661-E/SN
Changed lines of the file:
@@
 P 5400 5000
 F 0 "U703" H 5550 5250 50  0000 L CNN
-F 1 "MCP661" H 5500 5150 50  0000 L CNN
+F 1 "MCP661-E/SN" H 5500 5150 50  0000 L CNN
 F 2 "Package_SO:SOIC-8_3.9x4.9mm_P1.27mm" H 5500 5050 50  0001 C CNN
 F 3 "" H 5500 5150 50  0001 C CNN
