File: hardware/ETH1CLCR2/Connector.sch (KiCad schematic (older format))
At the start: 8 parts, among them J501 C64AC, K501 HE3621A0510, K502 HE3621A0510, K503 HE3621A0510, K504 HE3621A0510, K505 HE3621A0510, U501 ULN2003A

Commit message: Schematic design
Connections:
- net labels added: H_CUR, H_POT, L_CUR, L_POT
Changed lines of the file:
@@
 $Descr A4 11693 8268
 encoding utf-8
-Sheet 5 10
+Sheet 4 12
 Title "Connector"
 Date "2020-03-07"
@@
 	1    0    0    -1
 $EndComp
+$Comp
+L power:GND #PWR0101
+U 1 1 61964568
+P 2400 1750
+F 0 "#PWR0101" H 2400 1500 50  0001 C CNN
+F 1 "GND" V 2405 1622 50  0000 R CNN
+F 2 "" H 2400 1750 50  0001 C CNN
+F 3 "" H 2400 1750 50  0001 C CNN
+	1    2400 1750
+	0    1    1    0
+$EndComp
+Text HLabel 2400 1050 0    50   Input ~ 0
+H_CUR
+Text HLabel 2400 1400 0    50   Input ~ 0
+L_CUR
+Text HLabel 2400 2100 0    50   Input ~ 0
+H_POT
+Text HLabel 2400 2450 0    50   Input ~ 0
+L_POT
 $EndSCHEMATC

Commit message: Footprints assigned.
Parts:
- renumbered C501 to C401, J501 to J401, K501 to K401, K502 to K402, K503 to K403, K504 to K404, K505 to K405, U501 to U401
Changed lines of the file:
@@
 	4250 5050 4300 5050
 $Comp
-L power:Earth #PWR0508
+L power:Earth #PWR0409
 U 1 1 5DECE77F
 P 4250 5050
-F 0 "#PWR0508" H 4250 4800 50  0001 C CNN
+F 0 "#PWR0409" H 4250 4800 50  0001 C CNN
 F 1 "Earth" H 4250 4900 50  0001 C CNN
 F 2 "" H 4250 5050 50  0001 C CNN
@@
 	4350 7100 4300 7100
 $Comp
-L Connector:C64AC J501
+L Connector:C64AC J401
 U 1 1 5DE8758D
 P 4650 4000
-F 0 "J501" H 4830 4096 50  0000 L CNN
+F 0 "J401" H 4830 4096 50  0000 L CNN
 F 1 "C64AC" H 4830 4005 50  0000 L CNN
 F 2 "ETH1CLCR2:Socket_DIN41612-CaseC1-AC-Male-64Pin-2rows" H 4650 4050 50  0001 C CNN
@@
 	4300 4300 4350 4300
 $Comp
-L power:Earth #PWR0507
+L power:Earth #PWR0408
 U 1 1 5DED2C4C
 P 4250 4250
-F 0 "#PWR0507" H 4250 4000 50  0001 C CNN
+F 0 "#PWR0408" H 4250 4000 50  0001 C CNN
 F 1 "Earth" H 4250 4100 50  0001 C CNN
 F 2 "" H 4250 4250 50  0001 C CNN
@@
 	4300 4250 4300 4300
 $Comp
-L power:GNDPWR #PWR0509
+L power:GNDPWR #PWR0410
 U 1 1 607E4852
 P 4250 6150
-F 0 "#PWR0509" H 4250 5950 50  0001 C CNN
+F 0 "#PWR0410" H 4250 5950 50  0001 C CNN
 F 1 "GNDPWR" V 4254 6041 50  0000 R CNN
 F 2 "" H 4250 6100 50  0001 C CNN
@@
 $EndComp
 $Comp
-L power:+24V #PWR0510
+L power:+24V #PWR0411
 U 1 1 607E51D3
 P 4250 6950
-F 0 "#PWR0510" H 4250 6800 50  0001 C CNN
+F 0 "#PWR0411" H 4250 6800 50  0001 C CNN
 F 1 "+24V" V 4265 7078 50  0000 L CNN
 F 2 "" H 4250 6950 50  0001 C CNN
@@
 $EndComp
 $Comp
-L ETH1CLCR2:GND_TRIG #PWR0506
+L ETH1CLCR2:GND_TRIG #PWR0407
 U 1 1 607EBE86
 P 4300 3900
-F 0 "#PWR0506" H 4300 3650 50  0001 C CNN
+F 0 "#PWR0407" H 4300 3650 50  0001 C CNN
 F 1 "GND_TRIG" V 4305 3772 50  0000 R CNN
 F 2 "" H 4300 3900 50  0001 C CNN
@@
 	4300 2100 4350 2100
 $Comp
-L ETH1CLCR2:HE3621A0510 K501
+L ETH1CLCR2:HE3621A0510 K401
 U 1 1 624DD31E
 P 2850 1050
-F 0 "K501" V 3065 1050 50  0000 C CNN
+F 0 "K401" V 3065 1050 50  0000 C CNN
 F 1 "HE3621A0510" V 2974 1050 50  0000 C CNN
 F 2 "ETH1CLCR2:HE360_x-5050462-8" H 3100 1000 50  0001 C CNN
@@
 $EndComp
 $Comp
-L ETH1CLCR2:HE3621A0510 K501
+L ETH1CLCR2:HE3621A0510 K401
 U 2 1 624DE370
 P 5200 1600
-F 0 "K501" H 5278 1646 50  0000 L CNN
+F 0 "K401" H 5278 1646 50  0000 L CNN
 F 1 "HE3621A0510" H 5278 1555 50  0000 L CNN
 F 2 "ETH1CLCR2:HE360_x-5050462-8" H 5450 1550 50  0001 C CNN
@@
 $EndComp
 $Comp
-L ETH1CLCR2:HE3621A0510 K502
+L ETH1CLCR2:HE3621A0510 K402
 U 1 1 624E3116
 P 2850 1400
-F 0 "K502" V 3065 1400 50  0000 C CNN
+F 0 "K402" V 3065 1400 50  0000 C CNN
 F 1 "HE3621A0510" V 2974 1400 50  0000 C CNN
 F 2 "ETH1CLCR2:HE360_x-5050462-8" H 3100 1350 50  0001 C CNN
@@
 $EndComp
 $Comp
-L ETH1CLCR2:HE3621A0510 K502
+L ETH1CLCR2:HE3621A0510 K402
 U 2 1 624E311C
 P 5900 1600
-F 0 "K502" H 5978 1646 50  0000 L CNN
+F 0 "K402" H 5978 1646 50  0000 L CNN
 F 1 "HE3621A0510" H 5978 1555 50  0000 L CNN
 F 2 "ETH1CLCR2:HE360_x-5050462-8" H 6150 1550 50  0001 C CNN
@@
 $EndComp
 $Comp
-L ETH1CLCR2:HE3621A0510 K503
+L ETH1CLCR2:HE3621A0510 K403
 U 1 1 624E50C0
 P 2850 1750
-F 0 "K503" V 3065 1750 50  0000 C CNN
+F 0 "K403" V 3065 1750 50  0000 C CNN
 F 1 "HE3621A0510" V 2974 1750 50  0000 C CNN
 F 2 "ETH1CLCR2:HE360_x-5050462-8" H 3100 1700 50  0001 C CNN
@@
 $EndComp
 $Comp
-L ETH1CLCR2:HE3621A0510 K503
+L ETH1CLCR2:HE3621A0510 K403
 U 2 1 624E50C6
 P 6600 1600
-F 0 "K503" H 6678 1646 50  0000 L CNN
+F 0 "K403" H 6678 1646 50  0000 L CNN
 F 1 "HE3621A0510" H 6678 1555 50  0000 L CNN
 F 2 "ETH1CLCR2:HE360_x-5050462-8" H 6850 1550 50  0001 C CNN
@@
 $EndComp
 $Comp
-L ETH1CLCR2:HE3621A0510 K504
+L ETH1CLCR2:HE3621A0510 K404
 U 1 1 624E7466
 P 2850 2100
-F 0 "K504" V 3065 2100 50  0000 C CNN
+F 0 "K404" V 3065 2100 50  0000 C CNN
 F 1 "HE3621A0510" V 2974 2100 50  0000 C CNN
 F 2 "ETH1CLCR2:HE360_x-5050462-8" H 3100 2050 50  0001 C CNN
@@
 $EndComp
 $Comp
-L ETH1CLCR2:HE3621A0510 K504
+L ETH1CLCR2:HE3621A0510 K404
 U 2 1 624E746C
 P 7300 1600
-F 0 "K504" H 7378 1646 50  0000 L CNN
+F 0 "K404" H 7378 1646 50  0000 L CNN
 F 1 "HE3621A0510" H 7378 1555 50  0000 L CNN
 F 2 "ETH1CLCR2:HE360_x-5050462-8" H 7550 1550 50  0001 C CNN
@@
 $EndComp
 $Comp
-L ETH1CLCR2:HE3621A0510 K505
+L ETH1CLCR2:HE3621A0510 K405
 U 1 1 624E9C1A
 P 2850 2450
-F 0 "K505" V 3065 2450 50  0000 C CNN
+F 0 "K405" V 3065 2450 50  0000 C CNN
 F 1 "HE3621A0510" V 2974 2450 50  0000 C CNN
 F 2 "ETH1CLCR2:HE360_x-5050462-8" H 3100 2400 50  0001 C CNN
@@
 $EndComp
 $Comp
-L ETH1CLCR2:HE3621A0510 K505
+L ETH1CLCR2:HE3621A0510 K405
 U 2 1 624E9C20
 P 8000 1600
-F 0 "K505" H 8078 1646 50  0000 L CNN
+F 0 "K405" H 8078 1646 50  0000 L CNN
 F 1 "HE3621A0510" H 8078 1555 50  0000 L CNN
 F 2 "ETH1CLCR2:HE360_x-5050462-8" H 8250 1550 50  0001 C CNN
@@
 	5900 1400 6600 1400
 $Comp
-L power:+5V #PWR0501
+L power:+5V #PWR0401
 U 1 1 6259093E
 P 6600 1350
-F 0 "#PWR0501" H 6600 1200 50  0001 C CNN
+F 0 "#PWR0401" H 6600 1200 50  0001 C CNN
 F 1 "+5V" H 6615 1523 50  0000 C CNN
 F 2 "" H 6600 1350 50  0001 C CNN
@@
 	6600 1350 6600 1400
 $Comp
-L Transistor_Array:ULN2003A U501
+L Transistor_Array:ULN2003A U401
 U 1 1 625968E5
 P 9400 2000
-F 0 "U501" H 9400 2667 50  0000 C CNN
+F 0 "U401" H 9400 2667 50  0000 C CNN
 F 1 "ULN2003A" H 9400 2576 50  0000 C CNN
 F 2 "Package_SO:TSSOP-16_4.4x5mm_P0.65mm" H 9450 1450 50  0001 L CNN
@@
 $EndComp
 $Comp
-L power:+5V #PWR0502
+L power:+5V #PWR0402
 U 1 1 6259B37C
 P 9000 1600
-F 0 "#PWR0502" H 9000 1450 50  0001 C CNN
+F 0 "#PWR0402" H 9000 1450 50  0001 C CNN
 F 1 "+5V" V 9000 1750 50  0000 L CNN
 F 2 "" H 9000 1600 50  0001 C CNN
@@
 $EndComp
 $Comp
-L power:GND #PWR0505
+L power:GND #PWR0406
 U 1 1 625A0234
 P 9400 2600
-F 0 "#PWR0505" H 9400 2350 50  0001 C CNN
+F 0 "#PWR0406" H 9400 2350 50  0001 C CNN
 F 1 "GND" H 9405 2427 50  0000 C CNN
 F 2 "" H 9400 2600 50  0001 C CNN
@@
 	9850 2200 9800 2200
 $Comp
-L power:GND #PWR0504
+L power:GND #PWR0405
 U 1 1 626006E6
 P 10700 2100
-F 0 "#PWR0504" H 10700 1850 50  0001 C CNN
+F 0 "#PWR0405" H 10700 1850 50  0001 C CNN
 F 1 "GND" H 10705 1927 50  0000 C CNN
 F 2 "" H 10700 2100 50  0001 C CNN
@@
 $EndComp
 $Comp
-L Device:C C501
+L Device:C C401
 U 1 1 626011D0
 P 10700 1950
-F 0 "C501" H 10815 1996 50  0000 L CNN
+F 0 "C401" H 10815 1996 50  0000 L CNN
 F 1 "1u" H 10815 1905 50  0000 L CNN
 F 2 "Capacitor_SMD:C_0603_1608Metric_Pad1.08x0.95mm_HandSolder" H 10738 1800 50  0001 C CNN
@@
 $EndComp
 $Comp
-L power:+5V #PWR0503
+L power:+5V #PWR0404
 U 1 1 626034E9
 P 10700 1800
-F 0 "#PWR0503" H 10700 1650 50  0001 C CNN
+F 0 "#PWR0404" H 10700 1650 50  0001 C CNN
 F 1 "+5V" H 10715 1973 50  0000 C CNN
 F 2 "" H 10700 1800 50  0001 C CNN
@@
 $EndComp
 $Comp
-L power:GND #PWR0101
+L power:GND #PWR0403
 U 1 1 61964568
 P 2400 1750
-F 0 "#PWR0101" H 2400 1500 50  0001 C CNN
+F 0 "#PWR0403" H 2400 1500 50  0001 C CNN
 F 1 "GND" V 2405 1622 50  0000 R CNN
 F 2 "" H 2400 1750 50  0001 C CNN

Commit message: PCB done
Parts:
- added K406: HE3621A0510, ETH1CLCR2:HE360_x-5050462-8, symbol ETH1CLCR2:HE3621A0510
Connections:
- net +5V: now also K406.2
- net CXN_REL1: now also U401.1 (I1); no longer U401.5 (I5)
- net CXN_REL2: now also U401.2 (I2); no longer U401.4 (I4)
- net CXN_REL4: now also U401.4 (I4); no longer U401.2 (I2)
- net CXN_REL5: now also U401.5 (I5); no longer U401.1 (I1)
- net D: now also K404.4
- net E: now also K405.4; no longer K404.4
- net F: now also K406.4; no longer K405.4
- net GND: now also K404.1
- net H_POT: now also K405.1; no longer K404.1
- net L_POT: now also K406.1; no longer K405.1
- net at K401.3: now also U401.16 (O1); no longer U401.12 (O5)
- net at K402.3: now also U401.15 (O2); no longer U401.13 (O4)
- net at K404.3: now also U401.13 (O4); no longer U401.15 (O2)
- net at K405.3: now also U401.12 (O5); no longer U401.16 (O1)
- net at U401.11 (O6): now also K406.3
- net CXN_REL6: now reaches U401.6 (I6)
- no-connect marks 38 -> 36
Other:
- moved on the sheet: J401, K401A, K401B, K402A, K402B, K403A, K404A, K404B, K405A, K405B
