File: hardware/ETH1CLCR2/hardware/ETH1CLCR2/ADC.sch (KiCad schematic (older format))
At the start: 76 parts, among them K501 TQ2SA-5V, Q501 BC847, U501 ADS8681PWR, U502 AD8656, U503 OP1177AR, U504 AD8476_MSOP, U505 ADS8681PWR, U506 CS5361, U507 AD8656, U508 OP1177AR, U509 AD8476_MSOP

Commit message: PCB
Parts:
- added C534, C535, C536: 100n, Capacitor_SMD:C_0603_1608Metric_Pad1.08x0.95mm_HandSolder, symbol Device:C
Connections:
- net +3V3: now also C535.1, C536.1
- net +5V: now also C534.1
- net GND: now also C534.2, C535.2, C536.2
Changed lines of the file:
@@
 P 15000 6650
 F 0 "#PWR0538" H 15000 6500 50  0001 C CNN
-F 1 "+3.3V" H 14950 6800 50  0000 C CNN
+F 1 "+3.3V" H 15000 6800 50  0000 C CNN
 F 2 "" H 15000 6650 50  0001 C CNN
 F 3 "" H 15000 6650 50  0001 C CNN
@@
 Wire Wire Line
 	3250 8400 3750 8400
+$Comp
+L Device:C C535
+U 1 1 60B75A27
+P 9400 2750
+F 0 "C535" H 9515 2796 50  0000 L CNN
+F 1 "100n" H 9515 2705 50  0000 L CNN
+F 2 "Capacitor_SMD:C_0603_1608Metric_Pad1.08x0.95mm_HandSolder" H 9438 2600 50  0001 C CNN
+F 3 "~" H 9400 2750 50  0001 C CNN
+	1    9400 2750
+	1    0    0    -1
+$EndComp
+$Comp
+L Device:C C536
+U 1 1 60B75A2D
+P 9900 2750
+F 0 "C536" H 10015 2796 50  0000 L CNN
+F 1 "100n" H 10015 2705 50  0000 L CNN
+F 2 "Capacitor_SMD:C_0603_1608Metric_Pad1.08x0.95mm_HandSolder" H 9938 2600 50  0001 C CNN
+F 3 "~" H 9900 2750 50  0001 C CNN
+	1    9900 2750
+	1    0    0    -1
+$EndComp
+Wire Wire Line
+	9400 2900 9400 2950
+Wire Wire Line
+	9400 2950 9650 2950
+Wire Wire Line
+	9900 2950 9900 2900
+Wire Wire Line
+	9900 2550 9650 2550
+Wire Wire Line
+	9400 2550 9400 2600
+Wire Wire Line
+	9900 2600 9900 2550
+$Comp
+L power:GND #PWR0555
+U 1 1 60B75A39
+P 9650 3000
+F 0 "#PWR0555" H 9650 2750 50  0001 C CNN
+F 1 "GND" H 9655 2827 50  0000 C CNN
+F 2 "" H 9650 3000 50  0001 C CNN
+F 3 "" H 9650 3000 50  0001 C CNN
+	1    9650 3000
+	1    0    0    -1
+$EndComp
+Wire Wire Line
+	9650 3000 9650 2950
+Connection ~ 9650 2950
+Wire Wire Line
+	9650 2950 9900 2950
+Wire Wire Line
+	9650 2500 9650 2550
+Connection ~ 9650 2550
+Wire Wire Line
+	9650 2550 9400 2550
+$Comp
+L power:+3.3V #PWR0553
+U 1 1 60B75A45
+P 9650 2500
+F 0 "#PWR0553" H 9650 2350 50  0001 C CNN
+F 1 "+3.3V" H 9650 2650 50  0000 C CNN
+F 2 "" H 9650 2500 50  0001 C CNN
+F 3 "" H 9650 2500 50  0001 C CNN
+	1    9650 2500
+	1    0    0    -1
+$EndComp
+$Comp
+L Device:C C534
+U 1 1 60BA4D41
+P 8850 2750
+F 0 "C534" H 8965 2796 50  0000 L CNN
+F 1 "100n" H 8965 2705 50  0000 L CNN
+F 2 "Capacitor_SMD:C_0603_1608Metric_Pad1.08x0.95mm_HandSolder" H 8888 2600 50  0001 C CNN
+F 3 "~" H 8850 2750 50  0001 C CNN
+	1    8850 2750
+	1    0    0    -1
+$EndComp
+$Comp
+L power:GND #PWR0554
+U 1 1 60BA4D4B
+P 8850 3000
+F 0 "#PWR0554" H 8850 2750 50  0001 C CNN
+F 1 "GND" H 8855 2827 50  0000 C CNN
+F 2 "" H 8850 3000 50  0001 C CNN
+F 3 "" H 8850 3000 50  0001 C CNN
+	1    8850 3000
+	1    0    0    -1
+$EndComp
+$Comp
+L power:+5V #PWR0552
+U 1 1 60BA4D54
+P 8850 2500
+F 0 "#PWR0552" H 8850 2350 50  0001 C CNN
+F 1 "+5V" H 8850 2650 50  0000 C CNN
+F 2 "" H 8850 2500 50  0001 C CNN
+F 3 "" H 8850 2500 50  0001 C CNN
+	1    8850 2500
+	1    0    0    -1
+$EndComp
+Wire Wire Line
+	8850 2500 8850 2600
+Wire Wire Line
+	8850 2900 8850 3000
 $EndSCHEMATC

Commit message: Schematic and PCB modifications
Parts:
- added R532, R533, R534, R535: 10k, Resistor_SMD:R_0603_1608Metric_Pad0.98x0.95mm_HandSolder, symbol Device:R
- R501, R517, R518, R530: value 634 -> 634/.1%
- R505, R514, R519, R528: value 91 -> 91/.1%
- R509, R511, R525, R527: value 10k -> 10k/.1%
- U501, U505: value ADS8681PWR -> ADS8681IPWR
Connections:
- net GND: now also R532.2, R534.2; no longer U504.1 (-IN), U504.3 (VCOM), U509.1 (-IN), U509.3 (VCOM)
- new net: R532.1, R533.1, U504.1 (-IN), U504.3 (VCOM)
- new net: R534.1, R535.1, U509.1 (-IN), U509.3 (VCOM)
- new net +1V5: R533.2, R535.2
Changed lines of the file:
@@
 P 13150 1700
 F 0 "U501" H 13750 2250 50  0000 R CNN
-F 1 "ADS8681PWR" H 13950 2150 50  0000 R CNN
+F 1 "ADS8681IPWR" H 13950 2150 50  0000 R CNN
 F 2 "Package_SO:TSSOP-16_4.4x5mm_P0.65mm" H 13150 800 50  0001 C CNN
 F 3 "" H 13200 1950 50  0001 C CNN
@@
 P 13150 3700
 F 0 "U505" H 13750 4250 50  0000 R CNN
-F 1 "ADS8681PWR" H 13950 4150 50  0000 R CNN
+F 1 "ADS8681IPWR" H 13950 4150 50  0000 R CNN
 F 2 "Package_SO:TSSOP-16_4.4x5mm_P0.65mm" H 13150 2800 50  0001 C CNN
 F 3 "" H 13200 3950 50  0001 C CNN
@@
 P 6000 3950
 F 0 "R517" V 6200 3950 50  0000 C CNN
-F 1 "634" V 6100 3950 50  0000 C CNN
+F 1 "634/.1%" V 6100 3950 50  0000 C CNN
 F 2 "Resistor_SMD:R_0603_1608Metric_Pad0.98x0.95mm_HandSolder" V 5930 3950 50  0001 C CNN
 F 3 "~" H 6000 3950 50  0001 C CNN
@@
 P 6600 3100
 F 0 "R514" V 6800 3100 50  0000 C CNN
-F 1 "91" V 6700 3100 50  0000 C CNN
+F 1 "91/.1%" V 6700 3100 50  0000 C CNN
 F 2 "Resistor_SMD:R_0603_1608Metric_Pad0.98x0.95mm_HandSolder" V 6530 3100 50  0001 C CNN
 F 3 "~" H 6600 3100 50  0001 C CNN
@@
 P 5650 2700
 F 0 "R511" H 5720 2746 50  0000 L CNN
-F 1 "10k" H 5720 2655 50  0000 L CNN
+F 1 "10k/.1%" H 5720 2655 50  0000 L CNN
 F 2 "Resistor_SMD:R_0603_1608Metric_Pad0.98x0.95mm_HandSolder" V 5580 2700 50  0001 C CNN
 F 3 "~" H 5650 2700 50  0001 C CNN
@@
 P 5650 2300
 F 0 "R509" H 5720 2346 50  0000 L CNN
-F 1 "10k" H 5720 2255 50  0000 L CNN
+F 1 "10k/.1%" H 5720 2255 50  0000 L CNN
 F 2 "Resistor_SMD:R_0603_1608Metric_Pad0.98x0.95mm_HandSolder" V 5580 2300 50  0001 C CNN
 F 3 "~" H 5650 2300 50  0001 C CNN
@@
 P 6600 1900
 F 0 "R505" V 6393 1900 50  0000 C CNN
-F 1 "91" V 6484 1900 50  0000 C CNN
+F 1 "91/.1%" V 6484 1900 50  0000 C CNN
 F 2 "Resistor_SMD:R_0603_1608Metric_Pad0.98x0.95mm_HandSolder" V 6530 1900 50  0001 C CNN
 F 3 "~" H 6600 1900 50  0001 C CNN
@@
 P 6000 1050
 F 0 "R501" V 5793 1050 50  0000 C CNN
-F 1 "634" V 5884 1050 50  0000 C CNN
+F 1 "634/.1%" V 5884 1050 50  0000 C CNN
 F 2 "Resistor_SMD:R_0603_1608Metric_Pad0.98x0.95mm_HandSolder" V 5930 1050 50  0001 C CNN
 F 3 "~" H 6000 1050 50  0001 C CNN
@@
 	4350 2650 4300 2650
 Wire Wire Line
-	4350 3250 4350 2650
-Wire Wire Line
-	2200 3250 4350 3250
-Wire Wire Line
-	2200 2450 2200 3250
+	4350 3450 4350 2650
+Wire Wire Line
+	2200 3450 4350 3450
+Wire Wire Line
+	2200 2450 2200 3450
 Wire Wire Line
 	2250 2450 2200 2450
 Wire Wire Line
 	3200 2350 2850 2350
-Connection ~ 3150 2650
-Wire Wire Line
-	3150 2850 3150 2650
 $Comp
 L power:GND #PWR0514
 U 1 1 60B6DE2E
-P 3150 2850
-F 0 "#PWR0514" H 3150 2600 50  0001 C CNN
-F 1 "GND" H 3155 2677 50  0000 C CNN
-F 2 "" H 3150 2850 50  0001 C CNN
-F 3 "" H 3150 2850 50  0001 C CNN
-	1    3150 2850
+P 2650 3200
+F 0 "#PWR0514" H 2650 2950 50  0001 C CNN
+F 1 "GND" H 2655 3027 50  0000 C CNN
+F 2 "" H 2650 3200 50  0001 C CNN
+F 3 "" H 2650 3200 50  0001 C CNN
+	1    2650 3200
 	1    0    0    -1
 $EndComp
@@
 P 6000 7250
 F 0 "R530" V 6200 7250 50  0000 C CNN
-F 1 "634" V 6100 7250 50  0000 C CNN
+F 1 "634/.1%" V 6100 7250 50  0000 C CNN
 F 2 "Resistor_SMD:R_0603_1608Metric_Pad0.98x0.95mm_HandSolder" V 5930 7250 50  0001 C CNN
 F 3 "~" H 6000 7250 50  0001 C CNN
@@
 P 6600 6400
 F 0 "R528" V 6800 6400 50  0000 C CNN
-F 1 "91" V 6700 6400 50  0000 C CNN
+F 1 "91/.1%" V 6700 6400 50  0000 C CNN
 F 2 "Resistor_SMD:R_0603_1608Metric_Pad0.98x0.95mm_HandSolder" V 6530 6400 50  0001 C CNN
 F 3 "~" H 6600 6400 50  0001 C CNN
@@
 P 5650 6000
 F 0 "R527" H 5720 6046 50  0000 L CNN
-F 1 "10k" H 5720 5955 50  0000 L CNN
+F 1 "10k/.1%" H 5720 5955 50  0000 L CNN
 F 2 "Resistor_SMD:R_0603_1608Metric_Pad0.98x0.95mm_HandSolder" V 5580 6000 50  0001 C CNN
 F 3 "~" H 5650 6000 50  0001 C CNN
@@
 P 5650 5600
 F 0 "R525" H 5720 5646 50  0000 L CNN
-F 1 "10k" H 5720 5555 50  0000 L CNN
+F 1 "10k/.1%" H 5720 5555 50  0000 L CNN
 F 2 "Resistor_SMD:R_0603_1608Metric_Pad0.98x0.95mm_HandSolder" V 5580 5600 50  0001 C CNN
 F 3 "~" H 5650 5600 50  0001 C CNN
@@
 P 6600 5200
 F 0 "R519" V 6393 5200 50  0000 C CNN
-F 1 "91" V 6484 5200 50  0000 C CNN
+F 1 "91/.1%" V 6484 5200 50  0000 C CNN
 F 2 "Resistor_SMD:R_0603_1608Metric_Pad0.98x0.95mm_HandSolder" V 6530 5200 50  0001 C CNN
 F 3 "~" H 6600 5200 50  0001 C CNN
@@
 P 6000 4350
 F 0 "R518" V 5793 4350 50  0000 C CNN
-F 1 "634" V 5884 4350 50  0000 C CNN
+F 1 "634/.1%" V 5884 4350 50  0000 C CNN
 F 2 "Resistor_SMD:R_0603_1608Metric_Pad0.98x0.95mm_HandSolder" V 5930 4350 50  0001 C CNN
 F 3 "~" H 6000 4350 50  0001 C CNN
@@
 	4350 5950 4300 5950
 Wire Wire Line
-	4350 6550 4350 5950
-Wire Wire Line
-	2200 6550 4350 6550
-Wire Wire Line
-	2200 5750 2200 6550
+	4350 6800 4350 5950
+Wire Wire Line
+	2200 6800 4350 6800
+Wire Wire Line
+	2200 5750 2200 6800
 Wire Wire Line
 	2250 5750 2200 5750
 Wire Wire Line
 	3200 5650 2850 5650
-Connection ~ 3150 5950
-Wire Wire Line
-	3150 6150 3150 5950
-$Comp
-L power:GND #PWR0535
-U 1 1 60E5AA7F
-P 3150 6150
-F 0 "#PWR0535" H 3150 5900 50  0001 C CNN
-F 1 "GND" H 3155 5977 50  0000 C CNN
-F 2 "" H 3150 6150 50  0001 C CNN
-F 3 "" H 3150 6150 50  0001 C CNN
-	1    3150 6150
-	1    0    0    -1
-$EndComp
 Wire Wire Line
 	3150 5800 3200 5800
@@
 Wire Wire Line
 	8850 2900 8850 3000
+$Comp
+L Device:R R532
+U 1 1 60C1082C
+P 2650 3050
+F 0 "R532" H 2720 3096 50  0000 L CNN
+F 1 "10k" H 2720 3005 50  0000 L CNN
+F 2 "Resistor_SMD:R_0603_1608Metric_Pad0.98x0.95mm_HandSolder" V 2580 3050 50  0001 C CNN
+F 3 "~" H 2650 3050 50  0001 C CNN
+	1    2650 3050
+	1    0    0    -1
+$EndComp
+Connection ~ 3150 2500
+Wire Wire Line
+	2650 2500 2650 2900
+Wire Wire Line
+	2650 2500 3150 2500
+$Comp
+L Device:R R533
+U 1 1 60CBA695
+P 3150 3050
+F 0 "R533" H 3220 3096 50  0000 L CNN
+F 1 "10k" H 3220 3005 50  0000 L CNN
+F 2 "Resistor_SMD:R_0603_1608Metric_Pad0.98x0.95mm_HandSolder" V 3080 3050 50  0001 C CNN
+F 3 "~" H 3150 3050 50  0001 C CNN
+	1    3150 3050
+	1    0    0    -1
+$EndComp
+$Comp
+L power:+1V5 #PWR0535
+U 1 1 60CBB004
+P 3150 3200
+F 0 "#PWR0535" H 3150 3050 50  0001 C CNN
+F 1 "+1V5" H 3165 3373 50  0000 C CNN
+F 2 "" H 3150 3200 50  0001 C CNN
+F 3 "" H 3150 3200 50  0001 C CNN
+	1    3150 3200
+	-1   0    0    1
+$EndComp
+Wire Wire Line
+	3150 2900 3150 2650
+$Comp
+L power:GND #PWR0556
+U 1 1 60CEC2A0
+P 2650 6500
+F 0 "#PWR0556" H 2650 6250 50  0001 C CNN
+F 1 "GND" H 2655 6327 50  0000 C CNN
+F 2 "" H 2650 6500 50  0001 C CNN
+F 3 "" H 2650 6500 50  0001 C CNN
+	1    2650 6500
+	1    0    0    -1
+$EndComp
+$Comp
+L Device:R R534
+U 1 1 60CEC2A6
+P 2650 6350
+F 0 "R534" H 2720 6396 50  0000 L CNN
+F 1 "10k" H 2720 6305 50  0000 L CNN
+F 2 "Resistor_SMD:R_0603_1608Metric_Pad0.98x0.95mm_HandSolder" V 2580 6350 50  0001 C CNN
+F 3 "~" H 2650 6350 50  0001 C CNN
+	1    2650 6350
+	1    0    0    -1
+$EndComp
+Wire Wire Line
+	2650 5800 2650 6200
+$Comp
+L Device:R R535
+U 1 1 60CEC2AD
+P 3150 6350
+F 0 "R535" H 3220 6396 50  0000 L CNN
+F 1 "10k" H 3220 6305 50  0000 L CNN
+F 2 "Resistor_SMD:R_0603_1608Metric_Pad0.98x0.95mm_HandSolder" V 3080 6350 50  0001 C CNN
+F 3 "~" H 3150 6350 50  0001 C CNN
+	1    3150 6350
+	1    0    0    -1
+$EndComp
+$Comp
+L power:+1V5 #PWR0557
+U 1 1 60CEC2B3
+P 3150 6500
+F 0 "#PWR0557" H 3150 6350 50  0001 C CNN
+F 1 "+1V5" H 3165 6673 50  0000 C CNN
+F 2 "" H 3150 6500 50  0001 C CNN
+F 3 "" H 3150 6500 50  0001 C CNN
+	1    3150 6500
+	-1   0    0    1
+$EndComp
+Wire Wire Line
+	3150 6200 3150 5950
+Connection ~ 3150 5800
+Wire Wire Line
+	3150 5800 2650 5800
+Connection ~ 3150 5950
+Connection ~ 3150 2650
 $EndSCHEMATC
