File: hardware/ETH1CLCR2/hardware/ETH1CLCR2/I_Diff_Amp.sch (KiCad schematic (older format))
At the start: 64 parts, among them U1001 MCP6L91T-E/SN, U1002 MCP661-E/SN, U1003 SN74LVC1G3157DBVR, U1004 SN74LVC1G3157DBVR, U1005 MCP661-E/SN, U1006 MCP6L91T-E/SN, U1007 SN74LVC1T45DBV, U1008 SN74LVC1G3157DBVR, U1009 SN74LVC1G3157DBVR, U1010 MCP661-E/SN, U1011 MCP6L91T-E/SN, U1012 SN74LVC1T45DBV

Commit message: Schematic and PCB modifications
Other:
- moved on the sheet: R1010, R1022
Changed lines of the file:
@@
 L Device:R R?
 U 1 1 610191A3
-P 9600 4900
+P 9550 4900
 AR Path="/621B52CA/610191A3" Ref="R?"  Part="1"
 AR Path="/60FFA72B/610191A3" Ref="R1010"  Part="1"
-F 0 "R1010" V 9393 4900 50  0000 C CNN
-F 1 "2k/.1%" V 9484 4900 50  0000 C CNN
-F 2 "Resistor_SMD:R_0603_1608Metric_Pad0.98x0.95mm_HandSolder" V 9530 4900 50  0001 C CNN
-F 3 "~" H 9600 4900 50  0001 C CNN
-	1    9600 4900
+F 0 "R1010" V 9343 4900 50  0000 C CNN
+F 1 "2k/.1%" V 9434 4900 50  0000 C CNN
+F 2 "Resistor_SMD:R_0603_1608Metric_Pad0.98x0.95mm_HandSolder" V 9480 4900 50  0001 C CNN
+F 3 "~" H 9550 4900 50  0001 C CNN
+	1    9550 4900
 	0    1    1    0
 $EndComp
@@
 	9800 4250 9800 4900
 Wire Wire Line
-	9800 4900 9750 4900
+	9800 4900 9700 4900
 $Comp
 L Device:R R?
@@
 $EndComp
 Wire Wire Line
-	10150 4900 10050 4900
+	10150 4900 9800 4900
 Connection ~ 9800 4900
 $Comp
@@
 $EndComp
 Wire Wire Line
-	10150 5250 10050 5250
-Wire Wire Line
-	10050 5250 10050 4900
-Connection ~ 10050 4900
-Wire Wire Line
-	10050 4900 9800 4900
+	10150 5250 9800 5250
+Wire Wire Line
+	9800 5250 9800 4900
 Wire Wire Line
 	10450 5250 10550 5250
@@
 Connection ~ 9300 4900
 Wire Wire Line
-	9300 4900 9450 4900
+	9300 4900 9400 4900
 Wire Wire Line
 	9300 4300 9300 4050
@@
 L Device:R R?
 U 1 1 61019227
-P 9600 7300
+P 9550 7300
 AR Path="/621B52CA/61019227" Ref="R?"  Part="1"
 AR Path="/60FFA72B/61019227" Ref="R1022"  Part="1"
-F 0 "R1022" V 9393 7300 50  0000 C CNN
-F 1 "2k/.1%" V 9484 7300 50  0000 C CNN
-F 2 "Resistor_SMD:R_0603_1608Metric_Pad0.98x0.95mm_HandSolder" V 9530 7300 50  0001 C CNN
-F 3 "~" H 9600 7300 50  0001 C CNN
-	1    9600 7300
+F 0 "R1022" V 9343 7300 50  0000 C CNN
+F 1 "2k/.1%" V 9434 7300 50  0000 C CNN
+F 2 "Resistor_SMD:R_0603_1608Metric_Pad0.98x0.95mm_HandSolder" V 9480 7300 50  0001 C CNN
+F 3 "~" H 9550 7300 50  0001 C CNN
+	1    9550 7300
 	0    1    1    0
 $EndComp
@@
 	9800 6650 9800 7300
 Wire Wire Line
-	9800 7300 9750 7300
+	9800 7300 9700 7300
 $Comp
 L Device:R R?
@@
 $EndComp
 Wire Wire Line
-	10150 7300 10050 7300
+	10150 7300 9800 7300
 Connection ~ 9800 7300
 $Comp
@@
 $EndComp
 Wire Wire Line
-	10150 7650 10050 7650
-Wire Wire Line
-	10050 7650 10050 7300
-Connection ~ 10050 7300
-Wire Wire Line
-	10050 7300 9800 7300
+	10150 7650 9800 7650
+Wire Wire Line
+	9800 7650 9800 7300
 Wire Wire Line
 	10450 7650 10550 7650
@@
 Connection ~ 9300 7300
 Wire Wire Line
-	9300 7300 9450 7300
+	9300 7300 9400 7300
 Wire Wire Line
 	9300 6700 9300 6450
