File: hardware/ETH1CLCR2/hardware/ETH1CLCR2/V_Diff_Amp.sch (KiCad schematic (older format))
At the start: 83 parts, among them K801 TQ2SA-5V, Q801 BC847, U801 MCP6L91T-E/SN, U802 MCP661-E/SN, U803 MCP661-E/SN, U804 SN74LVC1G3157DBVR, U805 SN74LVC1G3157DBVR, U806 MCP661-E/SN, U807 MCP6L91T-E/SN, U808 MCP661-E/SN, U809 SN74LVC1T45DBV, U810 SN74LVC1G3157DBVR, U811 SN74LVC1G3157DBVR, U812 MCP661-E/SN, U813 MCP6L91T-E/SN, U814 SN74LVC1T45DBV, U815 SN74LVC1T45DBV

Commit message: Schematic and PCB modifications
Other:
- moved on the sheet: R816, R829
Changed lines of the file:
@@
 L Device:R R816
 U 1 1 60C97EBC
-P 9950 4600
-F 0 "R816" V 9743 4600 50  0000 C CNN
-F 1 "2k/.1%" V 9834 4600 50  0000 C CNN
-F 2 "Resistor_SMD:R_0603_1608Metric_Pad0.98x0.95mm_HandSolder" V 9880 4600 50  0001 C CNN
-F 3 "~" H 9950 4600 50  0001 C CNN
-	1    9950 4600
+P 9900 4600
+F 0 "R816" V 9693 4600 50  0000 C CNN
+F 1 "2k/.1%" V 9784 4600 50  0000 C CNN
+F 2 "Resistor_SMD:R_0603_1608Metric_Pad0.98x0.95mm_HandSolder" V 9830 4600 50  0001 C CNN
+F 3 "~" H 9900 4600 50  0001 C CNN
+	1    9900 4600
 	0    1    1    0
 $EndComp
@@
 	10150 3950 10150 4600
 Wire Wire Line
-	10150 4600 10100 4600
+	10150 4600 10050 4600
 $Comp
 L Device:R R817
@@
 $EndComp
 Wire Wire Line
-	10500 4600 10400 4600
+	10500 4600 10150 4600
 Connection ~ 10150 4600
 $Comp
@@
 $EndComp
 Wire Wire Line
-	10500 4950 10400 4950
-Wire Wire Line
-	10400 4950 10400 4600
-Connection ~ 10400 4600
-Wire Wire Line
-	10400 4600 10150 4600
+	10500 4950 10150 4950
+Wire Wire Line
+	10150 4950 10150 4600
 Wire Wire Line
 	10800 4950 10900 4950
@@
 Connection ~ 9650 4600
 Wire Wire Line
-	9650 4600 9800 4600
+	9650 4600 9750 4600
 Wire Wire Line
 	9650 4000 9650 3750
@@
 L Device:R R829
 U 1 1 60D37BF3
-P 9950 7000
-F 0 "R829" V 9743 7000 50  0000 C CNN
-F 1 "2k/.1%" V 9834 7000 50  0000 C CNN
-F 2 "Resistor_SMD:R_0603_1608Metric_Pad0.98x0.95mm_HandSolder" V 9880 7000 50  0001 C CNN
-F 3 "~" H 9950 7000 50  0001 C CNN
-	1    9950 7000
+P 9900 7000
+F 0 "R829" V 9693 7000 50  0000 C CNN
+F 1 "2k/.1%" V 9784 7000 50  0000 C CNN
+F 2 "Resistor_SMD:R_0603_1608Metric_Pad0.98x0.95mm_HandSolder" V 9830 7000 50  0001 C CNN
+F 3 "~" H 9900 7000 50  0001 C CNN
+	1    9900 7000
 	0    1    1    0
 $EndComp
@@
 	10150 6350 10150 7000
 Wire Wire Line
-	10150 7000 10100 7000
+	10150 7000 10050 7000
 $Comp
 L Device:R R830
@@
 $EndComp
 Wire Wire Line
-	10500 7000 10400 7000
+	10500 7000 10150 7000
 Connection ~ 10150 7000
 $Comp
@@
 $EndComp
 Wire Wire Line
-	10500 7350 10400 7350
-Wire Wire Line
-	10400 7350 10400 7000
-Connection ~ 10400 7000
-Wire Wire Line
-	10400 7000 10150 7000
+	10500 7350 10150 7350
+Wire Wire Line
+	10150 7350 10150 7000
 Wire Wire Line
 	10800 7350 10900 7350
@@
 Connection ~ 9650 7000
 Wire Wire Line
-	9650 7000 9800 7000
+	9650 7000 9750 7000
 Wire Wire Line
 	9650 6400 9650 6150
